File: sat-receiver-audit/build/kicad/E1.kicad_sch (KiCad schematic)
At the start: 0 parts

Commit message: Complete SR-RX-v2.1 schematics and verification package
Replace five empty sheets with reviewed KiCad schematics and portable resources. Correct power, control, USB and RF interfaces; document hardware acceptance gates and unimplemented firmware/PCB work. Validate 754 components, 2189 connected contacts and 466 nets with zero ERC violations and two independent graph/netlist comparisons. Include PDF, SVG, BOM, reproducible tools and offline documentation.
Parts:
- added BT101: Molicel INR21700-P50B 5Ah, symbol sr_rx_v2_completed:C_BT101
- added BT102: Molicel INR21700-P50B 5Ah, symbol sr_rx_v2_completed:C_BT102
- added BT103: Molicel INR21700-P50B 5Ah, symbol sr_rx_v2_completed:C_BT103
- added BT104: Molicel INR21700-P50B 5Ah, symbol sr_rx_v2_completed:C_BT104
- added C101: 100 nF (Adafruit C1), symbol sr_rx_v2_completed:C_C101
- added C102: 10 µF (Adafruit C2), symbol sr_rx_v2_completed:C_C102
- added C103: 2.2µF50VX7R (effective≥1µF), symbol sr_rx_v2_completed:C_C103
- added C104: 4.7µF10VX7R (effective≥2.2µF), symbol sr_rx_v2_completed:C_C104
- added C105: 100nF10VX7R, symbol sr_rx_v2_completed:C_C105
- added C106: 100nF10VX7R, symbol sr_rx_v2_completed:C_C106
- added C107: 100µF35VlowESR, symbol sr_rx_v2_completed:C_C107
- added C108: 1µF50VX7R, symbol sr_rx_v2_completed:C_C108
- added C109: 100µF35VlowESR, symbol sr_rx_v2_completed:C_C109
- added C110: 1µF50VX7R, symbol sr_rx_v2_completed:C_C110
- added C111: 35SVPF22M 22 µF 35 V ±20% OS-CON, symbol sr_rx_v2_completed:C_C111
- added C112: 35SVPF22M 22 µF 35 V ±20% OS-CON, symbol sr_rx_v2_completed:C_C112
- added C113: 16SVPC100M 100 µF 16 V ±20% OS-CON, symbol sr_rx_v2_completed:C_C113
- added C114: 100nF10V, symbol sr_rx_v2_completed:C_C114
- added D101: BAT54,215, Package_TO_SOT_SMD:SOT-23, symbol sr_rx_v2_completed:C_D101
- added D102: BAT54,215, Package_TO_SOT_SMD:SOT-23, symbol sr_rx_v2_completed:C_D102
- added D103: BAT54,215, Package_TO_SOT_SMD:SOT-23, symbol sr_rx_v2_completed:C_D103
- added D104: SMBJ17A-E3/52, symbol sr_rx_v2_completed:C_D104
- added D105: SMBJ17A-E3/52, symbol sr_rx_v2_completed:C_D105
- added F101: Mini-blade 7.5 A DC ≥32 V, symbol sr_rx_v2_completed:C_F101
- added F102: 4 A DC ≥32 V LAB5, symbol sr_rx_v2_completed:C_F102
- added F103: 5A DC≥32V service, symbol sr_rx_v2_completed:C_F103
- added J101: XT30 сервісний заряд/розряд, symbol sr_rx_v2_completed:C_J101
- added J102: DNP — зовнішній balance 4S (GATE), symbol sr_rx_v2_completed:C_J102
- added J103: USB-C PD заряд, symbol sr_rx_v2_completed:C_J103
- added L101: XAL6060-103MEC 10 µH ±20%, symbol sr_rx_v2_completed:C_L101
- added R101: 15 mΩ 1% 2 W (Adafruit R1), symbol sr_rx_v2_completed:C_R101
- added R102: 10k1%, symbol sr_rx_v2_completed:C_R102
- added R103: 3.30M0.1%25ppm, symbol sr_rx_v2_completed:C_R103
- added R104: 332k0.1%25ppm, symbol sr_rx_v2_completed:C_R104
- added R105: 4.02k0.1%25ppm TRIM, symbol sr_rx_v2_completed:C_R105
- added R106: 100k1%, symbol sr_rx_v2_completed:C_R106
- added R107: 4.22M1%, symbol sr_rx_v2_completed:C_R107
- added R108: 10.0k1%, symbol sr_rx_v2_completed:C_R108
- added R109: 1.00k1%, symbol sr_rx_v2_completed:C_R109
- added R110: WSL2512R3300FEA 0.330 Ω 1%, symbol sr_rx_v2_completed:C_R110
- added R111: 100k1%, symbol sr_rx_v2_completed:C_R111
- added R112: 20.0k1%, symbol sr_rx_v2_completed:C_R112
- added TP101: PG_SYS12резерв, symbol sr_rx_v2_completed:C_TP101
- added TP102: PG_LAB5резерв, symbol sr_rx_v2_completed:C_TP102
- added U101: Daly DL-J05G-L4S15ATJ 4S15A, symbol sr_rx_v2_completed:C_U101
- added U102: INA228AIDGSR на Adafruit 5832, Package_SO:MSOP-10_3x3mm_P0.5mm, symbol sr_rx_v2_completed:C_U102
- added U103: TPS70933DBVR, Package_TO_SOT_SMD:SOT-23-5, symbol sr_rx_v2_completed:C_U103
- added U104: MCP65R41T-1202E/CHY, Package_TO_SOT_SMD:SOT-23-6, symbol sr_rx_v2_completed:C_U104
- added U106: Pololu 2813 HP, symbol sr_rx_v2_completed:C_U106
- added U107: Pololu D36V50F12#4095, symbol sr_rx_v2_completed:C_U107
- added U108: Pololu D36V50F5 #4091 — LAB5 default, symbol sr_rx_v2_completed:C_U108
Connections:
- new net 3V3_Q6A: R102.1
- new net AON3V3: C101.1, C102.1, C104.1, C105.1, U102.6 (VS), U103.5 (OUT), U104.6 (VDD)
- new net CHASSIS: J103.SHIELD
- new net E1_BAT_ADC: C114.1, R111.2, R112.1
- new net E1_CELL0: BT101.- (−), J102.B0, U101.B- (B− силовий), U101.B0 (sense B0)
- new net E1_CELL1: BT101.+, BT102.- (−), J102.B1, U101.B1 (sense B1)
- new net E1_CELL2: BT102.+, BT103.- (−), J102.B2, U101.B2 (sense B2)
- new net E1_CELL3: BT103.+, BT104.- (−), J102.B3, U101.B3 (sense B3)
- new net E1_CELL4: BT104.+, F101.1, J102.B4, U101.B4 (sense B4)
- new net E1_CHG_CC1: J103.CC1
- new net E1_CHG_CC2: J103.CC2
- new net E1_EN_SYS12: R108.2, R109.1, U107.EN
- new net E1_LAB5_DAMP: C113.1 (+), R110.2
- new net E1_LAB5_FUSED: C111.1 (+), F102.2, L101.1
- new net E1_LAB5_RAW: F102.1, U108.VOUT
- new net E1_MASTER_OFF: D101.3 (K), D102.3 (K), U106.OFF
- new net E1_N: C103.1, D104.K, F103.1, R101.2, R103.1, U102.9 (IN−), U103.1 (IN), U106.VIN
- new net E1_PG_LAB5: TP102.1 (PG), U108.PG
- new net E1_PG_SYS12: TP101.1 (PG), U107.PG
- new net E1_SERVICE_P: F103.2, J101.+
- new net E1_SHUNT_P: F101.2, R101.1, U102.10 (IN+), U102.8 (VBUS)
- new net E1_SW: C107.1, C108.1, C109.1, C110.1, D105.K, R108.1, R111.1, U106.VOUT, U107.VIN, U108.VIN
- new net E1_SWITCH_A: D103.1 (A), U106.A
- new net E1_USB_PD_RAW: J103.VBUS
- new net E1_UV_OFF: D101.1 (A), R107.1, U104.1 (OUT)
- new net E1_UV_REF: R106.1, U104.5 (VREF 1.21 V)
- new net E1_UV_REFH: R106.2, R107.2, U104.3 (IN+)
- new net E1_UV_SENSE: C106.1, R103.2, R104.1, U104.4 (IN−)
- new net E1_UV_TRIM: R104.2, R105.1
- new net GND: C101.2, C102.2, C103.2, C104.2, C105.2, C106.2, C107.2, C108.2, C109.2, C110.2, C111.2 (−), C112.2 (−), C113.2 (−), C114.2, D104.A, D105.A, J101.- (−), J103.GND, R105.2, R109.2, R112.2, U101.P- (P− силовий), U102.1 (A1), U102.2 (A0), U102.7 (GND), U103.2 (GND), U104.2 (VSS), U106.GND, U107.GND, U108.GND
- new net I2C0_SCL: U102.5 (SCL)
- new net I2C0_SDA: U102.4 (SDA)
- new net INA228_ALERT: R102.2, U102.3 (ALERT)
- new net LAB5: C112.1 (+), L101.2, R110.1
- new net PICO_OFF: D102.1 (A)
- new net PWR_BUTTON: D103.3 (K)
- new net SYS12: U107.VOUT
- no-connect marks 0 -> 11
Other:
- note added: "AON і UV"
- note added: "E1 - Акумулятор, заряд, AON і головні перетворювачі (1/2)"
- note added: "LAB5"
- note added: "SYS12"
- note added: "Аварійний ADC"
- note added: "Головний вимикач"
- note added: "Заряд IP2368"
- note added: "Лічильник заряду"
- note added: "Мережі з однаковими глобальними мітками електрично з'єднані на всіх аркушах. Фізичні/функціональні контакти: див. design/ і OPEN_ITEMS.md."
- note added: "Пак 4S1P"
- note added: "Сервісний заряд"
- company: (none) -> SR-RX-v2
- title: (none) -> E1 - Акумулятор, заряд, AON і головні перетворювачі (1/2)
