File: sat-receiver-audit/build/kicad/E1.kicad_sch (KiCad schematic)
At the start: 51 parts, among them J101 XT30 сервісний заряд/розряд, J102 DNP — зовнішній balance 4S (G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, J103 USB-C PD заряд, U101 Daly DL-J05G-L4S15ATJ 4S15A, U102 INA228AIDGSR на Adafruit 5832, U103 TPS70933DBVR, U104 MCP65R41T-1202E/CHY, U106 Pololu 2813 HP, U107 Pololu D36V50F12#4095, U108 Pololu D36V50F5 #4091 — LAB5 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

Commit message: WIP: integration follow-ups
Made by the GPT/Codex run on 23.10.2026 (pushed as 5455b1e under the name "Claude");
re-attributed to Codex when integrated into ccr-1537979d-cj7q9t.
Parts:
- R102: now not fitted
Changed lines of the file:
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@@
 (wire (pts (xy 91.44 281.94) (xy 93.98 281.94)) (stroke (width 0) (type default)))
 (global_label "GND" (shape bidirectional) (at 93.98 281.94 0) (effects (font (size 0.889 0.889)) (justify left)) (property "Intersheetrefs" "${INTERSHEET_REFS}" (at 93.98 281.94 0) (effects (font (size 1.016 1.016)) (hide yes))))
-(symbol (lib_id "sr_rx_v2_completed:C_R102") (at 81.28 303.53 0) (unit 1) (exclude_from_sim no) (in_bom yes) (on_board yes) (dnp no)
+(symbol (lib_id "sr_rx_v2_completed:C_R102") (at 81.28 303.53 0) (unit 1) (exclude_from_sim no) (in_bom yes) (on_board yes) (dnp yes)
 (property "Reference" "R102" (at 81.28 293.37 0) (effects (font (size 1.27 1.27)) ))
 (property "Value" "10k1%" (at 81.28 296.545 0) (effects (font (size 1.016 1.016)) ))
