File: sat-receiver-audit/build/kicad/E1.kicad_sch (KiCad schematic)
At the start: 51 parts, among them J101 XT30 сервісний заряд/розряд, J102 DNP — зовнішній balance 4S (G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, J103 USB-C PD заряд, U101 Daly DL-J05G-L4S15ATJ 4S15A, U102 INA228AIDGSR на Adafruit 5832, U103 TPS70933DBVR, U104 MCP65R41T-1202E/CHY, U106 Pololu 2813 HP, U107 Pololu D36V50F12#4095, U108 Pololu D36V50F5 #4091 — LAB5 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

Commit message: SR-RX-v2.1: review fixes on the Codex branch, readable schematic, one-file bundle
Independent review of the Codex branch (schematic vs STACK.md, hard rules,
security, tests) found no blockers; this commit applies its findings:

- rules in code: Cospas-Sarsat 406.0-406.1 MHz added to the no-data mask;
  Q6A Wi-Fi/BT off in the field/QUIET root (modprobe blacklist, udev
  authorized=0 on FE1.1s port 4, rfkill) with self-checks; device denylist
  completed per STACK (gr-gsm, gr-iridium, kalibrate, pager/trunking decoders,
  TX-capable tools); W1-2 WIFI_PWR_EN as blocking open item E5-10
- STACK.md is the source of truth again; v2.1 changes recorded in it; the
  "historical" marker kept only on ISDT/raw-balance rows; gender-neutral wording
- schematic data: open values shown as TBD with start values and notes, U503
  TPS2553DBVR-1, Lime X2/X4 RX mapping TBD, 37 open items drawn on the sheets
- schematic readability: wired groups, junctions, GND symbols, standard
  transistor/diode symbols; netlist unchanged (603 nets identical)
- tooling: reproducible run_checks (no timestamps or machine paths), pinned
  dependencies, bundle excludes cache folders, clean-checkout bundle check
- regenerated: KiCad export (14 pages), netlist/ERC, module lab, PCB inputs,
  readiness contract, acceptance hashes, SR-RX-v2-ves-proekt.html

Checks: ERC 0 errors/0 warnings, netlist comparison PASS, 432 tests (431
passed, 1 skipped), deployment tests OK, bundle check PASS on a clean checkout.

History note: earlier versions of the generated SR-RX-v2-ves-proekt.html and
handoff/handoff-bundle.zip were removed from history; only the final versions
are kept. The Codex merge commit is now attributed to Codex.

Co-Authored-By: Claude Opus 5.5 <noreply@anthropic.com>
Claude-Session: https://claude.ai/code/session_01W9CKpimWpgkUmrDQQMiKtF
Parts:
- removed R102: 10k1%, symbol sr_rx_v2_completed:C_R102
- added C115: 3.3nF50VC0G, symbol sr_rx_v2_completed:C_C115
- added C116: 1µF50VX7R, symbol sr_rx_v2_completed:C_C116
- added C117: 1µF50VX7R, symbol sr_rx_v2_completed:C_C117
- added C118: 100nF50VnearNTCpad, symbol sr_rx_v2_completed:C_C118
- added Q101: 2N7002,215, Package_TO_SOT_SMD:SOT-23, symbol sr_rx_v2_completed:C_Q101
- added R113: 470k1%, symbol sr_rx_v2_completed:C_R113
- added R114: 174k0.1%, symbol sr_rx_v2_completed:C_R114
- added R115: 10.0k0.1%, symbol sr_rx_v2_completed:C_R115
- added R116: 953Ω1%, symbol sr_rx_v2_completed:C_R116
- added R117: 5.10k1% replacesR4, symbol sr_rx_v2_completed:C_R117
- added R118: 15.0k1% replacesR3, symbol sr_rx_v2_completed:C_R118
- added R119: 1.00k1% ISET_MODE, symbol sr_rx_v2_completed:C_R119
- added R120: 13.0k1%4Scellset, symbol sr_rx_v2_completed:C_R120
- added R121: 2.20k1%, symbol sr_rx_v2_completed:C_R121
- added R122: 1.00k1%, symbol sr_rx_v2_completed:C_R122
- added R123: 100k1%, symbol sr_rx_v2_completed:C_R123
- added TH101: NTC 10 kΩ B3380 при 25 °C, symbol sr_rx_v2_completed:C_TH101
- added TH102: KSD9700 70 °C NO, symbol sr_rx_v2_completed:C_TH102
- added TP103: PD_FLT service, symbol sr_rx_v2_completed:C_TP103
- added TP104: ВузолN, symbol sr_rx_v2_completed:C_TP104
- added TP105: ВузолSW, symbol sr_rx_v2_completed:C_TP105
- added TP106: AON3V3, symbol sr_rx_v2_completed:C_TP106
- added TP107: Protectedground, symbol sr_rx_v2_completed:C_TP107
- added TP108: UV_OFF, symbol sr_rx_v2_completed:C_TP108
- added U109: TPS259470ARPWR USB-C, symbol sr_rx_v2_completed:C_U109
- added U110: IP2368 COUT 4S retail board, symbol sr_rx_v2_completed:C_U110
Connections:
- net AON3V3: now also TP106.1 (AON3V3)
- net E1_CHG_CC1: now also U110.CC1
- net E1_CHG_CC2: now also U110.CC2
- net E1_N: now also TP104.1 (ВузолN), U110.BAT+
- net E1_SW: now also TP105.1 (ВузолSW)
- net E1_USB_PD_RAW: now also C116.1, R113.1, R114.1, U109.5 (IN)
- net E1_UV_OFF: now also TP108.1 (UV_OFF)
- net GND: now also C115.2, C116.2, C117.2, C118.2, Q101.2 (S), R115.2, R116.2, R117.2, R118.2, R119.2, R120.2, R123.2, TH101.2, TH102.2, TP107.1 (Protectedground), U109.8 (GND), U110.BAT- (BAT−)
- new net CHG_INHIBIT: R122.1
- new net E1_CHG_CELLSET: R120.1, U110.CELLSET (CELLSET modification node)
- new net E1_CHG_GATE: Q101.1 (G), R122.2, R123.1
- new net E1_CHG_INHIBIT_LOW: Q101.3 (D), R121.2, TH102.1
- new net E1_CHG_ISET: R118.1, U110.ISET (ISET modification node)
- new net E1_CHG_ISETMODE: R119.1, U110.ISET_MODE (ISET_MODE modification node)
- new net E1_CHG_NTC: C118.1, R121.1, TH101.1, U110.NTC (NTC modification node)
- new net E1_CHG_VSET: R117.1, U110.VSET (VSET modification node)
- new net E1_PD_DVDT: C115.1, U109.7 (DVDT)
- new net E1_PD_EN: R113.2, U109.1 (EN/UVLO)
- new net E1_PD_FLT: TP103.1 (FLT), U109.4 (FLT)
- new net E1_PD_ILM: R116.1, U109.9 (ILM)
- new net E1_PD_OVLO: R114.2, R115.1, U109.2 (OVLO)
- new net E1_USB_PD_SAFE: C117.1, U109.6 (OUT), U110.VBUS (VBUS після eFuse)
- no-connect marks 11 -> 13
Other:
- note added: "Balance B0 = raw B− може шунтувати Daly через спільну землю ISDT 608PD і пропускати силовий струм по тонкому sense-дроту. Ворота (стенд): J102 позначено DNP/service-only; місячний баланс ISDT вимкнути до затвердженого інтерфейсу. До підключення перевірити DMM ізоляцію output−/balance B0 ISDT без живлення та отримати принципову схему виробника. При спільній землі потрібне перепроєктування з явним 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"
- note added: "Default LAB5: D36V50F5 +4 A fuse; конкретні parts фільтра обрані. Агрегатний струм, converter/filter stability, температура і напруги на кінцевих навантаженнях не підтверджені. Ворота (стенд): U108 D36V50F5 #4091; F102 4 A; L101 XAL6060-103MEC; C111/C112 35SVPF22M; C113 16SVPC100M; R110 WSL2512R3300FEA. Звірити площу, висоту і land patterns. Виміряти всі режими: LAB5 ≤3.2 A continuous; blower res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"
- note added: "E1 - Акумулятор, заряд, AON і головні перетворювачі (1/1)"
- note added: "E1-01 — OPEN, блокує випуск — STACK §2.7 (IP2368); §5.1; §8 (IP2368); §8.1 (IP2368, матриця DRP)"
- note added: "E1-02 — OPEN, блокує випуск — STACK §2.7; §5.1; §8 (Daly DL-J05G; ISDT 608PD)"
- note added: "E1-03 — OPEN, блокує випуск — STACK §2.7 (Daly); §8 (Daly DL-J05G)"
- note added: "E1-04 — OPEN, блокує випуск — STACK §5.1 (AON, UV); §8 (Супервізор AON)"
- note added: "E1-05 — OPEN, блокує випуск — STACK §5.1 (LAB5); §8 (LAB5); §8.1 (нагрів запобіжників)"
- note added: "E1-06 — OPEN, блокує випуск — STACK §5.1; §5.6; §8.1 (J21 і USB-C; просідання дисплея і Q6A)"
- note added: "E1-07 — OPEN, блокує випуск — STACK §5.8; §8 (PCB, P5 G3)"
- note added: "USB-C feedthrough, XT30 та BMS мають функціональні контакти; механічні parts і land patterns не задано. Ворота (стенд): Перед PCB вибрати конкретні частини, відобразити їхні фізичні контакти на functional nets і незалежно перевірити pin mapping. Ця JSON описує схему, а не Gerber."
- note added: "UV ±0.1 V потребує індивідуальної калібровки; held OFF проти кнопки ще не перевірено. Ворота (стенд): До батареї current-limited sweep 14→12→14 V при 25 і 50 °C: trip 12.8±0.1 V, release 13.6±0.1 V, drift≤50 mV. Калібрувати R105. AON без INA ≤11 µA. Утримуванням кнопки не можна обійти UV. 20 PD cycles без самозапуску. При провалі fallback TLV3012 із нижнім плечем 346.04 kΩ і повним повтором тесту."
- note added: "Інгібування заряду"
- note added: "Дроти з'єднують контакти всередині функціональної групи; кожне дерево дротів має одну глобальну мітку з канонічною назвою мережі (рамка-стрілка — мережа виходить за межі групи, пряма рамка — мережа лише цієї групи). Однакові мітки з'єднані на всіх аркушах; земля — символ GND. Рамки OPEN — незакриті ворота з design/E#.json (повний реєстр: OPEN_ITEMS.md); «TBD» у значенні — STACK номіналу не задає,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"
- note added: "Захист USB-PD"
- note added: "Контрольні точки"
- note added: "Позначення фізичних джерел живлення (ERC)"
- note added: "Ревізія COUT і місця NTC/VSET/ISET/ISET_MODE/CELLSET не підтверджені офіційною схемою. Вікно 0…45 °C та inhibit не перевірені. Ворота (стенд): До модифікацій отримати ревізійну схему або фото обох боків з continuity до IC. Стенд: NTC 0/45 °C, обрив/КЗ, зупинка charge і reverse boost, 2 h при 3 A, 20 PD cycles, зовнішній VBUS=0 V, startup 5→20 V, CV кожної комірки. При провалі цей модуль не викори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"
- note added: "Термо, transient, ESD та узгодження захистів не доведені на реальному PCB. Ворота (стенд): Силова плата reflow. Перевірити USB-PD OVLO≈22 V, ILIM≈3.5 A, hot-plug 0→20 V і reverse blocking. TVS E1_SW не вважати гарантією захисту 28 V eFuse. SYS12: C4 RF A/B і 60 min при 4.2 A, входи 14/16.4 V; батарейний шлях 4.6 A при case 50 °C. Перед виготовленням PCB потрібні layout, ERC і DRC."
- note added: "Фізичний PHB2.0 pin order Daly та ревізія J05G/J04G3 нез’ясовані. Ворота (стенд): На прийманні звірити маркування з Daly DS саме цієї ревізії. Продзвонити B0…B4 зі знятим sense-штекером; послідовні напруги 3…4.2 V, сумарно 4S. Пробудження зарядником 3/3. До цього підключення sense заборонене."
- note removed: "E1 - Акумулятор, заряд, AON і головні перетворювачі (1/2)"
- note removed: "Мережі з однаковими глобальними мітками електрично з'єднані на всіх аркушах. Фізичні/функціональні контакти: див. design/ і OPEN_ITEMS.md."
- title: E1 - Акумулятор, заряд, AON і головні перетворювачі (1/2) -> E1 - Акумулятор, заряд, AON і головні перетворювачі (1/1)
- moved on the sheet: J101, U101, U102, U103, U104
