File: sat-receiver-audit/build/kicad/E1.kicad_sch (KiCad schematic)
At the start: 68 parts, among them J101 XT30 сервісний заряд/розряд, J102 DNP — зовнішній balance 4S (G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, Q101 2N7002,215, U101 Daly DL-J05G-L4S15ATJ 4S15A, U102 INA228AIDGSR на Adafruit 5832, U103 TPS70933DBVR, U104 MCP65R41T-1202E/CHY, U106 Pololu 2813 HP, U107 Pololu D36V50F12#4095, U108 Pololu D36V50F5 #4091 — LAB5 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, U109 TPS259470ARPWR USB-C

Commit message: GENERATED: CAD, netlist, ERC, documents and re-frozen DC_CORE PCB chain from CI
Applied verbatim from the cad-regenerated artifacts of run 40087342176
(for source commit c17ae81) and run 40090126917 (for the review fixes,
source commit 4740951); KiCad 10.0.7, refreeze_pcb=true.

Co-Authored-By: Claude Opus 5.5 <noreply@anthropic.com>
Parts:
- R108: value 10.0k1% -> 4.99k0.1%25ppm; footprint (none) -> Resistor_SMD:R_0603_1608Metric
- R109: value 1.00k1% -> 562R0.1%25ppm; footprint (none) -> Resistor_SMD:R_0603_1608Metric
Other:
- moved on the sheet: C103, C104, C105, C106, C109, C110, C111, C112, C113, C114, D101, F102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
