File: sat-receiver-audit/build/kicad/E4.kicad_sch (KiCad schematic)
At the start: 0 parts

Commit message: Complete SR-RX-v2.1 schematics and verification package
Replace five empty sheets with reviewed KiCad schematics and portable resources. Correct power, control, USB and RF interfaces; document hardware acceptance gates and unimplemented firmware/PCB work. Validate 754 components, 2189 connected contacts and 466 nets with zero ERC violations and two independent graph/netlist comparisons. Include PDF, SVG, BOM, reproducible tools and offline documentation.
Parts:
- added A401: Flamingo+ FM v2 #1, symbol sr_rx_v2_completed:C_A401
- added A402: SAWbird+ NOAA 100800, symbol sr_rx_v2_completed:C_A402
- added A403: Flamingo+ FM v2 #2 optional, symbol sr_rx_v2_completed:C_A403
- added A404: LNA V2 optional, symbol sr_rx_v2_completed:C_A404
- added A405: SMA attenuator 15/20/30 dB: bench selection, symbol sr_rx_v2_completed:C_A405
- added A406: Boni-Whip supplied bias-tee, symbol sr_rx_v2_completed:C_A406
- added A407: YAT-10A+ 10 dB, symbol sr_rx_v2_completed:C_A407
- added A408: H1 SMA pad 0/2/3 dB, symbol sr_rx_v2_completed:C_A408
- added A409: BLK-89-S+, symbol sr_rx_v2_completed:C_A409
- added A410: ANNE-50+ 50 Ω load, symbol sr_rx_v2_completed:C_A410
- added A411: RTL-SDR Blog V4L LABRXA, symbol sr_rx_v2_completed:C_A411
- added A412: RTL-SDR Blog V4L LABRXB, symbol sr_rx_v2_completed:C_A412
- added A414: Airspy HF+ Discovery, symbol sr_rx_v2_completed:C_A414
- added A415: LimeSDR Micro M.2 v1.2 receive-only, symbol sr_rx_v2_completed:C_A415
- added A418: Uputronics 440 Rev 3.0 external LNA, symbol sr_rx_v2_completed:C_A418
- added A419: GOES / H1 / iO / active patch external LNA, symbol sr_rx_v2_completed:C_A419
- added A420: Othernet Bullseye LNB, symbol sr_rx_v2_completed:C_A420
- added A421: AXING CFA 11-00 DC-isolated 75 Ω load, symbol sr_rx_v2_completed:C_A421
- added A422: Nooelec LaNA WB 100845, symbol sr_rx_v2_completed:C_A422
- added A423: sysmocom cf2235-kt30 2170–2300 MHz, symbol sr_rx_v2_completed:C_A423
- added A424: TCBT-2R5G+ ch4, symbol sr_rx_v2_completed:C_A424
- added J401: P1 VHF137 SMA: no DC, symbol sr_rx_v2_completed:C_J401
- added J402: P2 UHF SMA: 4.5 V, symbol sr_rx_v2_completed:C_J402
- added J403: P3 L-band SMA: 4.5 V, symbol sr_rx_v2_completed:C_J403
- added J404: P4 LNB F: 13.2 V, symbol sr_rx_v2_completed:C_J404
- added J405: P5 HF BNC: 13.8 V, symbol sr_rx_v2_completed:C_J405
- added J406: P6 VHF/AIS SMA: no DC, symbol sr_rx_v2_completed:C_J406
- added J407: P7 GNSS SMA, symbol sr_rx_v2_completed:C_J407
- added J408: P8 WIDE optional SMA, symbol sr_rx_v2_completed:C_J408
- added J409: BENCH internal SMA, symbol sr_rx_v2_completed:C_J409
- added J410: RTL-A RF internal SMA, symbol sr_rx_v2_completed:C_J410
- added J411: RTL-B RF internal SMA, symbol sr_rx_v2_completed:C_J411
- added J412: RX1 edge SMA, symbol sr_rx_v2_completed:C_J412
- added J413: RX1 panel SMA: captive loop, symbol sr_rx_v2_completed:C_J413
- added J414: RX2 panel SMA, symbol sr_rx_v2_completed:C_J414
- added J415: REF IN panel SMA, symbol sr_rx_v2_completed:C_J415
- added J416: UHF antenna feed / A418 input interface, symbol sr_rx_v2_completed:C_J416
- added J417: L-band antenna feed / A419 input interface, symbol sr_rx_v2_completed:C_J417
- added W401: Goobay 58814 75 Ω F-F 1 m, symbol sr_rx_v2_completed:C_W401
- added W402: 75 Ω shielded internal IF coax, symbol sr_rx_v2_completed:C_W402
- added W403: RX1 panel → Lime X2 MHF4 coax, symbol sr_rx_v2_completed:C_W403
- added W404: RX2 → Lime X4 MHF4 coax, symbol sr_rx_v2_completed:C_W404
- added W405: REF IN → J4 MHF4 coax, symbol sr_rx_v2_completed:C_W405
- added W406: CAB.01075 X1 → ANNE-50+ captive coax, symbol sr_rx_v2_completed:C_W406
- added W407: P7 SMA → LC76G IPEX coax, symbol sr_rx_v2_completed:C_W407
- added W408: RG316 common-mode choke FT240-77 +2631102002, symbol sr_rx_v2_completed:C_W408
- added W409: Captive RX1 edge → profile pad coax, symbol sr_rx_v2_completed:C_W409
- added W422: RG316 SMA-M/M 0.10 m helix → LaNA, symbol sr_rx_v2_completed:C_W422
- added W423: RG316 SMA-M/M 0.10 m LaNA → DC block, symbol sr_rx_v2_completed:C_W423
- added W424: RG316 SMA-M/M 1.00 m pod → RX2, symbol sr_rx_v2_completed:C_W424
Connections:
- new net BIAS_CH4: A424.1 (DC)
- new net BONI13V8: A406.DC
- new net E4_BENCH: J409.CENTER
- new net E4_CH4_RF_ONLY: A424.4 (RF)
- new net E4_HFP_ANT: A414.ANT
- new net E4_HF_BT: A406.RF
- new net E4_HF_CM: A406.ANT, W408.OUT_CENTER
- new net E4_LIME_REF: A415.J4_REF_IN, W405.END_B
- new net E4_LIME_RX2: A409.IN, J414.CENTER, W424.PANEL
- new net E4_LIME_RXA: A415.X2_RX_A, W403.END_B
- new net E4_LIME_RXB: A415.X4_RX_B, W404.END_B
- new net E4_LIME_TX: A415.X1_TX, W406.END_A
- new net E4_LNB_IF: A420.IF, W401.END_A
- new net E4_LNB_REF25: A420.REF25, A421.END_A
- new net E4_P1: A401.IN, J401.CENTER
- new net E4_P2: A418.OUT, J402.CENTER
- new net E4_P2_ANT: A418.IN, J416.CENTER
- new net E4_P3: A419.OUT, J403.CENTER
- new net E4_P3_ANT: A419.IN, J417.CENTER
- new net E4_P4: J404.CENTER, W401.END_B, W402.END_A
- new net E4_P5: J405.CENTER, W408.IN_CENTER
- new net E4_P6: J406.CENTER
- new net E4_P8: A403.IN, J408.CENTER
- new net E4_REF_IN: J415.CENTER, W405.END_A
- new net E4_RFC_A: A411.ANT, J410.CENTER
- new net E4_RFC_B: A412.ANT, J411.CENTER
- new net E4_RF_CH1: A402.OUT
- new net E4_RF_CH4: A404.OUT, A424.3 (RF_DC)
- new net E4_RF_CH5: W402.END_B
- new net E4_RF_CH5_ATT: A405.OUT
- new net E4_RF_CH5_DC: A405.IN
- new net E4_RF_P1_FM: A401.OUT, A402.IN
- new net E4_RF_P8_FM: A403.OUT, A404.IN
- new net E4_RX1_EDGE: J412.CENTER, W409.EDGE
- new net E4_RX1_PAD: A408.IN, W409.PAD
- new net E4_RX1_PANEL: A408.OUT, J413.CENTER, W403.END_A
- new net E4_RX2_ANT: W422.ANT
- new net E4_RX2_BLK: A409.OUT, W404.END_A
- new net E4_SB_FILTER_IN: A423.SMA_F_A
- new net E4_SB_FILTER_OUT: A423.SMA_F_B, W424.FILTER
- new net E4_SB_LNA_IN: A422.SMA_IN, W422.LNA
- new net E4_SB_LNA_OUT: A422.SMA_OUT, W423.LNA
- new net E4_SB_POD5: A422.USB_C_VBUS
- new net E4_SB_PREBLOCK: W423.BLOCK
- new net E4_TX_LOAD: A410.END_A, W406.END_B
- new net E4_YAT_IN: A407.2 (RF_IN)
- new net E4_YAT_OUT: A407.5 (RF_OUT)
- new net E5_PCIE_CLKREQ_N: A415.X9_CLKREQ_N
- new net E5_PCIE_PERST_N: A415.X9_PERST_N
- new net E5_PCIE_REFCLK_N: A415.X9_REFCLK_N
- new net E5_PCIE_REFCLK_P: A415.X9_REFCLK_P
- new net E5_PCIE_RX0_N: A415.X9_TX_N
- new net E5_PCIE_RX0_P: A415.X9_TX_P
- new net E5_PCIE_TX0_N: A415.X9_RX_N
- new net E5_PCIE_TX0_P: A415.X9_RX_P
- new net E5_PCIE_WAKE_N: A415.X9_WAKE_N
- new net GND: A401.SHIELDS, A402.SHIELDS, A403.SHIELDS, A404.SHIELDS, A405.SHIELDS, A406.SHIELDS, A407.1 (GND), A407.3 (GND), A407.4 (GND), A407.6 (GND), A407.EP (EP_GND), A408.SHIELDS, A409.SHIELDS, A410.END_B, A411.USB_GND, A411.USB_SHIELD, A412.USB_GND, A412.USB_SHIELD, A414.USB_GND, A414.USB_SHIELD, A415.X9_GND, A418.SHIELDS, A419.SHIELDS, A420.SHIELDS, A421.SHIELDS, A422.SHIELDS, A422.USB_C_GND, A423.SHIELDS, J401.SHIELD, J402.SHIELD, J403.SHIELD, J404.SHIELD, J405.SHIELD, J406.SHIELD, J407.SHIELD, J408.SHIELD, J409.SHIELD, J410.SHIELD, J411.SHIELD, J412.SHIELD, J413.SHIELD, J414.SHIELD, J415.SHIELD, J416.SHIELD, J417.SHIELD, W401.SHIELDS, W402.SHIELDS, W403.SHIELDS, W404.SHIELDS, W405.SHIELDS, W406.SHIELDS, W407.SHIELDS, W408.IN_SHIELD, W408.OUT_SHIELD, W409.SHIELD, W422.SHIELDS, W423.SHIELDS, W424.SHIELDS
- new net GNSS_ANT: J407.CENTER, W407.END_A, W407.END_B
- new net HFP_DM: A414.USB_DM
- new net HFP_DP: A414.USB_DP
- new net LIME3V3: A415.X9_3V3
- new net RTLA_DM: A411.USB_DM
- new net RTLA_DP: A411.USB_DP
- new net RTLB_DM: A412.USB_DM
- new net RTLB_DP: A412.USB_DP
- new net VBUS_HFP: A414.USB_VBUS
- new net VBUS_RTLA: A411.USB_VBUS
- new net VBUS_RTLB: A412.USB_VBUS
- no-connect marks 0 -> 1
Other:
- note added: "E4 - РЧ-тракт: DC-розвʼязка, перемикачі, реле та приймачі (1/4)"
- note added: "RF and receiver interfaces"
- note added: "S-band external inline pod"
- note added: "Мережі з однаковими глобальними мітками електрично з'єднані на всіх аркушах. Фізичні/функціональні контакти: див. design/ і OPEN_ITEMS.md."
- company: (none) -> SR-RX-v2
- title: (none) -> E4 - РЧ-тракт і DC-захист (1/4)
