File: sat-receiver-audit/build/kicad/E4.kicad_sch (KiCad schematic)
At the start: 50 parts, among them J401 P1 VHF137 SMA: no DC, J402 P2 UHF SMA: 4.5 V, J403 P3 L-band SMA: 4.5 V, J404 P4 LNB F: 13.2 V, J405 P5 HF BNC: 13.8 V, J406 P6 VHF/AIS SMA: no DC, J407 P7 GNSS SMA, J408 P8 WIDE optional SMA, J409 BENCH internal SMA, J410 RTL-A RF internal SMA, J411 RTL-B RF internal SMA, J412 RX1 edge SMA, J413 RX1 panel SMA: captive loop, J414 RX2 panel SMA, J415 REF IN panel SMA, J416 UHF antenna feed / A418 input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, J417 L-band antenna feed / A419 in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

Commit message: SR-RX-v2.1: review fixes on the Codex branch, readable schematic, one-file bundle
Independent review of the Codex branch (schematic vs STACK.md, hard rules,
security, tests) found no blockers; this commit applies its findings:

- rules in code: Cospas-Sarsat 406.0-406.1 MHz added to the no-data mask;
  Q6A Wi-Fi/BT off in the field/QUIET root (modprobe blacklist, udev
  authorized=0 on FE1.1s port 4, rfkill) with self-checks; device denylist
  completed per STACK (gr-gsm, gr-iridium, kalibrate, pager/trunking decoders,
  TX-capable tools); W1-2 WIFI_PWR_EN as blocking open item E5-10
- STACK.md is the source of truth again; v2.1 changes recorded in it; the
  "historical" marker kept only on ISDT/raw-balance rows; gender-neutral wording
- schematic data: open values shown as TBD with start values and notes, U503
  TPS2553DBVR-1, Lime X2/X4 RX mapping TBD, 37 open items drawn on the sheets
- schematic readability: wired groups, junctions, GND symbols, standard
  transistor/diode symbols; netlist unchanged (603 nets identical)
- tooling: reproducible run_checks (no timestamps or machine paths), pinned
  dependencies, bundle excludes cache folders, clean-checkout bundle check
- regenerated: KiCad export (14 pages), netlist/ERC, module lab, PCB inputs,
  readiness contract, acceptance hashes, SR-RX-v2-ves-proekt.html

Checks: ERC 0 errors/0 warnings, netlist comparison PASS, 432 tests (431
passed, 1 skipped), deployment tests OK, bundle check PASS on a clean checkout.

History note: earlier versions of the generated SR-RX-v2-ves-proekt.html and
handoff/handoff-bundle.zip were removed from history; only the final versions
are kept. The Codex merge commit is now attributed to Codex.

Co-Authored-By: Claude Opus 5.5 <noreply@anthropic.com>
Claude-Session: https://claude.ai/code/session_01W9CKpimWpgkUmrDQQMiKtF
Parts:
- removed A410: ANNE-50+ 50 Ω load, symbol sr_rx_v2_completed:C_A410
- removed A418: Uputronics 440 Rev 3.0 external LNA, symbol sr_rx_v2_completed:C_A418
- removed A419: GOES / H1 / iO / active patch external LNA, symbol sr_rx_v2_completed:C_A419
- removed A422: Nooelec LaNA WB 100845, symbol sr_rx_v2_completed:C_A422
- removed A423: sysmocom cf2235-kt30 2170–2300 MHz, symbol sr_rx_v2_completed:C_A423
- removed J402: P2 UHF SMA: 4.5 V, symbol sr_rx_v2_completed:C_J402
- removed J403: P3 L-band SMA: 4.5 V, symbol sr_rx_v2_completed:C_J403
- removed J416: UHF antenna feed / A418 input interface, symbol sr_rx_v2_completed:C_J416
- removed J417: L-band antenna feed / A419 input interface, symbol sr_rx_v2_completed:C_J417
- removed W406: CAB.01075 X1 → ANNE-50+ captive coax, symbol sr_rx_v2_completed:C_W406
- removed W422: RG316 SMA-M/M 0.10 m helix → LaNA, symbol sr_rx_v2_completed:C_W422
- removed W423: RG316 SMA-M/M 0.10 m LaNA → DC block, symbol sr_rx_v2_completed:C_W423
- removed W424: RG316 SMA-M/M 1.00 m pod → RX2, symbol sr_rx_v2_completed:C_W424
- added C447: 100 pF C0G 50 V, symbol sr_rx_v2_completed:C_C447
- added C448: 10 nF C0G 50 V, symbol sr_rx_v2_completed:C_C448
- added C449: 100 pF C0G 50 V, symbol sr_rx_v2_completed:C_C449
- added C450: 10 nF C0G 50 V, symbol sr_rx_v2_completed:C_C450
- added C451: 100 pF C0G 50 V, symbol sr_rx_v2_completed:C_C451
- added C452: 10 nF C0G 50 V, symbol sr_rx_v2_completed:C_C452
- J413: value RX1 panel SMA: captive loop -> RX1 panel SMA: captive coax assembly
Connections:
- net GND: now also C447.2, C448.2, C449.2, C450.2, C451.2, C452.2
- net E4_LIME_RXA renamed E4_LIME_X2_RX
- net E4_LIME_X2_RX: now also A415.X2_RX; no longer A415.X2_RX_A
- net E4_LIME_RXB renamed E4_LIME_X4_RX
- net E4_LIME_X4_RX: now also A415.X4_RX; no longer A415.X4_RX_B
- new net BIAS_CH1: C447.1, C448.1
- new net BIAS_CH2: C449.1, C450.1
- new net BIAS_CH3: C451.1, C452.1
Other:
- note added: "BENCH RF sled is not delivered as a separate HMC7992 + PE4312 PCB here. Ворота (стенд): Deliver its PCB/netlist, controls and 31.5 dB startup test if installed. Until then use the internal BENCH SMA with a qualified external conducted source."
- note added: "Boni supplied bias-tee port labels, DC socket polarity and receiver DC block require actual hardware. Ворота (стенд): Measure continuity/polarity, antenna DC and RADIO port <0.1 V before connecting HF+."
- note added: "E4 - РЧ-тракт: DC-розв'язка, перемикачі, приймачі (1/4)"
- note added: "E4-03 — OPEN, блокує випуск — STACK §5.3; §8.1 HF-9, HF-11"
- note added: "E4-05 — OPEN, блокує випуск — STACK §2.11.1; §8.1 L-12"
- note added: "E4-08 — OPEN, блокує випуск — STACK §5.3 (RX1, YAT-10A+, H1)"
- note added: "E4-09 — умова опції, не блокує випуск — STACK §3.1; §5.3 (BENCH); §8.1 RF-11"
- note added: "Lime X2/X4 are the v1.2 RX ports, but which of them is RX-A and which RX-B is TBD (STACK §2.11.1, §8.1 L-12: check against the board marking). Pins are named X2_RX/X4_RX and nets E4_LIME_X2_RX/E4_LIME_X4_RX, so the drawing fixes no channel; supplied-board cable labels need confirmation. Ворота (стенд): Check the exact revision schematic and conduct a one-port-at-a-time RX test. Generic setup X3 w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"
- note added: "RF bias injector local decoupling"
- note added: "RX1 captive edge/pad/panel assembly and H1 attenuation have not been measured. Ворота (стенд): Confirm edge → pad → panel → X2 without bypass. YAT 10±0.5 dB and RL ≥20 dB; H1 total ≥12.0 dB at 1420 MHz, using 3 dB pad if the 2 dB pad fails."
- note added: "Дроти з'єднують контакти всередині функціональної групи; кожне дерево дротів має одну глобальну мітку з канонічною назвою мережі (рамка-стрілка — мережа виходить за межі групи, пряма рамка — мережа лише цієї групи). Однакові мітки з'єднані на всіх аркушах; земля — символ GND. Рамки OPEN — незакриті ворота з design/E#.json (повний реєстр: OPEN_ITEMS.md); «TBD» у значенні — STACK номіналу не задає,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"
- note removed: "E4 - РЧ-тракт: DC-розвʼязка, перемикачі, реле та приймачі (1/4)"
- note removed: "S-band external inline pod"
- note removed: "Мережі з однаковими глобальними мітками електрично з'єднані на всіх аркушах. Фізичні/функціональні контакти: див. design/ і OPEN_ITEMS.md."
- title: E4 - РЧ-тракт і DC-захист (1/4) -> E4 - РЧ-тракт: DC-розв'язка, перемикачі, приймачі (1/4)
- moved on the sheet: A407, A424

Commit message: Stage 2 integration: CAD and DC_CORE re-freeze from CI run 40094234222; bound-count test and PCB hash lists follow
Co-Authored-By: Claude Opus 5.5 <noreply@anthropic.com>
Parts:
- removed A409: BLK-89-S+, symbol sr_rx_v2_completed:C_A409
- removed J414: RX2 panel SMA, symbol sr_rx_v2_completed:C_J414
- removed J415: REF IN panel SMA, symbol sr_rx_v2_completed:C_J415
- removed W404: RX2 → Lime X4 MHF4 coax, symbol sr_rx_v2_completed:C_W404
- removed W405: REF IN → J4 MHF4 coax, symbol sr_rx_v2_completed:C_W405
Connections:
- net BIAS_CH2 renamed BIAS_CH2_PORT
- net BIAS_CH3 renamed BIAS_CH3_PORT
- net BONI13V8 renamed BONI13V8_PORT
Other:
- note added: "Boni supplied bias-tee port labels, DC socket polarity and receiver DC block require actual hardware. Ворота (стенд): Measure continuity/polarity, antenna DC and RADIO port <0.1 V before connecting HF+. v2.1: A406 DC is BONI13V8_PORT behind the E2 blocking element Q2903 — confirm on the supplied Einspeiseweiche a DC current rating ≥0.16 A (ILIM max 0.153 A, 0.154 A with TCR, RILM 7.15k) and DC-bl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"
- note removed: "Boni supplied bias-tee port labels, DC socket polarity and receiver DC block require actual hardware. Ворота (стенд): Measure continuity/polarity, antenna DC and RADIO port <0.1 V before connecting HF+."
- moved on the sheet: A403, A404, A406, A408, A411, A412, A415, A424, J405, J406, J407, J408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
