File: sat-receiver-audit/build/kicad/E5.kicad_sch (KiCad schematic)
At the start: 0 parts

Commit message: Complete SR-RX-v2.1 schematics and verification package
Replace five empty sheets with reviewed KiCad schematics and portable resources. Correct power, control, USB and RF interfaces; document hardware acceptance gates and unimplemented firmware/PCB work. Validate 754 components, 2189 connected contacts and 466 nets with zero ERC violations and two independent graph/netlist comparisons. Include PDF, SVG, BOM, reproducible tools and offline documentation.
Parts:
- added C501: 100nF X7R 10V, symbol sr_rx_v2_completed:C_C501
- added C502: 4.7uF X7R 10V, symbol sr_rx_v2_completed:C_C502
- added C503: 47uF 10V, symbol sr_rx_v2_completed:C_C503
- added C504: 100nF X7R 10V, symbol sr_rx_v2_completed:C_C504
- added C505: 4.7uF X7R 10V, symbol sr_rx_v2_completed:C_C505
- added C506: 150uF 10V low-ESR, symbol sr_rx_v2_completed:C_C506
- added C507: 100nF X7R 10V, symbol sr_rx_v2_completed:C_C507
- added C508: 100nF X7R 10V, symbol sr_rx_v2_completed:C_C508
- added C509: 4.7uF X7R 10V, symbol sr_rx_v2_completed:C_C509
- added C510: 1uF X7R 10V, symbol sr_rx_v2_completed:C_C510
- added C511: EEU-FR1C101 100uF 16V, symbol sr_rx_v2_completed:C_C511
- added C512: 220uF 16V low-ESR, symbol sr_rx_v2_completed:C_C512
- added C513: 100nF X7R 10V, symbol sr_rx_v2_completed:C_C513
- added C514: 100nF X7R 10V, symbol sr_rx_v2_completed:C_C514
- added C515: 4.7uF X7R 10V, symbol sr_rx_v2_completed:C_C515
- added C516: 150uF 10V low-ESR, symbol sr_rx_v2_completed:C_C516
- added J501: LAB USB-A panel receptacle, symbol sr_rx_v2_completed:C_J501
- added J503: J21 service harness 3pin locking, symbol sr_rx_v2_completed:C_J503
- added J511: Q6A J5 stacked USB3 lower / USB2 upper, symbol sr_rx_v2_completed:C_J511
- added J512: Q6A J2 stacked USB2 bank1 P3 / bank2 P2, symbol sr_rx_v2_completed:C_J512
- added J520: Q6A HDMI Type-A existing port, symbol sr_rx_v2_completed:C_J520
- added J521: Q6A J21 existing header pads, symbol sr_rx_v2_completed:C_J521
- added J541: RTL-B split-VBUS USB cable endpoint, symbol sr_rx_v2_completed:C_J541
- added J543: RTL-A USB cable endpoint, symbol sr_rx_v2_completed:C_J543
- added J544: HF+ microUSB-B cable endpoint, symbol sr_rx_v2_completed:C_J544
- added L501: SRR1260-101M 100uH, symbol sr_rx_v2_completed:C_L501
- added R501: 43.2k 1%, Resistor_SMD:R_0603_1608Metric, symbol sr_rx_v2_completed:C_R501
- added R502: 100k, Resistor_SMD:R_0603_1608Metric, symbol sr_rx_v2_completed:C_R502
- added R503: 10k, Resistor_SMD:R_0603_1608Metric, symbol sr_rx_v2_completed:C_R503
- added R504: 10k, Resistor_SMD:R_0603_1608Metric, symbol sr_rx_v2_completed:C_R504
- added R505: 34.8k 1%, Resistor_SMD:R_0603_1608Metric, symbol sr_rx_v2_completed:C_R505
- added R506: 100k, Resistor_SMD:R_0603_1608Metric, symbol sr_rx_v2_completed:C_R506
- added R507: 10k, Resistor_SMD:R_0603_1608Metric, symbol sr_rx_v2_completed:C_R507
- added R508: 10k, Resistor_SMD:R_0603_1608Metric, symbol sr_rx_v2_completed:C_R508
- added R509: 28.7k 1%, Resistor_SMD:R_0603_1608Metric, symbol sr_rx_v2_completed:C_R509
- added R510: 100k, Resistor_SMD:R_0603_1608Metric, symbol sr_rx_v2_completed:C_R510
- added R511: 10k, Resistor_SMD:R_0603_1608Metric, symbol sr_rx_v2_completed:C_R511
- added R512: 1Ohm 0.5W, Resistor_SMD:R_0603_1608Metric, symbol sr_rx_v2_completed:C_R512
- added R513: 10k, Resistor_SMD:R_0603_1608Metric, symbol sr_rx_v2_completed:C_R513
- added R514: 15.8k 1%, Resistor_SMD:R_0603_1608Metric, symbol sr_rx_v2_completed:C_R514
- added R515: 100k, Resistor_SMD:R_0603_1608Metric, symbol sr_rx_v2_completed:C_R515
- added R516: 10k, Resistor_SMD:R_0603_1608Metric, symbol sr_rx_v2_completed:C_R516
- added R517: 10k, Resistor_SMD:R_0603_1608Metric, symbol sr_rx_v2_completed:C_R517
- added TP501: T7 FAULT_N test point, symbol sr_rx_v2_completed:C_TP501
- added U500: Q6A onboard peripheral rail sources, symbol sr_rx_v2_completed:C_U500
- added U501: TPS2553DBVR-1, Package_TO_SOT_SMD:SOT-23-6, symbol sr_rx_v2_completed:C_U501
- added U502: TPS2553DBVR-1, Package_TO_SOT_SMD:SOT-23-6, symbol sr_rx_v2_completed:C_U502
- added U503: TPS2553DBVR, Package_TO_SOT_SMD:SOT-23-6, symbol sr_rx_v2_completed:C_U503
- added U505: TPS2553DRVR, Package_SON:WSON-6-1EP_2x2mm_P0.65mm_EP1x1.6mm, symbol sr_rx_v2_completed:C_U505
- added U510: Adafruit5997 CH334F revC board, symbol sr_rx_v2_completed:C_U510
- added U540: Samsung T7 + intact A-to-C USB3 cable, symbol sr_rx_v2_completed:C_U540
Connections:
- new net 3V3_Q6A: R503.2, R507.2, R511.2, R516.2
- new net E5_FAULT_T7: R516.1, TP501.1 (FAULT_N), U505.3 (FAULT_N)
- new net E5_HDMI_5V_Q6A: J520.18 (+5V)
- new net E5_HDMI_CEC: J520.13 (CEC)
- new net E5_HDMI_CLK_N: J520.12 (TMDSCLK−)
- new net E5_HDMI_CLK_P: J520.10 (TMDSCLK+)
- new net E5_HDMI_D0_N: J520.9 (TMDS0−)
- new net E5_HDMI_D0_P: J520.7 (TMDS0+)
- new net E5_HDMI_D1_N: J520.6 (TMDS1−)
- new net E5_HDMI_D1_P: J520.4 (TMDS1+)
- new net E5_HDMI_D2_N: J520.3 (TMDS2−)
- new net E5_HDMI_D2_P: J520.1 (TMDS2+)
- new net E5_HDMI_HPD: J520.19 (HPD)
- new net E5_HDMI_SCL: J520.15 (DDC SCL)
- new net E5_HDMI_SDA: J520.16 (DDC SDA)
- new net E5_HFP_DAMP: C512.1 (+), R512.2
- new net E5_HUB_DM: J512.2 (P3 D− to hub), U510.JP5_3 (UP D−)
- new net E5_HUB_DP: J512.3 (P3 D+ to hub), U510.JP5_2 (UP D+)
- new net E5_LABPORT_DM: J501.2 (D−), U510.JP3_3 (H3/D−)
- new net E5_LABPORT_DP: J501.3 (D+), U510.JP3_2 (H3/D+)
- new net E5_T7_DM: J511.2 (J5 lower D−), U540.DM (D−)
- new net E5_T7_DP: J511.3 (J5 lower D+), U540.DP (D+)
- new net E5_T7_HOST_RX_N: J511.5 (J5 lower SSRX−), U540.TXN (device SSTX−)
- new net E5_T7_HOST_RX_P: J511.6 (J5 lower SSRX+), U540.TXP (device SSTX+)
- new net E5_T7_HOST_TX_N: J511.8 (J5 lower SSTX−), U540.RXN (device SSRX−)
- new net E5_T7_HOST_TX_P: J511.9 (J5 lower SSTX+), U540.RXP (device SSRX+)
- new net E5_TOUCH_DM: J512.6 (P2 D− to touch)
- new net E5_TOUCH_DP: J512.7 (P2 D+ to touch)
- new net E5_U501_ILIM: R501.1, U501.5 (ILIM)
- new net E5_U502_ILIM: R505.1, U502.5 (ILIM)
- new net E5_U503_ILIM: R509.1, U503.5 (ILIM)
- new net E5_U505_ILIM: R514.1, U505.2 (ILIM)
- new net E5_VBUS_HFP_SW: C510.1 (+), L501.1 (IN), U503.6 (OUT)
- new net E5_VBUS_J5: C514.1 (+), C515.1 (+), J511.1 (J5 lower VBUS), U505.6 (IN)
- new net E5_VBUS_T7: C516.1 (+), R517.1, U505.1 (OUT), U540.VBUS (5V)
- new net EN_HFP: R510.1, U503.3 (EN)
- new net EN_LABPORT: R506.1, U502.3 (EN)
- new net EN_RTLA: R502.1, U501.3 (EN)
- new net EN_T7: R515.1, U505.4 (EN)
- new net FAULT_HFP: R511.1, U503.4 (FAULT_N)
- new net FAULT_LABPORT: R507.1, U502.4 (FAULT_N)
- new net FAULT_RTLA: R503.1, U501.4 (FAULT_N)
- new net GND: C501.2 (−), C502.2 (−), C503.2 (−), C504.2 (−), C505.2 (−), C506.2 (−), C507.2 (−), C508.2 (−), C509.2 (−), C510.2 (−), C511.2 (−), C512.2 (−), C513.2 (−), C514.2 (−), C515.2 (−), C516.2 (−), J501.4 (GND), J501.S (cable shield), J503.2 (GND), J511.13 (J5 upper GND), J511.19 (onboard TAB/GND), J511.20 (onboard TAB/GND), J511.21 (onboard TAB/GND), J511.22 (onboard TAB/GND), J511.4 (J5 lower GND), J511.7 (SS GND), J512.10 (onboard shell/GND), J512.11 (onboard shell/GND), J512.12 (onboard shell/GND), J512.4 (P3 GND), J512.8 (P2 GND), J512.9 (onboard shell/GND), J520.11 (TMDSCLK shield), J520.17 (DDC ground), J520.2 (TMDS2 shield), J520.5 (TMDS1 shield), J520.8 (TMDS0 shield), J521.2 (GND), J541.4 (GND), J543.4 (GND), J544.5 (GND), J544.S (shield), R501.2, R502.2, R504.2, R505.2, R506.2, R508.2, R509.2, R510.2, R513.2, R514.2, R515.2, R517.2, U500.GND, U501.2 (GND), U502.2 (GND), U503.2 (GND), U505.5 (GND), U505.7 (exposed pad), U510.JP1_4 (H2/GND), U510.JP2_4 (H1/GND), U510.JP3_4 (H3/GND), U510.JP4_4 (H4/GND), U510.JP5_4 (UP GND), U540.GND (signal ground), U540.SHIELD (cable shield)
- new net HFP_DM: J544.2 (D−), U510.JP4_3 (H4/D−)
- new net HFP_DP: J544.3 (D+), U510.JP4_2 (H4/D+)
- new net J21: J503.1 (12V), J521.1 (ADP12V_IN), U500.VIN (from protected J21)
- new net LAB5: C501.1 (+), C502.1 (+), C504.1 (+), C505.1 (+), C508.1 (+), C509.1 (+), U501.1 (IN), U502.1 (IN), U503.1 (IN), U510.JP5_1 (UP 5V input)
- new net PWR_ON_KEY: J503.3 (KEY), J521.3 (PWR_ON_KEY)
- new net RTLA_DM: J543.2 (D−), U510.JP1_3 (H2/D−)
- new net RTLA_DP: J543.3 (D+), U510.JP1_2 (H2/D+)
- new net RTLB_DM: J511.11 (J5 upper D−), J541.2 (D− from J5_11)
- new net RTLB_DP: J511.12 (J5 upper D+), J541.3 (D+ from J5_12)
- new net VBUS_HFP: C511.1 (+), C513.1 (+), J544.1 (VBUS filtered), L501.2 (OUT), R512.1, R513.1
- new net VBUS_LABPORT: C506.1 (+), C507.1 (+), J501.1 (VBUS), R508.1, U502.6 (OUT)
- new net VBUS_RTLA: C503.1 (+), J543.1 (VBUS from U501), R504.1, U501.6 (OUT)
- new net VBUS_RTLB: J541.1 (VBUS from E2)
- new net VCC_3V3_MKEY: U500.MKEY_3V3 (VCC_3V3_MKEY source)
- new net VCC_5V_PERI: U500.5V (VCC_5V_PERI source)
- no-connect marks 0 -> 11
Other:
- note added: "CH334F і USB2 кабелі"
- note added: "E5 - USB, VBUS, PCIe та корпусні інтерфейси (1/2)"
- note added: "Q6A порти і живлення"
- note added: "T7 USB3 VBUS"
- note added: "VBUS HF+ з демпфованим LC"
- note added: "VBUS RTL-A і LAB PORT"
- note added: "Дисплей HDMI, DC і USB touch"
- note added: "Мережі з однаковими глобальними мітками електрично з'єднані на всіх аркушах. Фізичні/функціональні контакти: див. design/ і OPEN_ITEMS.md."
- company: (none) -> SR-RX-v2
- title: (none) -> E5 - USB, VBUS, PCIe та корпусні інтерфейси (1/2)
