File: sat-receiver-audit/build/kicad/E5.kicad_sch (KiCad schematic)
At the start: 0 parts

Commit message: KiCad sheets E1/E2/E5 partial (work before agent limit)
Co-Authored-By: Claude Opus 5.5 <noreply@anthropic.com>
Claude-Session: https://claude.ai/code/session_01W9CKpimWpgkUmrDQQMiKtF
Parts:
- added C501: EEU-FR1C101, symbol Device:C_Polarized
- added C502: 220u TBD, symbol Device:C_Polarized
- added D501: Schottky TBD, symbol Device:D_Schottky
- added FB501, FB502: 2631480002 (на пігтейлі HF+), symbol Device:FerriteBead
- added FB503: 74271112 (на Lindy RTL-B), symbol Device:FerriteBead
- added FB504: 74271140 (на дроті сенсора), symbol Device:FerriteBead
- added FB505: ферит TBD (кабель T7), symbol Device:FerriteBead
- added FB506, FB507: 0431164281 (на кабелі HDMI), symbol Device:FerriteBead
- added J501: Radxa Q6A J2 (USB 2.0 x2), symbol Connector:USB_A_Stacked
- added J502: Radxa Q6A J5 (USB 3.1 низ / USB 2.0 верх), symbol Connector:USB3_A_Stacked
- added J503: Radxa Q6A M.2 M-key 2230 (pcie1), symbol Connector:Bus_M.2_Socket_M
- added J504: Radxa Q6A HDMI, symbol Connector:HDMI_A
- added J505: USB-A F пігтейла H2 (RTL-A), symbol Connector:USB_A
- added J506: Lindy 36700 A-F (RTL-B), symbol Connector:USB_A
- added J507: LAB USB-A (панель, низ), symbol Connector:USB_A
- added J508: Samsung T7 MU-PC1T0T/WW (символічно), symbol Connector_Generic:Conn_01x08
- added J509: HDMI IN плати Wisecoco, symbol Connector:HDMI_A
- added J510: Olimex GX16-4 (IMU, задня стінка), symbol Connector_Generic_Shielded:Conn_01x04_Shielded
- added J511: LAB BUS 6-pin з фіксацією (низ), symbol Connector_Generic:Conn_01x06
- added J512: вхід силової плати, джгут 5 жил, symbol Connector_Generic:Conn_01x05
- added J513: консоль UART5 (лючок), symbol Connector_Generic:Conn_01x03
- added L501: SRR1260-101M, symbol Device:L
- added R502, R503, R505: RILIM TBD, symbol Device:R
- added R504: 34.8k, symbol Device:R
- added R506: 1R TBD, symbol Device:R
- added SW501: EDL (лючок), symbol Switch:SW_Push
- added TP501: пад SW1 Q6A (EDL) т.1, symbol Connector:TestPoint
- added TP502: пад SW1 Q6A (EDL) т.2, symbol Connector:TestPoint
- added U501: Adafruit 5997 (CH334F #1), symbol sr_rx_v2_sig:Adafruit_5997_CH334F_Hub
- added U502, U503, U504, U505: TPS2553DBVR-1, Package_TO_SOT_SMD:SOT-23-6, symbol sr_rx_v2_pwr:TPS2553DBVR-1
- added U506: ключ VBUS T7 TBD, symbol Simulation_SPICE:SWITCH
- added U507: Wisecoco 7" HDMI (плата дисплея), symbol sr_rx_v2_sig:Wisecoco_7in_HDMI_Display
- added U508: TPD4E1U06DBVR, Package_TO_SOT_SMD:SOT-23-6, symbol sr_rx_v2_sig:TPD4E1U06DBV
Connections:
- new net: R502.1, U502.5 (ILIM)
- new net: J502.1 (VBUS1), U506.1 (N+)
- new net: D501.2 (A), J504.18 (+5V)
- new net: D501.1 (K), J509.18 (+5V)
- new net: R504.1, U504.5 (ILIM)
- new net: J508.1 (Pin_1), U506.2 (N-)
- new net: R505.1, U505.5 (ILIM)
- new net: L501.1, U505.6 (OUT)
- new net: SW501.1, TP501.1
- new net: SW501.2, TP502.1
- new net: R503.1, U503.5 (ILIM)
- new net: C502.1, R506.2
- new net 3V3_Q6A: J512.1 (Pin_1)
- new net AUX12: J511.3 (Pin_3)
- new net DISP12: U507.DC+ (DC_IN)
- new net EN_HFP: U505.3 (EN)
- new net EN_LABPORT: U504.3 (EN)
- new net EN_RTLA: U502.3 (EN)
- new net EN_RTLB: U503.3 (EN)
- new net EN_T7: U506.3 (C+)
- new net FAULT_HFP: U505.4 (~{FAULT})
- new net FAULT_LABPORT: U504.4 (~{FAULT})
- new net FAULT_RTLA: U502.4 (~{FAULT})
- new net FAULT_RTLB: U503.4 (~{FAULT})
- new net GND: C501.2, C502.2, J501.4 (GND1), J501.8 (GND2), J501.SH (Shield), J502.13 (GND2), J502.4 (GND1), J502.7 (DRAIN1), J502.SH (SHIELD), J502.SH (SHIELD), J503.1 (GND), J503.15 (GND), J503.21 (GND), J503.27 (GND), J503.3 (GND), J503.33 (GND), J503.39 (GND), J503.45 (GND), J503.51 (GND), J503.57 (GND), J503.71 (GND), J503.73 (GND), J503.75 (GND), J503.9 (GND), J504.11 (CKS), J504.17 (GND), J504.2 (D2S), J504.5 (D1S), J504.8 (D0S), J505.4 (GND), J506.4 (GND), J506.SH (Shield), J507.4 (GND), J508.8 (Pin_8), J509.11 (CKS), J509.17 (GND), J509.2 (D2S), J509.5 (D1S), J509.8 (D0S), J510.4 (Pin_4), J511.4 (Pin_4), J512.2 (Pin_2), J513.3 (Pin_3), R502.2, R503.2, R504.2, R505.2, U501.JP1-4 (H2_GND), U501.JP3-4 (H3_GND), U501.JP4-4 (H4_GND), U501.JP5-4 (GND), U502.2 (GND), U503.2 (GND), U504.2 (GND), U505.2 (GND), U506.4 (C-), U507.DC- (DC_GND), U507.TPG (TP_GND), U508.2 (GND)
- new net HDMI_CEC: J504.13 (CEC), J509.13 (CEC)
- new net HDMI_CKN: J504.12 (CK-), J509.12 (CK-)
- new net HDMI_CKP: J504.10 (CK+), J509.10 (CK+)
- new net HDMI_D0N: J504.9 (D0-), J509.9 (D0-)
- new net HDMI_D0P: J504.7 (D0+), J509.7 (D0+)
- new net HDMI_D1N: J504.6 (D1-), J509.6 (D1-)
- new net HDMI_D1P: J504.4 (D1+), J509.4 (D1+)
- new net HDMI_D2N: J504.3 (D2-), J509.3 (D2-)
- new net HDMI_D2P: J504.1 (D2+), J509.1 (D2+)
- new net HDMI_HPD: J504.19 (HPD), J509.19 (HPD)
- new net HDMI_SCL: J504.15 (SCL), J509.15 (SCL)
- new net HDMI_SDA: J504.16 (SDA), J509.16 (SDA)
- new net HDMI_SHELL: J504.SH, J509.SH
- new net HDMI_UTIL: J504.14 (UTILITY), J509.14 (UTILITY)
- new net HFP_DM: U501.JP4-3 (H4_D-)
- new net HFP_DP: U501.JP4-2 (H4_D+)
- new net HUB_DM: J501.2 (D1-), U501.JP5-3 (DMH(D-))
- new net HUB_DP: J501.3 (D1+), U501.JP5-2 (DPH(D+))
- new net I2C2_SCL: J512.4 (Pin_4)
- new net I2C2_SDA: J512.3 (Pin_3)
- new net I2CB_SCL: J511.2 (Pin_2)
- new net I2CB_SDA: J511.1 (Pin_1)
- new net IMU_RX: J510.3 (Pin_3), U508.3 (D2+)
- new net IMU_SHIELD: J510.SH (Shield)
- new net IMU_TX: J510.2 (Pin_2), U508.6 (D1-)
- new net LAB5: J510.1 (Pin_1), U501.JP5-1 (VBUS), U502.1 (IN), U503.1 (IN), U504.1 (IN), U505.1 (IN), U508.1 (D1+)
- new net LAB_DM: J507.2 (D-), U501.JP3-3 (H3_D-)
- new net LAB_DP: J507.3 (D+), U501.JP3-2 (H3_D+)
- new net MCP_INT: J512.5 (Pin_5)
- new net PCIE1_CLKREQ_N: J503.52 (~{CLKREQ})
- new net PCIE1_PERST_N: J503.50 (~{PERST})
- new net PCIE1_REFCLK_N: J503.53 (REFCLKn)
- new net PCIE1_REFCLK_P: J503.55 (REFCLKp)
- new net PCIE1_RX0_N: J503.41 (PERn0/SATA-B+)
- new net PCIE1_RX0_P: J503.43 (PERp0/SATA-B-)
- new net PCIE1_TX0_N: J503.47 (PETn0/SATA-A-)
- new net PCIE1_TX0_P: J503.49 (PETp0/SATA-A+)
- new net RTLA_DM: J505.2 (D-), U501.JP1-3 (H2_D-)
- new net RTLA_DP: J505.3 (D+), U501.JP1-2 (H2_D+)
- new net RTLB_DM: J502.11 (D2-), J506.2 (D-)
- new net RTLB_DP: J502.12 (D2+), J506.3 (D+)
- new net TP_DM: J501.6 (D2-), U507.TP- (TP_D-)
- new net TP_DP: J501.7 (D2+), U507.TP+ (TP_D+)
- new net U0_DM: J502.2 (D1-), J508.2 (Pin_2)
- new net U0_DP: J502.3 (D1+), J508.3 (Pin_3)
- new net U0_RXN: J502.5 (SSRX1-), J508.4 (Pin_4)
- new net U0_RXP: J502.6 (SSRX1+), J508.5 (Pin_5)
- new net U0_TXN: J502.8 (SSTX1-), J508.6 (Pin_6)
- new net U0_TXP: J502.9 (SSTX1+), J508.7 (Pin_7)
- new net UART5_RX: J513.2 (Pin_2)
- new net UART5_TX: J513.1 (Pin_1)
- new net VBUS_HFP: C501.1, L501.2, R506.1
- new net VBUS_LABPORT: J507.1 (VBUS), U504.6 (OUT)
- new net VBUS_RTLA: J505.1 (VBUS), U502.6 (OUT)
- new net VBUS_RTLB: J506.1 (VBUS), U503.6 (OUT)
- new net VCC_3V3_MKEY: J503.12 (3.3V), J503.14 (3.3V), J503.16 (3.3V), J503.18 (3.3V), J503.2 (3.3V), J503.4 (3.3V), J503.70 (3.3V), J503.72 (3.3V), J503.74 (3.3V)
- no-connect marks 0 -> 54
