File: sat-receiver-audit/build/kicad/E5.kicad_sch (KiCad schematic)
At the start: 51 parts, among them J501 LAB USB-A panel receptacle, J503 J21 service harness 3pin lock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, J511 Q6A J5 stacked USB3 lower / U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, J512 Q6A J2 stacked USB2 bank1 P3 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, J520 Q6A HDMI Type-A existing port, J521 Q6A J21 existing header pads, J541 RTL-B split-VBUS USB cable en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, J543 RTL-A USB cable endpoint, J544 HF+ microUSB-B cable endpoint, U500 Q6A onboard peripheral rail s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, U501 TPS2553DBVR-1, U502 TPS2553DBVR-1, U503 TPS2553DBVR, U505 TPS2553DRVR, U510 Adafruit5997 CH334F revC board, U540 Samsung T7 + intact A-to-C US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

Commit message: WIP: integration follow-ups
Made by the GPT/Codex run on 23.10.2026 (pushed as 5455b1e under the name "Claude");
re-attributed to Codex when integrated into ccr-1537979d-cj7q9t.
Parts:
- R512: footprint Resistor_SMD:R_0603_1608Metric -> Resistor_SMD:R_1210_3225Metric
Changed lines of the file:
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@@
 (property "Reference" "R512" (at 365.76 299.72 0) (effects (font (size 1.27 1.27)) ))
 (property "Value" "1Ohm 0.5W" (at 365.76 302.895 0) (effects (font (size 1.016 1.016)) ))
-(property "Footprint" "Resistor_SMD:R_0603_1608Metric" (at 365.76 298.45 0) (effects (font (size 1.016 1.016)) (hide yes)))
+(property "Footprint" "Resistor_SMD:R_1210_3225Metric" (at 365.76 298.45 0) (effects (font (size 1.016 1.016)) (hide yes)))
 (property "Datasheet" "STACK.md §5.2 / engineering design" (at 365.76 298.45 0) (effects (font (size 1.016 1.016)) (hide yes)))
 (property "Description" "" (at 365.76 298.45 0) (effects (font (size 1.016 1.016)) (hide yes)))
