File: sat-receiver-audit/build/kicad/E5.kicad_sch (KiCad schematic)
At the start: 51 parts, among them J501 LAB USB-A panel receptacle, J503 J21 service harness 3pin lock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, J511 Q6A J5 stacked USB3 lower / U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, J512 Q6A J2 stacked USB2 bank1 P3 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, J520 Q6A HDMI Type-A existing port, J521 Q6A J21 existing header pads, J541 RTL-B split-VBUS USB cable en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, J543 RTL-A USB cable endpoint, J544 HF+ microUSB-B cable endpoint, U500 Q6A onboard peripheral rail s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, U501 TPS2553DBVR-1, U502 TPS2553DBVR-1, U503 TPS2553DBVR, U505 TPS2553DRVR, U510 Adafruit5997 CH334F revC board, U540 Samsung T7 + intact A-to-C US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

Commit message: SR-RX-v2.1: review fixes on the Codex branch, readable schematic, one-file bundle
Independent review of the Codex branch (schematic vs STACK.md, hard rules,
security, tests) found no blockers; this commit applies its findings:

- rules in code: Cospas-Sarsat 406.0-406.1 MHz added to the no-data mask;
  Q6A Wi-Fi/BT off in the field/QUIET root (modprobe blacklist, udev
  authorized=0 on FE1.1s port 4, rfkill) with self-checks; device denylist
  completed per STACK (gr-gsm, gr-iridium, kalibrate, pager/trunking decoders,
  TX-capable tools); W1-2 WIFI_PWR_EN as blocking open item E5-10
- STACK.md is the source of truth again; v2.1 changes recorded in it; the
  "historical" marker kept only on ISDT/raw-balance rows; gender-neutral wording
- schematic data: open values shown as TBD with start values and notes, U503
  TPS2553DBVR-1, Lime X2/X4 RX mapping TBD, 37 open items drawn on the sheets
- schematic readability: wired groups, junctions, GND symbols, standard
  transistor/diode symbols; netlist unchanged (603 nets identical)
- tooling: reproducible run_checks (no timestamps or machine paths), pinned
  dependencies, bundle excludes cache folders, clean-checkout bundle check
- regenerated: KiCad export (14 pages), netlist/ERC, module lab, PCB inputs,
  readiness contract, acceptance hashes, SR-RX-v2-ves-proekt.html

Checks: ERC 0 errors/0 warnings, netlist comparison PASS, 432 tests (431
passed, 1 skipped), deployment tests OK, bundle check PASS on a clean checkout.

History note: earlier versions of the generated SR-RX-v2-ves-proekt.html and
handoff/handoff-bundle.zip were removed from history; only the final versions
are kept. The Codex merge commit is now attributed to Codex.

Co-Authored-By: Claude Opus 5.5 <noreply@anthropic.com>
Claude-Session: https://claude.ai/code/session_01W9CKpimWpgkUmrDQQMiKtF
Parts:
- removed J520: Q6A HDMI Type-A existing port, symbol sr_rx_v2_completed:C_J520
- removed R503: 10k, Resistor_SMD:R_0603_1608Metric, symbol sr_rx_v2_completed:C_R503
- removed R507: 10k, Resistor_SMD:R_0603_1608Metric, symbol sr_rx_v2_completed:C_R507
- removed R511: 10k, Resistor_SMD:R_0603_1608Metric, symbol sr_rx_v2_completed:C_R511
- added C550: 100nF X7R 10V, symbol sr_rx_v2_completed:C_C550
- added C551: 100nF X7R 10V, symbol sr_rx_v2_completed:C_C551
- added J530: Q6A MKEY host lane0 functional interface, symbol sr_rx_v2_completed:C_J530
- added R550: 4.7k 1%, Resistor_SMD:R_0603_1608Metric, symbol sr_rx_v2_completed:C_R550
- added R551: 4.7k 1%, Resistor_SMD:R_0603_1608Metric, symbol sr_rx_v2_completed:C_R551
- added U507: TCA9517DR, Package_SO:SOIC-8_3.9x4.9mm_P1.27mm, symbol sr_rx_v2_completed:C_U507
- added U530: ADT-Link R44SF 5cm modified riser, symbol sr_rx_v2_completed:C_U530
- R501: value 43.2k 1% -> RILIM TBD (start 43.2k 1%)
- R509: value 28.7k 1% -> RILIM TBD (start 28.7k 1%)
- R514: value 15.8k 1% -> RILIM TBD (start 15.8k 1%)
- U503: value TPS2553DBVR -> TPS2553DBVR-1
Connections:
- net 3V3_Q6A: now also C550.1, C551.1, R550.2, R551.2, U507.1 (VCCA), U507.5 (EN), U507.8 (VCCB)
- net GND: now also C550.2, C551.2, J530.GND, U507.4 (GND), U530.GND (common GND)
- new net E5_PCIE_CLKREQ_N: J530.CLKREQ_N (CLKREQ#), U530.C_CLKREQ_N (card CLKREQ#), U530.H_CLKREQ_N (host CLKREQ#)
- new net E5_PCIE_PERST_N: J530.PERST_N (PERST#), U530.C_PERST_N (card PERST#), U530.H_PERST_N (host PERST#)
- new net E5_PCIE_REFCLK_N: J530.REFCLK_N (REFCLK−), U530.C_REFCLK_N (card REFCLK−), U530.H_REFCLK_N (host REFCLK−)
- new net E5_PCIE_REFCLK_P: J530.REFCLK_P (REFCLK+), U530.C_REFCLK_P (card REFCLK+), U530.H_REFCLK_P (host REFCLK+)
- new net E5_PCIE_RX0_N: J530.RX0_N (host RX−), U530.C_RX0_N (card host RX−), U530.H_RX0_N (host host RX−)
- new net E5_PCIE_RX0_P: J530.RX0_P (host RX+), U530.C_RX0_P (card host RX+), U530.H_RX0_P (host host RX+)
- new net E5_PCIE_TX0_N: J530.TX0_N (host TX−), U530.C_TX0_N (card host TX−), U530.H_TX0_N (host host TX−)
- new net E5_PCIE_TX0_P: J530.TX0_P (host TX+), U530.C_TX0_P (card host TX+), U530.H_TX0_P (host host TX+)
- new net E5_PCIE_WAKE_N: J530.WAKE_N (WAKE#), U530.C_WAKE_N (card WAKE#), U530.H_WAKE_N (host WAKE#)
- new net I2C2_SCL: U507.2 (SCLA)
- new net I2C2_SDA: U507.3 (SDAA)
- new net I2CB_SCL: R551.1, U507.7 (SCLB)
- new net I2CB_SDA: R550.1, U507.6 (SDAB)
- new net LIME3V3: U530.C_3V3 (card 3V3 switched)
Other:
- note added: "ADT-Link R44SF connector variant and removal of ALL host 3.3 V paths are not yet confirmed. Ворота (стенд): Confirm the part with ADT-Link; continuity-test every 3.3 V contact after modification. Validate 8 GT/s x1, cold/warm boots and zero AER. Validate a genuine power-cycle with LIME3V3 off, including signal backfeed."
- note added: "Current-setting resistors R501 (RTL-A), R509 (HF+) and R514 (T7) are engineering starting values (RILIM TBD); STACK §5.1 fixes only the rule 1.5–2× measured current. No measured device steady/startup currents or hot-corner proof. Ворота (стенд): Measure current/inrush; set the RTL-A/HF+/T7 limits to 1.5–2× the measured current as STACK §5.1 requires; confirm HF+ minimum startup ≥0.75 A. Run the S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"
- note added: "E5-03 — OPEN, блокує випуск — STACK §2.11.1; §8.1 L-1, L-12"
- note added: "E5-04 — OPEN, блокує випуск — STACK §5.1 (VBUS RTL-A, HF+); §8 (TPS2553DBVR-1 п. 2–3)"
- note added: "E5-05 — OPEN, блокує випуск — STACK §5.1; §5.2; §8.1 (T7)"
- note added: "E5-09 — OPEN, блокує випуск — STACK §5.7; §8 (A/B-матриця); §8.2"
- note added: "E5-10 — OPEN, блокує випуск — STACK §5.2 (FE1.1s P4, WIFI_PWR_EN); §5.7 (рівень плати); §8 (блокування Wi-Fi/BT, W1-2); §1.2 (#8)"
- note added: "LAB BUS I2C buffer"
- note added: "N-E5-01 — примітка — STACK §5.1 (VBUS RTL-A); §8 (TPS2553DBVR-1 п. 2–3)"
- note added: "N-E5-02 — примітка — STACK §5.1, §5.2 (VBUS HF+); §8 (TPS2553DBVR-1 п. 3)"
- note added: "N-E5-03 — примітка — STACK §5.1; §8.1 (T7)"
- note added: "PCIe x1 riser та Lime"
- note added: "R501 = RILIM TBD (старт 43.2k 1%, 0.544–0.673 A). STACK для VBUS RTL-A задає лише правило RILIM = 1.5–2× виміряного струму; номінал STACK є тільки для порту LAB (R505 34.8k). Ворота: E5-04."
- note added: "R514 = RILIM TBD (старт 15.8k 1%, 1.51–1.73 A). STACK не задає RILIM для ключа T7 (U505 TPS2553DRVR без засувки — проєктне рішення R-E5-03/R-E5-04). Ворота: E5-04, E5-05."
- note added: "Radiated-noise behavior and USB2 touch enumeration are physical integration gates, not determined by netlist. Ворота (стенд): Run the STACK A/B noise matrix (HF+, GNSS, L-band, T7 authorized=0/off), cable strain relief and environmental tests; do not mark production-ready before passes."
- note added: "T7 VBUS rail capacity and modified cable SuperSpeed signal integrity untested. Ворота (стенд): With a real T7 prove J5 load <1.5 A expected operating budget, VCC_5V_PERI <=14 W, 5000M/UAS, no USB resets, fio, hot-corner TJ <=105 C for 1.5 A. Re-evaluate rail/switch/cable if failed."
- note added: "U503 = TPS2553DBVR-1 (засувка), як у STACK §5.1/§5.2. TPS2553DBVR зі сталим струмом (LCSC C55266) — лише на цьому каналі й лише якщо канал HF+ не пройде тест пускового струму STACK §8 (TPS2553DBVR-1, п. 3) при остаточному RILIM: LC 100 µH/100 µF + демпфер 220 µF ≈ 5.3 ms проти мін. deglitch 5 ms. R509 = RILIM TBD (старт 28.7k 1%). Ворота: E5-04."
- note added: "Wi-Fi/BT Q6A (FCU760K, AIC8800 на порту 4 FE1.1s) у польовому/QUIET root вимкнено лише програмно: blacklist з install /bin/false, udev authorized=0 за шляхом порту 4 і rfkill як другий шар. Апаратне утримання WIFI_PWR_EN (GPIO TLMM через CJ3134K до WIFI_PWR_EN_3V3, схема Radxa v1.21, с. 4) на отриманій платі не знайдено; gpio-hog у польовому DTBO не створено й не виміряно. Ворота (стенд): W1-2 (S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"
- note added: "Дроти з'єднують контакти всередині функціональної групи; кожне дерево дротів має одну глобальну мітку з канонічною назвою мережі (рамка-стрілка — мережа виходить за межі групи, пряма рамка — мережа лише цієї групи). Однакові мітки з'єднані на всіх аркушах; земля — символ GND. Рамки OPEN — незакриті ворота з design/E#.json (повний реєстр: OPEN_ITEMS.md); «TBD» у значенні — STACK номіналу не задає,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"
- note added: "Позначення фізичних джерел живлення (ERC)"
- note removed: "Дисплей HDMI, DC і USB touch"
- note removed: "Мережі з однаковими глобальними мітками електрично з'єднані на всіх аркушах. Фізичні/функціональні контакти: див. design/ і OPEN_ITEMS.md."
- moved on the sheet: J501, J503, J511, J512, J521, J541, J543, J544, U500, U501, U502, U503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
