File: sat-receiver-audit/build/kicad/sr-rx-v2.kicad_sch (KiCad schematic)
At the start: 0 parts

Commit message: Complete SR-RX-v2.1 schematics and verification package
Replace five empty sheets with reviewed KiCad schematics and portable resources. Correct power, control, USB and RF interfaces; document hardware acceptance gates and unimplemented firmware/PCB work. Validate 754 components, 2189 connected contacts and 466 nets with zero ERC violations and two independent graph/netlist comparisons. Include PDF, SVG, BOM, reproducible tools and offline documentation.
Other:
- removed sheet E1 Живлення: акумулятор, захист, перетворювачі
- removed sheet E2 Живлення: захищені канали і LNB
- removed sheet E3 Керування: Q6A, I2C, GPIO, GNSS
- removed sheet E4 РЧ-тракт
- removed sheet E5 USB, VBUS і роз'єми корпусу
- added sheet E1 (E1.kicad_sch)
- added sheet E1_02 (E1_02.kicad_sch)
- added sheet E2 (E2.kicad_sch)
- added sheet E2_02 (E2_02.kicad_sch)
- added sheet E2_03 (E2_03.kicad_sch)
- added sheet E2_04 (E2_04.kicad_sch)
- added sheet E2_05 (E2_05.kicad_sch)
- added sheet E3 (E3.kicad_sch)
- added sheet E3_02 (E3_02.kicad_sch)
- added sheet E3_03 (E3_03.kicad_sch)
- added sheet E4 (E4.kicad_sch)
- added sheet E4_02 (E4_02.kicad_sch)
- added sheet E4_03 (E4_03.kicad_sch)
- added sheet E4_04 (E4_04.kicad_sch)
- added sheet E5 (E5.kicad_sch)
- added sheet E5_02 (E5_02.kicad_sch)
- note added: "SR-RX-v2: приймач і портативна радіолабораторія"
- note added: "USB, VBUS, PCIe та корпусні інтерфейси (1/2)"
- note added: "USB, VBUS, PCIe та корпусні інтерфейси (2/2)"
- note added: "Акумулятор, заряд, AON і головні перетворювачі (1/2)"
- note added: "Акумулятор, заряд, AON і головні перетворювачі (2/2)"
- note added: "Захищені рейки, LNA і моніторинг струму (1/5)"
- note added: "Захищені рейки, LNA і моніторинг струму (2/5)"
- note added: "Захищені рейки, LNA і моніторинг струму (3/5)"
- note added: "Захищені рейки, LNA і моніторинг струму (4/5)"
- note added: "Захищені рейки, LNA і моніторинг струму (5/5)"
- note added: "Керування, Pico HMI, GPIO, GNSS і IMU (1/3)"
- note added: "Керування, Pico HMI, GPIO, GNSS і IMU (2/3)"
- note added: "Керування, Pico HMI, GPIO, GNSS і IMU (3/3)"
- note added: "Лише прийом в ефірі. Інженерна редакція від 4653188. Статус і незакриті ворота: ../../COMPLETION.md та ../../OPEN_ITEMS.md."
- note added: "РЧ-тракт: DC-розвʼязка, перемикачі, реле та приймачі (1/4)"
- note added: "РЧ-тракт: DC-розвʼязка, перемикачі, реле та приймачі (2/4)"
- note added: "РЧ-тракт: DC-розвʼязка, перемикачі, реле та приймачі (3/4)"
- note added: "РЧ-тракт: DC-розвʼязка, перемикачі, реле та приймачі (4/4)"
- note removed: "SR-RX-v2 — супутниковий приймач лише на прийом і портативна радіолабораторія. Схема електрична принципова за STACK.md v2 (18.10.2026). Теоретичний проєкт — перевірити на стенді. Аркуші: E1 живлення, E2 захищені канали і LNB, E3 керування, E4 РЧ-тракт, E5 USB/VBUS і роз'єми."
- company: (none) -> SR-RX-v2
- title: (none) -> SR-RX-v2 - зміст електричної схеми
