File: sat-receiver-audit/build/kicad/sr-rx-v2.kicad_sch (KiCad schematic)
At the start: 0 parts

Commit message: SR-RX-v2.1: review fixes on the Codex branch, readable schematic, one-file bundle
Independent review of the Codex branch (schematic vs STACK.md, hard rules,
security, tests) found no blockers; this commit applies its findings:

- rules in code: Cospas-Sarsat 406.0-406.1 MHz added to the no-data mask;
  Q6A Wi-Fi/BT off in the field/QUIET root (modprobe blacklist, udev
  authorized=0 on FE1.1s port 4, rfkill) with self-checks; device denylist
  completed per STACK (gr-gsm, gr-iridium, kalibrate, pager/trunking decoders,
  TX-capable tools); W1-2 WIFI_PWR_EN as blocking open item E5-10
- STACK.md is the source of truth again; v2.1 changes recorded in it; the
  "historical" marker kept only on ISDT/raw-balance rows; gender-neutral wording
- schematic data: open values shown as TBD with start values and notes, U503
  TPS2553DBVR-1, Lime X2/X4 RX mapping TBD, 37 open items drawn on the sheets
- schematic readability: wired groups, junctions, GND symbols, standard
  transistor/diode symbols; netlist unchanged (603 nets identical)
- tooling: reproducible run_checks (no timestamps or machine paths), pinned
  dependencies, bundle excludes cache folders, clean-checkout bundle check
- regenerated: KiCad export (14 pages), netlist/ERC, module lab, PCB inputs,
  readiness contract, acceptance hashes, SR-RX-v2-ves-proekt.html

Checks: ERC 0 errors/0 warnings, netlist comparison PASS, 432 tests (431
passed, 1 skipped), deployment tests OK, bundle check PASS on a clean checkout.

History note: earlier versions of the generated SR-RX-v2-ves-proekt.html and
handoff/handoff-bundle.zip were removed from history; only the final versions
are kept. The Codex merge commit is now attributed to Codex.

Co-Authored-By: Claude Opus 5.5 <noreply@anthropic.com>
Claude-Session: https://claude.ai/code/session_01W9CKpimWpgkUmrDQQMiKtF
Other:
- removed sheet E1_02
- removed sheet E2_05
- removed sheet E3_03
- note added: "Акумулятор, заряд, AON і головні перетворювачі (1/1)"
- note added: "Захищені рейки, LNA і моніторинг струму (1/4)"
- note added: "Захищені рейки, LNA і моніторинг струму (2/4)"
- note added: "Захищені рейки, LNA і моніторинг струму (3/4)"
- note added: "Захищені рейки, LNA і моніторинг струму (4/4)"
- note added: "Керування, Pico HMI, GPIO, GNSS і IMU (1/2)"
- note added: "Керування, Pico HMI, GPIO, GNSS і IMU (2/2)"
- note added: "РЧ-тракт: DC-розв'язка, перемикачі, приймачі (1/4)"
- note added: "РЧ-тракт: DC-розв'язка, перемикачі, приймачі (2/4)"
- note added: "РЧ-тракт: DC-розв'язка, перемикачі, приймачі (3/4)"
- note added: "РЧ-тракт: DC-розв'язка, перемикачі, приймачі (4/4)"
- note removed: "Акумулятор, заряд, AON і головні перетворювачі (1/2)"
- note removed: "Акумулятор, заряд, AON і головні перетворювачі (2/2)"
- note removed: "Захищені рейки, LNA і моніторинг струму (1/5)"
- note removed: "Захищені рейки, LNA і моніторинг струму (2/5)"
- note removed: "Захищені рейки, LNA і моніторинг струму (3/5)"
- note removed: "Захищені рейки, LNA і моніторинг струму (4/5)"
- note removed: "Захищені рейки, LNA і моніторинг струму (5/5)"
- note removed: "Керування, Pico HMI, GPIO, GNSS і IMU (1/3)"
- note removed: "Керування, Pico HMI, GPIO, GNSS і IMU (2/3)"
- note removed: "Керування, Pico HMI, GPIO, GNSS і IMU (3/3)"
- note removed: "РЧ-тракт: DC-розвʼязка, перемикачі, реле та приймачі (1/4)"
- note removed: "РЧ-тракт: DC-розвʼязка, перемикачі, реле та приймачі (2/4)"
- note removed: "РЧ-тракт: DC-розвʼязка, перемикачі, реле та приймачі (3/4)"
- note removed: "РЧ-тракт: DC-розвʼязка, перемикачі, реле та приймачі (4/4)"
