File: sat-receiver-audit/build/kicad/sr-rx-v2.kicad_sch (KiCad schematic)
At the start: 0 parts

Commit message: GENERATED: CAD, netlist, ERC, documents and re-frozen DC_CORE PCB chain from CI
Applied verbatim from the cad-regenerated artifacts of run 40087342176
(for source commit c17ae81) and run 40090126917 (for the review fixes,
source commit 4740951); KiCad 10.0.7, refreeze_pcb=true.

Co-Authored-By: Claude Opus 5.5 <noreply@anthropic.com>
Other:
- added sheet E2_05 (E2_05.kicad_sch)
- note added: "Захищені рейки, LNA і моніторинг струму (1/5)"
- note added: "Захищені рейки, LNA і моніторинг струму (2/5)"
- note added: "Захищені рейки, LNA і моніторинг струму (3/5)"
- note added: "Захищені рейки, LNA і моніторинг струму (4/5)"
- note added: "Захищені рейки, LNA і моніторинг струму (5/5)"
- note removed: "Захищені рейки, LNA і моніторинг струму (1/4)"
- note removed: "Захищені рейки, LNA і моніторинг струму (2/4)"
- note removed: "Захищені рейки, LNA і моніторинг струму (3/4)"
- note removed: "Захищені рейки, LNA і моніторинг струму (4/4)"
Changed lines of the file:
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@@
  (property "Sheetfile" "E2.kicad_sch" (at 364.49 63.5 0) (effects (font (size 1.016 1.016)) ))
  (instances (project "sr-rx-v2" (path "/fb9ec709-453b-5b24-a782-9cee42ec6d25" (page "4")))))
-(text "Захищені рейки, LNA і моніторинг струму (1/4)" (at 304.8 52.07 0) (effects (font (size 1.016 1.016)) (justify left top)))
+(text "Захищені рейки, LNA і моніторинг струму (1/5)" (at 304.8 52.07 0) (effects (font (size 1.016 1.016)) (justify left top)))
 (sheet (at 441.96 43.18) (size 129.54 27.94)
  (stroke (width 0.254) (type default)) (fill (color 0 0 0 0))
@@
  (property "Sheetfile" "E2_02.kicad_sch" (at 506.73 63.5 0) (effects (font (size 1.016 1.016)) ))
  (instances (project "sr-rx-v2" (path "/fb9ec709-453b-5b24-a782-9cee42ec6d25" (page "5")))))
-(text "Захищені рейки, LNA і моніторинг струму (2/4)" (at 447.04 52.07 0) (effects (font (size 1.016 1.016)) (justify left top)))
+(text "Захищені рейки, LNA і моніторинг струму (2/5)" (at 447.04 52.07 0) (effects (font (size 1.016 1.016)) (justify left top)))
 (sheet (at 15.24 81.28) (size 129.54 27.94)
  (stroke (width 0.254) (type default)) (fill (color 0 0 0 0))
@@
  (property "Sheetfile" "E2_03.kicad_sch" (at 80.01 101.6 0) (effects (font (size 1.016 1.016)) ))
  (instances (project "sr-rx-v2" (path "/fb9ec709-453b-5b24-a782-9cee42ec6d25" (page "6")))))
-(text "Захищені рейки, LNA і моніторинг струму (3/4)" (at 20.32 90.17 0) (effects (font (size 1.016 1.016)) (justify left top)))
+(text "Захищені рейки, LNA і моніторинг струму (3/5)" (at 20.32 90.17 0) (effects (font (size 1.016 1.016)) (justify left top)))
 (sheet (at 157.48 81.28) (size 129.54 27.94)
  (stroke (width 0.254) (type default)) (fill (color 0 0 0 0))
@@
  (property "Sheetfile" "E2_04.kicad_sch" (at 222.25 101.6 0) (effects (font (size 1.016 1.016)) ))
  (instances (project "sr-rx-v2" (path "/fb9ec709-453b-5b24-a782-9cee42ec6d25" (page "7")))))
-(text "Захищені рейки, LNA і моніторинг струму (4/4)" (at 162.56 90.17 0) (effects (font (size 1.016 1.016)) (justify left top)))
+(text "Захищені рейки, LNA і моніторинг струму (4/5)" (at 162.56 90.17 0) (effects (font (size 1.016 1.016)) (justify left top)))
 (sheet (at 299.72 81.28) (size 129.54 27.94)
  (stroke (width 0.254) (type default)) (fill (color 0 0 0 0))
- (property "Sheetname" "E3" (at 364.49 85.725 0) (effects (font (size 1.016 1.016)) ))
- (property "Sheetfile" "E3.kicad_sch" (at 364.49 101.6 0) (effects (font (size 1.016 1.016)) ))
+ (property "Sheetname" "E2_05" (at 364.49 85.725 0) (effects (font (size 1.016 1.016)) ))
+ (property "Sheetfile" "E2_05.kicad_sch" (at 364.49 101.6 0) (effects (font (size 1.016 1.016)) ))
  (instances (project "sr-rx-v2" (path "/fb9ec709-453b-5b24-a782-9cee42ec6d25" (page "8")))))
-(text "Керування, Pico HMI, GPIO, GNSS і IMU (1/2)" (at 304.8 90.17 0) (effects (font (size 1.016 1.016)) (justify left top)))
+(text "Захищені рейки, LNA і моніторинг струму (5/5)" (at 304.8 90.17 0) (effects (font (size 1.016 1.016)) (justify left top)))
 (sheet (at 441.96 81.28) (size 129.54 27.94)
  (stroke (width 0.254) (type default)) (fill (color 0 0 0 0))
- (property "Sheetname" "E3_02" (at 506.73 85.725 0) (effects (font (size 1.016 1.016)) ))
- (property "Sheetfile" "E3_02.kicad_sch" (at 506.73 101.6 0) (effects (font (size 1.016 1.016)) ))
+ (property "Sheetname" "E3" (at 506.73 85.725 0) (effects (font (size 1.016 1.016)) ))
+ (property "Sheetfile" "E3.kicad_sch" (at 506.73 101.6 0) (effects (font (size 1.016 1.016)) ))
  (instances (project "sr-rx-v2" (path "/fb9ec709-453b-5b24-a782-9cee42ec6d25" (page "9")))))
-(text "Керування, Pico HMI, GPIO, GNSS і IMU (2/2)" (at 447.04 90.17 0) (effects (font (size 1.016 1.016)) (justify left top)))
+(text "Керування, Pico HMI, GPIO, GNSS і IMU (1/2)" (at 447.04 90.17 0) (effects (font (size 1.016 1.016)) (justify left top)))
 (sheet (at 15.24 119.38) (size 129.54 27.94)
  (stroke (width 0.254) (type default)) (fill (color 0 0 0 0))
- (property "Sheetname" "E4" (at 80.01 123.825 0) (effects (font (size 1.016 1.016)) ))
- (property "Sheetfile" "E4.kicad_sch" (at 80.01 139.7 0) (effects (font (size 1.016 1.016)) ))
+ (property "Sheetname" "E3_02" (at 80.01 123.825 0) (effects (font (size 1.016 1.016)) ))
+ (property "Sheetfile" "E3_02.kicad_sch" (at 80.01 139.7 0) (effects (font (size 1.016 1.016)) ))
  (instances (project "sr-rx-v2" (path "/fb9ec709-453b-5b24-a782-9cee42ec6d25" (page "10")))))
-(text "РЧ-тракт: DC-розв'язка, перемикачі, приймачі\n(1/4)" (at 20.32 128.27 0) (effects (font (size 1.016 1.016)) (justify left top)))
+(text "Керування, Pico HMI, GPIO, GNSS і IMU (2/2)" (at 20.32 128.27 0) (effects (font (size 1.016 1.016)) (justify left top)))
 (sheet (at 157.48 119.38) (size 129.54 27.94)
  (stroke (width 0.254) (type default)) (fill (color 0 0 0 0))
- (property "Sheetname" "E4_02" (at 222.25 123.825 0) (effects (font (size 1.016 1.016)) ))
- (property "Sheetfile" "E4_02.kicad_sch" (at 222.25 139.7 0) (effects (font (size 1.016 1.016)) ))
+ (property "Sheetname" "E4" (at 222.25 123.825 0) (effects (font (size 1.016 1.016)) ))
+ (property "Sheetfile" "E4.kicad_sch" (at 222.25 139.7 0) (effects (font (size 1.016 1.016)) ))
  (instances (project "sr-rx-v2" (path "/fb9ec709-453b-5b24-a782-9cee42ec6d25" (page "11")))))
-(text "РЧ-тракт: DC-розв'язка, перемикачі, приймачі\n(2/4)" (at 162.56 128.27 0) (effects (font (size 1.016 1.016)) (justify left top)))
+(text "РЧ-тракт: DC-розв'язка, перемикачі, приймачі\n(1/4)" (at 162.56 128.27 0) (effects (font (size 1.016 1.016)) (justify left top)))
 (sheet (at 299.72 119.38) (size 129.54 27.94)
  (stroke (width 0.254) (type default)) (fill (color 0 0 0 0))
- (property "Sheetname" "E4_03" (at 364.49 123.825 0) (effects (font (size 1.016 1.016)) ))
- (property "Sheetfile" "E4_03.kicad_sch" (at 364.49 139.7 0) (effects (font (size 1.016 1.016)) ))
+ (property "Sheetname" "E4_02" (at 364.49 123.825 0) (effects (font (size 1.016 1.016)) ))
+ (property "Sheetfile" "E4_02.kicad_sch" (at 364.49 139.7 0) (effects (font (size 1.016 1.016)) ))
  (instances (project "sr-rx-v2" (path "/fb9ec709-453b-5b24-a782-9cee42ec6d25" (page "12")))))
-(text "РЧ-тракт: DC-розв'язка, перемикачі, приймачі\n(3/4)" (at 304.8 128.27 0) (effects (font (size 1.016 1.016)) (justify left top)))
+(text "РЧ-тракт: DC-розв'язка, перемикачі, приймачі\n(2/4)" (at 304.8 128.27 0) (effects (font (size 1.016 1.016)) (justify left top)))
 (sheet (at 441.96 119.38) (size 129.54 27.94)
  (stroke (width 0.254) (type default)) (fill (color 0 0 0 0))
- (property "Sheetname" "E4_04" (at 506.73 123.825 0) (effects (font (size 1.016 1.016)) ))
- (property "Sheetfile" "E4_04.kicad_sch" (at 506.73 139.7 0) (effects (font (size 1.016 1.016)) ))
+ (property "Sheetname" "E4_03" (at 506.73 123.825 0) (effects (font (size 1.016 1.016)) ))
+ (property "Sheetfile" "E4_03.kicad_sch" (at 506.73 139.7 0) (effects (font (size 1.016 1.016)) ))
  (instances (project "sr-rx-v2" (path "/fb9ec709-453b-5b24-a782-9cee42ec6d25" (page "13")))))
-(text "РЧ-тракт: DC-розв'язка, перемикачі, приймачі\n(4/4)" (at 447.04 128.27 0) (effects (font (size 1.016 1.016)) (justify left top)))
+(text "РЧ-тракт: DC-розв'язка, перемикачі, приймачі\n(3/4)" (at 447.04 128.27 0) (effects (font (size 1.016 1.016)) (justify left top)))
 (sheet (at 15.24 157.48) (size 129.54 27.94)
  (stroke (width 0.254) (type default)) (fill (color 0 0 0 0))
- (property "Sheetname" "E5" (at 80.01 161.925 0) (effects (font (size 1.016 1.016)) ))
- (property "Sheetfile" "E5.kicad_sch" (at 80.01 177.8 0) (effects (font (size 1.016 1.016)) ))
+ (property "Sheetname" "E4_04" (at 80.01 161.925 0) (effects (font (size 1.016 1.016)) ))
+ (property "Sheetfile" "E4_04.kicad_sch" (at 80.01 177.8 0) (effects (font (size 1.016 1.016)) ))
  (instances (project "sr-rx-v2" (path "/fb9ec709-453b-5b24-a782-9cee42ec6d25" (page "14")))))
-(text "USB, VBUS, PCIe та корпусні інтерфейси (1/2)" (at 20.32 166.37 0) (effects (font (size 1.016 1.016)) (justify left top)))
+(text "РЧ-тракт: DC-розв'язка, перемикачі, приймачі\n(4/4)" (at 20.32 166.37 0) (effects (font (size 1.016 1.016)) (justify left top)))
 (sheet (at 157.48 157.48) (size 129.54 27.94)
  (stroke (width 0.254) (type default)) (fill (color 0 0 0 0))
- (property "Sheetname" "E5_02" (at 222.25 161.925 0) (effects (font (size 1.016 1.016)) ))
- (property "Sheetfile" "E5_02.kicad_sch" (at 222.25 177.8 0) (effects (font (size 1.016 1.016)) ))
+ (property "Sheetname" "E5" (at 222.25 161.925 0) (effects (font (size 1.016 1.016)) ))
+ (property "Sheetfile" "E5.kicad_sch" (at 222.25 177.8 0) (effects (font (size 1.016 1.016)) ))
  (instances (project "sr-rx-v2" (path "/fb9ec709-453b-5b24-a782-9cee42ec6d25" (page "15")))))
-(text "USB, VBUS, PCIe та корпусні інтерфейси (2/2)" (at 162.56 166.37 0) (effects (font (size 1.016 1.016)) (justify left top)))
+(text "USB, VBUS, PCIe та корпусні інтерфейси (1/2)" (at 162.56 166.37 0) (effects (font (size 1.016 1.016)) (justify left top)))
+(sheet (at 299.72 157.48) (size 129.54 27.94)
+ (stroke (width 0.254) (type default)) (fill (color 0 0 0 0))
+ (property "Sheetname" "E5_02" (at 364.49 161.925 0) (effects (font (size 1.016 1.016)) ))
+ (property "Sheetfile" "E5_02.kicad_sch" (at 364.49 177.8 0) (effects (font (size 1.016 1.016)) ))
+ (instances (project "sr-rx-v2" (path "/fb9ec709-453b-5b24-a782-9cee42ec6d25" (page "16")))))
+(text "USB, VBUS, PCIe та корпусні інтерфейси (2/2)" (at 304.8 166.37 0) (effects (font (size 1.016 1.016)) (justify left top)))
 (sheet_instances (path "/" (page "1")))
 )
