File: sat-receiver-audit/build/kicad/sr-rx-v2.kicad_sch (KiCad schematic)
At the start: 0 parts

Commit message: Stage 2 integration: CAD and DC_CORE re-freeze from CI run 40094234222; bound-count test and PCB hash lists follow
Co-Authored-By: Claude Opus 5.5 <noreply@anthropic.com>
Other:
- removed sheet E1_02
- added sheet E2_05 (E2_05.kicad_sch)
- note added: "Акумулятор, заряд, AON і головні перетворювачі (1/1)"
- note added: "Захищені рейки, LNA і моніторинг струму (1/5)"
- note added: "Захищені рейки, LNA і моніторинг струму (2/5)"
- note added: "Захищені рейки, LNA і моніторинг струму (3/5)"
- note added: "Захищені рейки, LNA і моніторинг струму (4/5)"
- note added: "Захищені рейки, LNA і моніторинг струму (5/5)"
- note removed: "Акумулятор, заряд, AON і головні перетворювачі (1/2)"
- note removed: "Акумулятор, заряд, AON і головні перетворювачі (2/2)"
- note removed: "Захищені рейки, LNA і моніторинг струму (1/4)"
- note removed: "Захищені рейки, LNA і моніторинг струму (2/4)"
- note removed: "Захищені рейки, LNA і моніторинг струму (3/4)"
- note removed: "Захищені рейки, LNA і моніторинг струму (4/4)"
Changed lines of the file:
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@@
  (property "Sheetfile" "E1.kicad_sch" (at 80.01 63.5 0) (effects (font (size 1.016 1.016)) ))
  (instances (project "sr-rx-v2" (path "/fb9ec709-453b-5b24-a782-9cee42ec6d25" (page "2")))))
-(text "Акумулятор, заряд, AON і головні\nперетворювачі (1/2)" (at 20.32 52.07 0) (effects (font (size 1.016 1.016)) (justify left top)))
+(text "Акумулятор, заряд, AON і головні\nперетворювачі (1/1)" (at 20.32 52.07 0) (effects (font (size 1.016 1.016)) (justify left top)))
 (sheet (at 157.48 43.18) (size 129.54 27.94)
  (stroke (width 0.254) (type default)) (fill (color 0 0 0 0))
- (property "Sheetname" "E1_02" (at 222.25 47.625 0) (effects (font (size 1.016 1.016)) ))
- (property "Sheetfile" "E1_02.kicad_sch" (at 222.25 63.5 0) (effects (font (size 1.016 1.016)) ))
+ (property "Sheetname" "E2" (at 222.25 47.625 0) (effects (font (size 1.016 1.016)) ))
+ (property "Sheetfile" "E2.kicad_sch" (at 222.25 63.5 0) (effects (font (size 1.016 1.016)) ))
  (instances (project "sr-rx-v2" (path "/fb9ec709-453b-5b24-a782-9cee42ec6d25" (page "3")))))
-(text "Акумулятор, заряд, AON і головні\nперетворювачі (2/2)" (at 162.56 52.07 0) (effects (font (size 1.016 1.016)) (justify left top)))
+(text "Захищені рейки, LNA і моніторинг струму (1/5)" (at 162.56 52.07 0) (effects (font (size 1.016 1.016)) (justify left top)))
 (sheet (at 299.72 43.18) (size 129.54 27.94)
  (stroke (width 0.254) (type default)) (fill (color 0 0 0 0))
- (property "Sheetname" "E2" (at 364.49 47.625 0) (effects (font (size 1.016 1.016)) ))
- (property "Sheetfile" "E2.kicad_sch" (at 364.49 63.5 0) (effects (font (size 1.016 1.016)) ))
+ (property "Sheetname" "E2_02" (at 364.49 47.625 0) (effects (font (size 1.016 1.016)) ))
+ (property "Sheetfile" "E2_02.kicad_sch" (at 364.49 63.5 0) (effects (font (size 1.016 1.016)) ))
  (instances (project "sr-rx-v2" (path "/fb9ec709-453b-5b24-a782-9cee42ec6d25" (page "4")))))
-(text "Захищені рейки, LNA і моніторинг струму (1/4)" (at 304.8 52.07 0) (effects (font (size 1.016 1.016)) (justify left top)))
+(text "Захищені рейки, LNA і моніторинг струму (2/5)" (at 304.8 52.07 0) (effects (font (size 1.016 1.016)) (justify left top)))
 (sheet (at 441.96 43.18) (size 129.54 27.94)
  (stroke (width 0.254) (type default)) (fill (color 0 0 0 0))
- (property "Sheetname" "E2_02" (at 506.73 47.625 0) (effects (font (size 1.016 1.016)) ))
- (property "Sheetfile" "E2_02.kicad_sch" (at 506.73 63.5 0) (effects (font (size 1.016 1.016)) ))
+ (property "Sheetname" "E2_03" (at 506.73 47.625 0) (effects (font (size 1.016 1.016)) ))
+ (property "Sheetfile" "E2_03.kicad_sch" (at 506.73 63.5 0) (effects (font (size 1.016 1.016)) ))
  (instances (project "sr-rx-v2" (path "/fb9ec709-453b-5b24-a782-9cee42ec6d25" (page "5")))))
-(text "Захищені рейки, LNA і моніторинг струму (2/4)" (at 447.04 52.07 0) (effects (font (size 1.016 1.016)) (justify left top)))
+(text "Захищені рейки, LNA і моніторинг струму (3/5)" (at 447.04 52.07 0) (effects (font (size 1.016 1.016)) (justify left top)))
 (sheet (at 15.24 81.28) (size 129.54 27.94)
  (stroke (width 0.254) (type default)) (fill (color 0 0 0 0))
- (property "Sheetname" "E2_03" (at 80.01 85.725 0) (effects (font (size 1.016 1.016)) ))
- (property "Sheetfile" "E2_03.kicad_sch" (at 80.01 101.6 0) (effects (font (size 1.016 1.016)) ))
+ (property "Sheetname" "E2_04" (at 80.01 85.725 0) (effects (font (size 1.016 1.016)) ))
+ (property "Sheetfile" "E2_04.kicad_sch" (at 80.01 101.6 0) (effects (font (size 1.016 1.016)) ))
  (instances (project "sr-rx-v2" (path "/fb9ec709-453b-5b24-a782-9cee42ec6d25" (page "6")))))
-(text "Захищені рейки, LNA і моніторинг струму (3/4)" (at 20.32 90.17 0) (effects (font (size 1.016 1.016)) (justify left top)))
+(text "Захищені рейки, LNA і моніторинг струму (4/5)" (at 20.32 90.17 0) (effects (font (size 1.016 1.016)) (justify left top)))
 (sheet (at 157.48 81.28) (size 129.54 27.94)
  (stroke (width 0.254) (type default)) (fill (color 0 0 0 0))
- (property "Sheetname" "E2_04" (at 222.25 85.725 0) (effects (font (size 1.016 1.016)) ))
- (property "Sheetfile" "E2_04.kicad_sch" (at 222.25 101.6 0) (effects (font (size 1.016 1.016)) ))
+ (property "Sheetname" "E2_05" (at 222.25 85.725 0) (effects (font (size 1.016 1.016)) ))
+ (property "Sheetfile" "E2_05.kicad_sch" (at 222.25 101.6 0) (effects (font (size 1.016 1.016)) ))
  (instances (project "sr-rx-v2" (path "/fb9ec709-453b-5b24-a782-9cee42ec6d25" (page "7")))))
-(text "Захищені рейки, LNA і моніторинг струму (4/4)" (at 162.56 90.17 0) (effects (font (size 1.016 1.016)) (justify left top)))
+(text "Захищені рейки, LNA і моніторинг струму (5/5)" (at 162.56 90.17 0) (effects (font (size 1.016 1.016)) (justify left top)))
 (sheet (at 299.72 81.28) (size 129.54 27.94)
  (stroke (width 0.254) (type default)) (fill (color 0 0 0 0))
