File: sat-receiver-audit/build/kicad/E2.kicad_sch (KiCad schematic)
At the start: 0 parts

Commit message: KiCad sheets E1/E2/E5 partial (work before agent limit)
Co-Authored-By: Claude Opus 5.5 <noreply@anthropic.com>
Claude-Session: https://claude.ai/code/session_01W9CKpimWpgkUmrDQQMiKtF
Parts:
- added C201, C207, C208, C209, C216, C221: CdVdT TBD, symbol Device:C
- added C202, C203, C205, C206, C212, C213, C217, C218: C TBD, symbol Device:C
- added C204: UHE1E221MPD, symbol Device:C_Polarized
- added C210: EEU-FR1C101, symbol Device:C_Polarized
- added C211: 220u, symbol Device:C_Polarized
- added C214, C219: CNR TBD, symbol Device:C
- added C215, C220: COUT TBD, symbol Device:C
- added D201: SMBJ13A, Diode_SMD:D_SMB, symbol sr_rx_v2_pwr:SMBJ13A
- added D202, D203: Schottky TBD, symbol Device:D_Schottky
- added F201: 0297004.WXNV, symbol Device:Fuse
- added F202: MF-MSMF075/24-2, symbol Device:Polyfuse
- added JP201: 13V2, symbol Jumper:SolderJumper_2_Bridged
- added JP202, JP203: 12V5, symbol Jumper:SolderJumper_2_Open
- added L201, L202, L204, L205: L TBD, symbol Device:L
- added L203: SRR1260-101M, symbol Device:L
- added Q201: AO3407A, symbol Transistor_FET:Q_PMOS_GSD
- added Q202: 2N7002, Package_TO_SOT_SMD:SOT-23, symbol Transistor_FET:2N7002
- added R201, R208: R1 TBD, symbol Device:R
- added R202, R209: R2 TBD, symbol Device:R
- added R203, R210: R3 TBD, symbol Device:R
- added R204, R207, R211: RILM TBD, symbol Device:R
- added R205, R212, R230: ROV1 TBD, symbol Device:R
- added R206, R213, R231: ROV2 TBD, symbol Device:R
- added R214: 1.65k, symbol Device:R
- added R215: 34.8k, symbol Device:R
- added R216, R218, R219: RILIM TBD, symbol Device:R
- added R217: ≈1R, symbol Device:R
- added R220, R221, R222: 88.7k, symbol Device:R
- added R223: 162k, symbol Device:R
- added R224: 110k 0.5%, symbol Device:R
- added R225: 10.0k 0.5%, symbol Device:R
- added R226: 2.05k 1%, symbol Device:R
- added R227, R232: RPG1 TBD, symbol Device:R
- added R228, R233: RPG2 TBD, symbol Device:R
- added R229: 7.87k, symbol Device:R
- added R234, R235: 10k, symbol Device:R
- added U201, U202, U203, U204: TPS259470ARPWR, symbol sr_rx_v2_pwr:TPS259470ARPWR
- added U205, U206, U207, U208, U209, U210, U211, U212: TPS2553DBVR-1, Package_TO_SOT_SMD:SOT-23-6, symbol sr_rx_v2_pwr:TPS2553DBVR-1
- added U213, U216: TPS7A4701RGWT, Package_DFN_QFN:Texas_RGW0020A_VQFN-20-1EP_5x5mm_P0.65mm_EP3.15x3.15mm_ThermalVias, symbol sr_rx_v2_pwr:TPS7A4701RGWT
- added U214, U217: TPS259630DDAR, Package_SO:TI_SO-PowerPAD-8_ThermalVias, symbol Power_Management:TPS2596xx
- added U215, U218: TLV3011, symbol sr_rx_v2_pwr:TLV3011
Connections:
- new net: C201.1, U201.7 (DVDT)
- new net: R220.1, U209.5 (ILIM)
- new net: C218.1, L205.2, U216.15 (IN), U216.16 (IN)
- new net: C215.1, D202.1 (K), R224.1, U213.1 (OUT), U213.20 (OUT), U213.3 (SENSE/FB), U214.4 (VIN)
- new net: R224.2, R225.1, U214.8 (OVLO/OVCSEL)
- new net: R229.1, U217.7 (ILM)
- new net: R227.2, R228.1, U215.3 (IN+)
- new net: C209.1, U204.7 (DVDT)
- new net: R214.1, U204.9 (ILM)
- new net: F201.2, R201.1, U201.5 (IN)
- new net: R218.1, U207.5 (ILIM)
- new net: R215.1, U205.5 (ILIM)
- new net: C206.1, L202.2, R205.1, U202.5 (IN)
- new net: R216.1, U206.5 (ILIM)
- new net: C211.1, R217.2
- new net: R223.1, U212.5 (ILIM)
- new net: C202.1, L201.1, U201.6 (OUT)
- new net: R204.1, U201.9 (ILM)
- new net: C208.1, U203.7 (DVDT)
- new net: R211.1, U203.9 (ILM)
- new net: R222.1, U211.5 (ILIM)
- new net: C219.1, U216.14 (NR)
- new net: C220.1, D203.1 (K), R230.1, U216.1 (OUT), U216.20 (OUT), U216.3 (SENSE/FB), U217.4 (VIN)
- new net: C214.1, U213.14 (NR)
- new net: Q201.1 (G), R234.1, R235.2
- new net: R219.1, U208.5 (ILIM)
- new net: R230.2, R231.1, U217.8 (OVLO/OVCSEL)
- new net: C216.1, U214.2 (dV/dT)
- new net: C213.1, L204.2, U213.15 (IN), U213.16 (IN)
- new net: R207.1, U202.9 (ILM)
- new net: L203.1, U206.6 (OUT)
- new net: R221.1, U210.5 (ILIM)
- new net: R226.1, U214.7 (ILM)
- new net: C221.1, U217.2 (dV/dT)
- new net: R232.2, R233.1, U218.3 (IN+)
- new net: F202.1, Q201.3 (D)
- new net: C207.1, U202.7 (DVDT)
- new net 3V3_Q6A: U215.6 (V+), U218.6 (V+)
- new net AUX12: F202.2
- new net AUX12_ND: Q202.3 (D), R235.1
- new net BONI13V8_EF: R232.1, U217.5 (OUT)
- new net BONI_REF: U218.4 (IN-), U218.5 (REF)
- new net DISP12: U202.6 (OUT)
- new net DISP12_OV: R205.2, R206.1, U202.2 (OVLO)
- new net EN_AUX12: Q202.1 (G)
- new net EN_BONI: U216.13 (EN), U217.3 (EN/UVLO)
- new net EN_DISP12: U202.1 (EN/UVLO)
- new net EN_HFP: U206.3 (EN)
- new net EN_LABPORT: U205.3 (EN)
- new net EN_LIME3V3: U204.1 (EN/UVLO)
- new net EN_LNA1: U209.3 (EN)
- new net EN_LNA2: U210.3 (EN)
- new net EN_LNA3: U211.3 (EN)
- new net EN_LNA4: U212.3 (EN)
- new net EN_LNB: U213.13 (EN), U214.3 (EN/UVLO)
- new net EN_RTLA: U207.3 (EN)
- new net EN_RTLB: U208.3 (EN)
- new net FAULT_HFP: U206.4 (~{FAULT})
- new net FAULT_LABPORT: U205.4 (~{FAULT})
- new net FAULT_LNA1: U209.4 (~{FAULT})
- new net FAULT_LNA2: U210.4 (~{FAULT})
- new net FAULT_LNA3: U211.4 (~{FAULT})
- new net FAULT_LNA4: U212.4 (~{FAULT})
- new net FAULT_RTLA: U207.4 (~{FAULT})
- new net FAULT_RTLB: U208.4 (~{FAULT})
- new net FLT_BONI: U217.6 (~{FLT})
- new net FLT_LIME3V3: U204.4 (~{FLT})
- new net FLT_LNB: U214.6 (~{FLT})
- new net GND: C201.2, C202.2, C203.2, C204.2, C205.2, C206.2, C207.2, C208.2, C209.2, C210.2, C211.2, C212.2, C213.2, C214.2, C215.2, C216.2, C217.2, C218.2, C219.2, C220.2, C221.2, D201.2 (A), D202.2 (A), D203.2 (A), JP201.1 (A), JP202.1 (A), JP203.1 (A), Q202.2 (S), R203.2, R204.2, R206.2, R207.2, R210.2, R211.2, R213.2, R214.2, R215.2, R216.2, R218.2, R219.2, R220.2, R221.2, R222.2, R223.2, R225.2, R226.2, R228.2, R229.2, R231.2, R233.2, U201.8 (GND), U202.8 (GND), U203.8 (GND), U204.8 (GND), U205.2 (GND), U206.2 (GND), U207.2 (GND), U208.2 (GND), U209.2 (GND), U210.2 (GND), U211.2 (GND), U212.2 (GND), U213.10 (0P4V), U213.11 (0P2V), U213.21 (EP), U213.5 (6P4V1), U213.6 (3P2V), U213.7 (GND), U214.1 (GND), U214.9 (GND), U215.2 (V-), U216.10 (0P4V), U216.21 (EP), U216.5 (6P4V1), U216.6 (3P2V), U216.7 (GND), U216.8 (1P6V), U216.9 (0P8V), U217.1 (GND), U217.9 (GND), U218.2 (V-)
- new net J21: C203.1, C204.1, D201.1 (K), L201.2
- new net J21_OV: R202.2, R203.1, U201.2 (OVLO)
- new net J21_UV: R201.2, R202.1, U201.1 (EN/UVLO)
- new net LAB5: U205.1 (IN), U206.1 (IN), U207.1 (IN), U208.1 (IN)
- new net LIME3V3: U204.6 (OUT)
- new net LIME_OV: R212.2, R213.1, U204.2 (OVLO)
- new net LNA4V5: U209.1 (IN), U210.1 (IN), U211.1 (IN), U212.1 (IN)
- new net LNA_CH1_EF: U209.6 (OUT)
- new net LNA_CH2_EF: U210.6 (OUT)
- new net LNA_CH3_EF: U211.6 (OUT)
- new net LNA_CH4_EF: U212.6 (OUT)
- new net LNB13V2_EF: R227.1, U214.5 (OUT)
- new net LNB_0P1V: JP203.2 (B), U213.12 (0P1V)
- new net LNB_0P8V: JP202.2 (B), U213.9 (0P8V)
- new net LNB_1P6V: JP201.2 (B), U213.8 (1P6V)
- new net LNB_REF: U215.4 (IN-), U215.5 (REF)
- new net PG_BONI: U218.1 (OUT)
- new net PG_LNB: U215.1 (OUT)
- new net SW: C212.1, C217.1, L204.1, L205.1
- new net SYS12: C205.1, F201.1, L202.1, Q201.2 (S), R234.2
- new net USBC_OV: R209.2, R210.1, U203.2 (OVLO)
- new net USBC_UV: R208.2, R209.1, U203.1 (EN/UVLO)
- new net VBUS_HFP: C210.1, L203.2, R217.1
- new net VBUS_IP2368: U203.6 (OUT)
- new net VBUS_LABPORT: U205.6 (OUT)
- new net VBUS_RTLA: U207.6 (OUT)
- new net VBUS_RTLB: U208.6 (OUT)
- new net VBUS_USBC: R208.1, U203.5 (IN)
- new net VCC_3V3_MKEY: R212.1, U204.5 (IN)
- no-connect marks 0 -> 15
Other:
- note added: "AUX12 → LAB BUS (лише BENCH) (STACK §5.1)"
- note added: "BONI13V8: SW → LC → TPS7A4701 (ANY-OUT 13.8 V) → TPS259630DDAR → (INA3221 0.2 Ω, E1) → bias-tee Boni, без PTC (STACK §5.1)"
- note added: "DISP12 → Wisecoco: SYS12 → LC → TPS259470ARPWR (ILIM 1.5 A, OVLO ≈13.5 V), EN від Pico GP16 (STACK §5.1)"
- note added: "J21 → Q6A: SYS12 → 4 A → TPS259470ARPWR (OVLO ≈13.5 V, ILIM ≈4 A) → pi-LC → SMBJ13A + 220 мкФ (STACK §5.1, §2.7)"
- note added: "LIME3V3: M.2 3.3 V Q6A → TPS259470ARPWR (4-й) → riser R44SF (STACK §5.1, §2.11.1, §8 (a))"
- note added: "LNB13V2: SW → LC → TPS7A4701 (ANY-OUT 13.2 V) → TPS259630DDAR → (INA3221 0.1 Ω, E1) → дросель (E4) → P4 (STACK §5.1, §2.7)"
- note added: "Rail-good TLV3011 → MCP #3 (STACK §2.7, §5.1)"
- note added: "USB-C корпусу → TPS259470ARPWR (OVLO ≈22 V, ILIM ≈3.5 A) → VBUS IP2368 (STACK §5.1 «Заряд», §2.7)"
- note added: "Канали зміщення LNA ch1-ch4 від LNA4V5 (2× LT3045 — аркуш E1) (STACK §5.1 LNA4V5, §1.1 C9)"
- note added: "Ключі VBUS RTL-A (H2) і RTL-B (J5 верхній) від LAB5 (STACK §5.1 LAB5, §5.2 карта USB)"
- note added: "Ключі VBUS від LAB5: LAB USB-A (H3), HF+ (H4) з демпфованим LC (STACK §5.1 LAB5, §5.2)"
- title: (none) -> E2 Живлення: захищені канали і LNB
