File: sat-receiver-audit/build/kicad/E2.kicad_sch (KiCad schematic)
At the start: 0 parts

Commit message: Complete SR-RX-v2.1 schematics and verification package
Replace five empty sheets with reviewed KiCad schematics and portable resources. Correct power, control, USB and RF interfaces; document hardware acceptance gates and unimplemented firmware/PCB work. Validate 754 components, 2189 connected contacts and 466 nets with zero ERC violations and two independent graph/netlist comparisons. Include PDF, SVG, BOM, reproducible tools and offline documentation.
Parts:
- added C201: 3.3nF 50V C0G C1608C0G1H332J080AA, Capacitor_SMD:C_0603_1608Metric, symbol sr_rx_v2_completed:C_C201
- added C202: 1uF 50V X7R C2012X7R1H105K125AB, Capacitor_SMD:C_0805_2012Metric, symbol sr_rx_v2_completed:C_C202
- added C203: 1uF 50V X7R C2012X7R1H105K125AB, Capacitor_SMD:C_0805_2012Metric, symbol sr_rx_v2_completed:C_C203
- added C204: 10uF 50V X7R C3225X7R1H106K250AC, Capacitor_SMD:C_1210_3225Metric, symbol sr_rx_v2_completed:C_C204
- added C205: 10uF 50V X7R C3225X7R1H106K250AC, Capacitor_SMD:C_1210_3225Metric, symbol sr_rx_v2_completed:C_C205
- added C206: 47uF 50V EEUFR1H470, symbol sr_rx_v2_completed:C_C206
- added C207: 220uF/25V UHE1E221MPD, symbol sr_rx_v2_completed:C_C207
- added C208: 10uF 50V X7R C3225X7R1H106K250AC, Capacitor_SMD:C_1210_3225Metric, symbol sr_rx_v2_completed:C_C208
- added C209: 10uF 50V X7R C3225X7R1H106K250AC, Capacitor_SMD:C_1210_3225Metric, symbol sr_rx_v2_completed:C_C209
- added C210: 47uF 50V EEUFR1H470, symbol sr_rx_v2_completed:C_C210
- added C211: 3.3nF 50V C0G C1608C0G1H332J080AA, Capacitor_SMD:C_0603_1608Metric, symbol sr_rx_v2_completed:C_C211
- added C212: 1uF 50V X7R C2012X7R1H105K125AB, Capacitor_SMD:C_0805_2012Metric, symbol sr_rx_v2_completed:C_C212
- added C213: 1uF 50V X7R C2012X7R1H105K125AB, Capacitor_SMD:C_0805_2012Metric, symbol sr_rx_v2_completed:C_C213
- added C214: 3.3nF 50V C0G C1608C0G1H332J080AA, Capacitor_SMD:C_0603_1608Metric, symbol sr_rx_v2_completed:C_C214
- added C215: 1uF 50V X7R C2012X7R1H105K125AB, Capacitor_SMD:C_0805_2012Metric, symbol sr_rx_v2_completed:C_C215
- added C216: 1uF 50V X7R C2012X7R1H105K125AB, Capacitor_SMD:C_0805_2012Metric, symbol sr_rx_v2_completed:C_C216
- added C217: 10uF 50V X7R C3225X7R1H106K250AC, Capacitor_SMD:C_1210_3225Metric, symbol sr_rx_v2_completed:C_C217
- added C218: 10uF 50V X7R C3225X7R1H106K250AC, Capacitor_SMD:C_1210_3225Metric, symbol sr_rx_v2_completed:C_C218
- added C219: 47uF 50V EEUFR1H470, symbol sr_rx_v2_completed:C_C219
- added C220: 10uF 50V X7R C3225X7R1H106K250AC, Capacitor_SMD:C_1210_3225Metric, symbol sr_rx_v2_completed:C_C220
- added D201: SMBJ13A-E3/52, symbol sr_rx_v2_completed:C_D201
- added F201: Littelfuse0297004.WXNV 4A, symbol sr_rx_v2_completed:C_F201
- added F202: MF-MSMF075/24-2 0.75A, symbol sr_rx_v2_completed:C_F202
- added L201: 1uH XAL5030-102MEC, symbol sr_rx_v2_completed:C_L201
- added L202: 1uH XAL5030-102MEC, symbol sr_rx_v2_completed:C_L202
- added L203: 1uH XAL5030-102MEC, symbol sr_rx_v2_completed:C_L203
- added L204: 1uH XAL5030-102MEC, symbol sr_rx_v2_completed:C_L204
- added Q201: AO3407A, symbol sr_rx_v2_completed:C_Q201
- added Q202: 2N7002, symbol sr_rx_v2_completed:C_Q202
- added R201: 100k 1%, symbol sr_rx_v2_completed:C_R201
- added R202: 33.2k 1%, symbol sr_rx_v2_completed:C_R202
- added R203: 825R 1%, symbol sr_rx_v2_completed:C_R203
- added R204: 102k 0.1%, symbol sr_rx_v2_completed:C_R204
- added R205: 10.0k 0.1%, symbol sr_rx_v2_completed:C_R205
- added R206: 10.0k 1%, symbol sr_rx_v2_completed:C_R206
- added R207: 0.22R 1% 0.25W, symbol sr_rx_v2_completed:C_R207
- added R208: 0.22R 1% 0.25W, symbol sr_rx_v2_completed:C_R208
- added R209: 1.96k 1%, symbol sr_rx_v2_completed:C_R209
- added R210: 102k 0.1%, symbol sr_rx_v2_completed:C_R210
- added R211: 10.0k 0.1%, symbol sr_rx_v2_completed:C_R211
- added R212: 10.0k 1%, symbol sr_rx_v2_completed:C_R212
- added R213: 100k 1%, symbol sr_rx_v2_completed:C_R213
- added R214: 1.65k 1%, symbol sr_rx_v2_completed:C_R214
- added R215: 19.6k 0.1%, symbol sr_rx_v2_completed:C_R215
- added R216: 10.0k 0.1%, symbol sr_rx_v2_completed:C_R216
- added R218: 100k 1%, symbol sr_rx_v2_completed:C_R218
- added R219: 0.22R 1% 0.25W, symbol sr_rx_v2_completed:C_R219
- added R220: 100k 1%, symbol sr_rx_v2_completed:C_R220
- added R221: 10.0k 1%, symbol sr_rx_v2_completed:C_R221
- added R222: 10.0k 1%, symbol sr_rx_v2_completed:C_R222
- added TP201: J21, symbol sr_rx_v2_completed:C_TP201
- added TP202: DISP12, symbol sr_rx_v2_completed:C_TP202
- added TP203: LIME3V3, symbol sr_rx_v2_completed:C_TP203
- added TP213: E2_FAULT_J21, symbol sr_rx_v2_completed:C_TP213
- added TP214: E2_FAULT_DISP, symbol sr_rx_v2_completed:C_TP214
- added U201: TPS259470ARPWR, symbol sr_rx_v2_completed:C_U201
- added U202: TPS259470ARPWR, symbol sr_rx_v2_completed:C_U202
- added U203: TPS259470ARPWR, symbol sr_rx_v2_completed:C_U203
Connections:
- new net 3V3_Q6A: R206.2, R212.2
- new net AUX12: L204.2
- new net DISP12: C213.1, TP202.1 (TP), U202.6 (OUT)
- new net E2_AUX_GATE: Q201.1 (G), R221.2, R222.1
- new net E2_AUX_GSINK: Q202.3 (D), R222.2
- new net E2_AUX_PTC: C220.1, F202.2, L204.1
- new net E2_AUX_SWITCHED: F202.1, Q201.3 (D)
- new net E2_DISP_IN: C209.1, C212.1, L202.2, R208.1, R210.1, U202.5 (IN)
- new net E2_DISP_IN_DAMP: C210.1 (+), R208.2
- new net E2_FAULT_DISP: R212.1, TP214.1 (TP), U202.4 (FLT)
- new net E2_FAULT_J21: R206.1, TP213.1 (TP), U201.4 (FLT)
- new net E2_J21_EF: C203.1, C204.1, L201.1, U201.6 (OUT)
- new net E2_J21_EN: R201.2, R202.1, U201.1 (EN/UVLO)
- new net E2_J21_FUSED: C202.1, F201.2, R201.1, R204.1, U201.5 (IN)
- new net E2_LIME_EF: C216.1, C217.1, L203.1, U203.6 (OUT)
- new net E2_U201_DVDT: C201.1, U201.7 (DVDT)
- new net E2_U201_ILM: R203.1, U201.9 (ILM)
- new net E2_U201_OV: R204.2, R205.1, U201.2 (OVLO)
- new net E2_U202_DVDT: C211.1, U202.7 (DVDT)
- new net E2_U202_ILM: R209.1, U202.9 (ILM)
- new net E2_U202_OV: R210.2, R211.1, U202.2 (OVLO)
- new net E2_U203_DVDT: C214.1, U203.7 (DVDT)
- new net E2_U203_ILM: R214.1, U203.9 (ILM)
- new net E2_U203_OV: R215.2, R216.1, U203.2 (OVLO)
- new net EN_AUX12: Q202.1 (G), R220.1
- new net EN_LIME3V3: R218.1, U203.1 (EN/UVLO)
- new net FLT_LIME3V3: U203.4 (FLT)
- new net GND: C201.2, C202.2, C203.2, C204.2, C205.2, C206.2 (-), C207.2, C208.2, C209.2, C210.2 (-), C211.2, C212.2, C213.2, C214.2, C215.2, C216.2, C217.2, C218.2, C219.2 (-), C220.2, D201.A, Q202.2 (S), R202.2, R203.2, R205.2, R209.2, R211.2, R213.2, R214.2, R216.2, R218.2, R220.2, U201.8 (GND), U202.8 (GND), U203.8 (GND)
- new net J21: C205.1, C207.1, D201.K, L201.2, R207.1, TP201.1 (TP)
- new net J21_DAMP: C206.1 (+), R207.2
- new net LIME3V3: C218.1, L203.2, R219.1, TP203.1 (TP)
- new net LIME3V3_DAMP: C219.1 (+), R219.2
- new net PICO_DISP_EN: R213.1, U202.1 (EN/UVLO)
- new net SYS12: C208.1, F201.1, L202.1, Q201.2 (S), R221.1
- new net VCC_3V3_MKEY: C215.1, R215.1, U203.5 (IN)
- no-connect marks 0 -> 6
Other:
- note added: "AUX12: верхній ключ і PTC"
- note added: "E2 - Захищені рейки, LNA і моніторинг струму (1/5)"
- note added: "J21: захищене живлення 12 V"
- note added: "Lime M.2: комутована шина 3.3 V"
- note added: "Дисплей: захищене живлення 12 V"
- note added: "Мережі з однаковими глобальними мітками електрично з'єднані на всіх аркушах. Фізичні/функціональні контакти: див. design/ і OPEN_ITEMS.md."
- company: (none) -> SR-RX-v2
- title: (none) -> E2 - Захищені рейки, LNA і моніторинг струму (1/5)
