File: sat-receiver-audit/build/kicad/E2.kicad_sch (KiCad schematic)
At the start: 94 parts, among them Q201 AO3407A, Q202 2N7002, U201 TPS259470ARPWR, U202 TPS259470ARPWR, U203 TPS259470ARPWR, U206 TPS2553DBVR-1, U207 TPS2553DBVR-1, U217 TLV3011BIDBVR, U218 TLV3011BIDBVR

Commit message: Stage 2 integration: CAD and DC_CORE re-freeze from CI run 40094234222; bound-count test and PCB hash lists follow
Co-Authored-By: Claude Opus 5.5 <noreply@anthropic.com>
Parts:
- removed C236: 1uF 50V X7R C2012X7R1H105K125AB, Capacitor_SMD:C_0805_2012Metric, symbol sr_rx_v2_completed:C_C236
- removed C237: 1uF 50V X7R C2012X7R1H105K125AB, Capacitor_SMD:C_0805_2012Metric, symbol sr_rx_v2_completed:C_C237
- removed C238: 1uF 50V X7R C2012X7R1H105K125AB, Capacitor_SMD:C_0805_2012Metric, symbol sr_rx_v2_completed:C_C238
- removed C239: 47uF 50V EEUFR1H470, symbol sr_rx_v2_completed:C_C239
- removed L207: 1uH XAL5030-102MEC, symbol sr_rx_v2_completed:C_L207
- removed R233: 88.7k 1%, symbol sr_rx_v2_completed:C_R233
- removed R234: 100k 1%, symbol sr_rx_v2_completed:C_R234
- removed R236: 0.200R 0.1% 0.25W Kelvin, symbol sr_rx_v2_completed:C_R236
- removed R237: 0.22R 1% 0.25W, symbol sr_rx_v2_completed:C_R237
- removed TP207: BIAS_CH2, symbol sr_rx_v2_completed:C_TP207
- removed U207: TPS2553DBVR-1, symbol sr_rx_v2_completed:C_U207
- added C244: 1uF 50V X7R C2012X7R1H105K125AB, Capacitor_SMD:C_0805_2012Metric, symbol sr_rx_v2_completed:C_C244
- added C245: 1uF 50V X7R C2012X7R1H105K125AB, Capacitor_SMD:C_0805_2012Metric, symbol sr_rx_v2_completed:C_C245
- added C246: 1uF 50V X7R C2012X7R1H105K125AB, Capacitor_SMD:C_0805_2012Metric, symbol sr_rx_v2_completed:C_C246
- added C247: 47uF 50V EEUFR1H470, symbol sr_rx_v2_completed:C_C247
- added L209: 1uH XAL5030-102MEC, symbol sr_rx_v2_completed:C_L209
- added R243: 162k 1%, symbol sr_rx_v2_completed:C_R243
- added R244: 100k 1%, symbol sr_rx_v2_completed:C_R244
- added R246: 0.200R 0.1% 0.25W Kelvin, symbol sr_rx_v2_completed:C_R246
- added R247: 0.22R 1% 0.25W, symbol sr_rx_v2_completed:C_R247
- added TP209: BIAS_CH4, symbol sr_rx_v2_completed:C_TP209
- added U209: TPS2553DBVR-1, symbol sr_rx_v2_completed:C_U209
- R202: value 33.2k 1% -> 13.0k 1% 100ppm; footprint (none) -> Resistor_SMD:R_0603_1608Metric
Connections:
- net BIAS_CH4: now also C246.1, L209.2, R247.1, TP209.1 (TP)
- net GND: now also C244.2, C245.2, C246.2, C247.2 (-), R243.2, R244.2, U209.2 (GND)
- net LNA4V5: now also C244.1, U209.1 (IN)
- new net BIAS_CH4_DAMP: C247.1 (+), R247.2
- new net E2_LNA4_SHUNT: C245.1, L209.1, R246.2
- new net E2_LNA4_SW: R246.1, U209.6 (OUT)
- new net E2_U209_ILIM: R243.1, U209.5 (ILIM)
- new net EN_LNA4: R244.1, U209.3 (EN)
- new net FAULT_LNA4: U209.4 (FAULT)
Other:
- note added: "E2 - Захищені рейки, LNA і моніторинг струму (1/5)"
- note added: "LNA: канал 4"
- note added: "Відсутність фантомного живлення Q6A, вимкнення дисплея та фізична правильність кінцевих кабелів потребують перевірки з реальним обладнанням. Ворота (стенд): За активної LAB5 і вимкненої Q6A: 3V3_Q6A та upstream VBUS близько 0V, PICO_DISP_EN низький. Продзвонити розрізаний VBUS, ключовані роз’єми E3/E5 та сигнал PWR_ON_KEY. UVLO J21 (v2.1, R202 13.0k): джерело з обмеженням струму на E2_J21_FUSED, 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"
- note removed: "E2 - Захищені рейки, LNA і моніторинг струму (1/4)"
- note removed: "LNA: канал 2"
- note removed: "Відсутність фантомного живлення Q6A, вимкнення дисплея та фізична правильність кінцевих кабелів потребують перевірки з реальним обладнанням. Ворота (стенд): За активної LAB5 і вимкненої Q6A: 3V3_Q6A та upstream VBUS близько 0V, PICO_DISP_EN низький. Продзвонити розрізаний VBUS, ключовані роз’єми E3/E5 та сигнал PWR_ON_KEY."
- note removed: "Позначення фізичних джерел живлення (ERC)"
- title: E2 - Захищені рейки, LNA і моніторинг струму (1/4) -> E2 - Захищені рейки, LNA і моніторинг струму (1/5)
- moved on the sheet: C201, C202, C203, C204, C205, C206, C207, C208, C209, C210, C211, C212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

Commit message: GENERATED: CAD, documents, verification reports, DC_CORE re-freeze and module-lab inventory for f3f57e8
Applied unchanged from the cad-regenerated artifact of CI run 40109759054
(workflow_dispatch, refreeze_pcb=true, KiCad 10.0.7): schematics, SVG, PDF,
netlist, OPEN_ITEMS.md, COMPLETION.md, verification/{electrical-invariants,
independent-netlist-review,netlist,pcb-review,pcb-prototype-review,
pdf-export,validation}, pcb/generated and the re-frozen DC_CORE starter and
routed prototype with their pinned hashes. Inputs: the stage 3A merge,
design/E2.json (PICO-2 text) and STACK.md (2.7 row).

deployment/module_lab/inventory.json: source_snapshots only, from
deployment/module_lab/refresh_inventory.py (E2.json and STACK.md bytes).

Co-Authored-By: Claude Opus 5.5 <noreply@anthropic.com>
Parts:
- removed C244: 1uF 50V X7R C2012X7R1H105K125AB, Capacitor_SMD:C_0805_2012Metric, symbol sr_rx_v2_completed:C_C244
- removed C245: 1uF 50V X7R C2012X7R1H105K125AB, Capacitor_SMD:C_0805_2012Metric, symbol sr_rx_v2_completed:C_C245
- removed C246: 1uF 50V X7R C2012X7R1H105K125AB, Capacitor_SMD:C_0805_2012Metric, symbol sr_rx_v2_completed:C_C246
- removed C247: 47uF 50V EEUFR1H470, symbol sr_rx_v2_completed:C_C247
- removed L209: 1uH XAL5030-102MEC, symbol sr_rx_v2_completed:C_L209
- removed R243: 162k 1%, symbol sr_rx_v2_completed:C_R243
- removed R244: 100k 1%, symbol sr_rx_v2_completed:C_R244
- removed R246: 0.200R 0.1% 0.25W Kelvin, symbol sr_rx_v2_completed:C_R246
- removed R247: 0.22R 1% 0.25W, symbol sr_rx_v2_completed:C_R247
- removed TP209: BIAS_CH4, symbol sr_rx_v2_completed:C_TP209
- removed U209: TPS2553DBVR-1, symbol sr_rx_v2_completed:C_U209
- added C286: 10nF 50V C0G C1608C0G1H103J080AA, Capacitor_SMD:C_0603_1608Metric, symbol sr_rx_v2_completed:C_C286
- added C287: 100nF 50V X7R C1608X7R1H104K080AA, Capacitor_SMD:C_0603_1608Metric, symbol sr_rx_v2_completed:C_C287
- added R286: 73.2k 0.1%, symbol sr_rx_v2_completed:C_R286
- added R287: 10.0k 0.1%, symbol sr_rx_v2_completed:C_R287
- added U219: TLV3011BIDBVR, symbol sr_rx_v2_completed:C_U219
Connections:
- net 3V3_Q6A: now also C287.1, U219.6 (V+)
- net AUX12: now also R286.1
- net GND: now also C286.2, C287.2, R287.2, U219.2 (V-)
- new net E2_U219_REF: U219.4 (IN-), U219.5 (REF)
- new net E2_U219_SENSE: C286.1, R286.2, R287.1, U219.3 (IN+)
- new net PTC_AUX: U219.1 (OUT)
Other:
- note added: "AUX12: контроль напруги після PTC"
- note removed: "LNA: канал 4"
- moved on the sheet: C201, C202, C203, C204, C205, C206, C207, C208, C209, C210, C211, C212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
