File: sat-receiver-audit/build/kicad/E3.kicad_sch (KiCad schematic)
At the start: 0 parts

Commit message: Complete SR-RX-v2.1 schematics and verification package
Replace five empty sheets with reviewed KiCad schematics and portable resources. Correct power, control, USB and RF interfaces; document hardware acceptance gates and unimplemented firmware/PCB work. Validate 754 components, 2189 connected contacts and 466 nets with zero ERC violations and two independent graph/netlist comparisons. Include PDF, SVG, BOM, reproducible tools and offline documentation.
Parts:
- added BT301: CR2032 3V primary, symbol sr_rx_v2_completed:C_BT301
- added C301: 100n 16V, symbol sr_rx_v2_completed:C_C301
- added C302: 10u 10V, symbol sr_rx_v2_completed:C_C302
- added C303: 100n 16V, symbol sr_rx_v2_completed:C_C303
- added C304: 10u 10V, symbol sr_rx_v2_completed:C_C304
- added C305: 100n 16V, symbol sr_rx_v2_completed:C_C305
- added C306: 10u 10V, symbol sr_rx_v2_completed:C_C306
- added C307: 10u 10V, symbol sr_rx_v2_completed:C_C307
- added C308: 100n 16V, symbol sr_rx_v2_completed:C_C308
- added D301: SS14, Diode_SMD:D_SMA, symbol sr_rx_v2_completed:C_D301
- added J301: Q6A J20 2x20 3.3V GPIO, symbol sr_rx_v2_completed:C_J301
- added J302: Power-board control harness DESIGN, symbol sr_rx_v2_completed:C_J302
- added J303: Q6A J11 RTC battery 1.25mm, symbol sr_rx_v2_completed:C_J303
- added Q301: 2N7002, Package_TO_SOT_SMD:SOT-23, symbol sr_rx_v2_completed:C_Q301
- added R301: 10k, symbol sr_rx_v2_completed:C_R301
- added R302: 10k, symbol sr_rx_v2_completed:C_R302
- added R303: 10k DNP, symbol sr_rx_v2_completed:C_R303
- added R304: 10k DNP, symbol sr_rx_v2_completed:C_R304
- added R305: 10k, symbol sr_rx_v2_completed:C_R305
- added R306: 10k, symbol sr_rx_v2_completed:C_R306
- added R307: 10k, symbol sr_rx_v2_completed:C_R307
- added R308: 10k, symbol sr_rx_v2_completed:C_R308
- added R309: 10k, symbol sr_rx_v2_completed:C_R309
- added R310: 10k, symbol sr_rx_v2_completed:C_R310
- added R311: 10k, symbol sr_rx_v2_completed:C_R311
- added R312: 10k, symbol sr_rx_v2_completed:C_R312
- added R313: 10k, symbol sr_rx_v2_completed:C_R313
- added R314: 10k, symbol sr_rx_v2_completed:C_R314
- added R315: 10k, symbol sr_rx_v2_completed:C_R315
- added R316: 10k, symbol sr_rx_v2_completed:C_R316
- added R317: 10k, symbol sr_rx_v2_completed:C_R317
- added R318: 10k, symbol sr_rx_v2_completed:C_R318
- added R319: 10k, symbol sr_rx_v2_completed:C_R319
- added R320: 10k, symbol sr_rx_v2_completed:C_R320
- added R321: 10k, symbol sr_rx_v2_completed:C_R321
- added R322: 10k, symbol sr_rx_v2_completed:C_R322
- added R323: 10k, symbol sr_rx_v2_completed:C_R323
- added R324: 10k, symbol sr_rx_v2_completed:C_R324
- added R325: 10k, symbol sr_rx_v2_completed:C_R325
- added R326: 100k, symbol sr_rx_v2_completed:C_R326
- added R392: 10k, symbol sr_rx_v2_completed:C_R392
- added U301: MCP23017-E/SO #1 0x20, Package_SO:SOIC-28W_7.5x17.9mm_P1.27mm, symbol sr_rx_v2_completed:C_U301
- added U302: MCP23017-E/SO #3 0x22, Package_SO:SOIC-28W_7.5x17.9mm_P1.27mm, symbol sr_rx_v2_completed:C_U302
- added U303: MCP23017-E/SO #4 0x23, Package_SO:SOIC-28W_7.5x17.9mm_P1.27mm, symbol sr_rx_v2_completed:C_U303
- added U304: Waveshare LC76G GNSS 24370, symbol sr_rx_v2_completed:C_U304
- added U305: Raspberry Pi Pico SC0915, symbol sr_rx_v2_completed:C_U305
Connections:
- new net 3V3_Q6A: C301.1, C302.1, C303.1, C304.1, C305.1, C306.1, J301.1 (3V3), J301.17 (3V3), J302.1 (3V3_Q6A), R301.2, R302.2, R303.2, R304.2, R305.2, R306.2, R307.2, R308.2, R309.2, R310.2, R311.2, R312.2, R313.2, R314.2, R315.2, R316.2, R317.2, R318.2, R319.2, R320.2, R321.2, R322.2, R323.2, R324.2, R325.2, R392.2, U301.9 (VDD), U302.16 (A1), U302.9 (VDD), U303.15 (A0), U303.16 (A1), U303.9 (VDD)
- new net CHG_INHIBIT: U303.5 (GPB4)
- new net DCS_HF: R319.1, U302.5 (GPB4)
- new net DCS_LBAND: R318.1, U302.4 (GPB3)
- new net DCS_UHF: R317.1, U302.3 (GPB2)
- new net E1_BAT_ADC: U305.32 (GP27)
- new net E3_ADC3V0: U305.35 (ADC_VREF)
- new net E3_BLOWER_EN: U305.25 (GP19)
- new net E3_BUTTON_SENSE: U305.15 (GP11)
- new net E3_CASE_TEMP: U305.34 (GP28)
- new net E3_ENC1_A: U305.4 (GP2)
- new net E3_ENC1_B: U305.5 (GP3)
- new net E3_ENC2_A: U305.9 (GP6)
- new net E3_ENC2_B: U305.10 (GP7)
- new net E3_FAN_EN: U305.24 (GP18)
- new net E3_FAN_TACH: U305.29 (GP22)
- new net E3_GNSS_PPS: J301.7 (GPIO96), U304.P1.5 (1PPS)
- new net E3_GNSS_RESET_GATE: Q301.1 (G), R326.1, U303.22 (GPA1)
- new net E3_GNSS_RESET_N: Q301.3 (D), U304.P1.6 (RESET_N)
- new net E3_HMI_INT: U305.14 (GP10)
- new net E3_HMI_SCL: U305.7 (GP5)
- new net E3_HMI_SDA: U305.6 (GP4)
- new net E3_LED_DRIVE: U305.27 (GP21)
- new net E3_MCP_RESET_ASSERT: U305.22 (GP17)
- new net E3_MCP_RESET_N: R305.1, R306.1, R307.1, U301.18 (RESET_N), U302.18 (RESET_N), U303.18 (RESET_N)
- new net E3_PANEL_TEMP: U305.31 (GP26)
- new net E3_PICO3V3: C308.1, U305.36 (3V3_OUT)
- new net E3_PICO_RUN: J301.38 (GPIO98_RUN), U305.30 (RUN)
- new net E3_PICO_SWCLK: J301.12 (GPIO97_SWCLK), U305.SWCLK
- new net E3_PICO_SWDIO: J301.35 (GPIO100_SWDIO), U305.SWDIO
- new net E3_PICO_VSYS: C307.1, D301.1 (K), U305.39 (VSYS)
- new net E3_PIEZO_DRIVE: U305.26 (GP20)
- new net E3_Q6A_KEY_GATE: U305.16 (GP12)
- new net E3_Q6A_ON_SENSE: U305.19 (GP14)
- new net E3_RTC_BAT: BT301.+ (POS), J303.2 (CR2032_PLUS)
- new net EN_AUX12: U301.22 (GPA1)
- new net EN_BONI: U301.2 (GPB1)
- new net EN_HFP: U301.25 (GPA4)
- new net EN_LABPORT: U301.21 (GPA0)
- new net EN_LIME3V3: U303.21 (GPA0)
- new net EN_LNA1: U301.26 (GPA5)
- new net EN_LNA2: U301.27 (GPA6)
- new net EN_LNA3: U301.28 (GPA7)
- new net EN_LNA4: U302.28 (GPA7)
- new net EN_LNB: U301.1 (GPB0)
- new net EN_RTLA: U301.23 (GPA2)
- new net EN_RTLB: U301.24 (GPA3)
- new net EN_SB_LNA: U303.25 (GPA4)
- new net EN_T7: U302.8 (GPB7)
- new net FAULT_HFP: R323.1, U303.2 (GPB1)
- new net FAULT_LABPORT: R308.1, U302.21 (GPA0)
- new net FAULT_LNA1: R309.1, U302.22 (GPA1)
- new net FAULT_LNA2: R310.1, U302.23 (GPA2)
- new net FAULT_LNA3: R311.1, U302.24 (GPA3)
- new net FAULT_LNA4: R312.1, U302.25 (GPA4)
- new net FAULT_RTLA: R324.1, U303.3 (GPB2)
- new net FAULT_RTLB: R322.1, U303.1 (GPB0)
- new net FLT_BONI: R314.1, U302.27 (GPA6)
- new net FLT_LIME3V3: R325.1, U303.4 (GPB3)
- new net FLT_LNB: R313.1, U302.26 (GPA5)
- new net FLT_SB_LNA: R392.1, U303.26 (GPA5)
- new net GND: BT301.- (NEG), C301.2, C302.2, C303.2, C304.2, C305.2, C306.2, C307.2, C308.2, J301.14 (GND), J301.20 (GND), J301.25 (GND), J301.30 (GND), J301.34 (GND), J301.39 (GND), J301.6 (GND), J301.9 (GND), J302.2 (GND), J303.1 (GND), Q301.2 (S), R326.2, U301.10 (VSS), U301.15 (A0), U301.16 (A1), U301.17 (A2), U302.10 (VSS), U302.15 (A0), U302.17 (A2), U303.10 (VSS), U303.17 (A2), U304.GPS1.1 (GND), U304.GPS1.3 (GND), U304.GPS1.4 (GND), U304.P1.2 (GND), U305.13 (GND), U305.18 (GND), U305.23 (GND), U305.28 (GND), U305.3 (GND), U305.33 (GND), U305.38 (GND), U305.8 (GND), U305.SWD_GND
- new net GNSS_ANT: U304.GPS1.2 (ANT)
- new net I2C0_SCL: J301.15 (GPIO1_I2C0_SCL)
- new net I2C0_SDA: J301.13 (GPIO0_I2C0_SDA)
- new net I2C2_SCL: J301.28 (GPIO9_I2C2_SCL), J302.4 (SCL), R304.1, U301.12 (SCL), U302.12 (SCL), U303.12 (SCL)
- new net I2C2_SDA: J301.27 (GPIO8_I2C2_SDA), J302.3 (SDA), R303.1, U301.13 (SDA), U302.13 (SDA), U303.13 (SDA)
- new net IMU_RX: U305.11 (GP8)
- new net IMU_TX: U305.12 (GP9)
- new net INA228_ALERT: J301.3 (GPIO24), R301.1
- new net K1_ON: U301.3 (GPB2)
- new net K2_ON: U301.4 (GPB3)
- new net LAB5: D301.2 (A)
- new net MCP_INT: J301.5 (GPIO25), J302.5 (INT), R302.1, U302.19 (INTB), U302.20 (INTA), U303.19 (INTB), U303.20 (INTA)
- new net OVP_LNB_N: U303.6 (GPB5)
- new net PG_BONI: R316.1, U302.2 (GPB1)
- new net PG_LNB: R315.1, U302.1 (GPB0)
- new net PICO_DISP_EN: U305.21 (GP16)
- new net PICO_OFF: U305.17 (GP13)
- new net PTC_AUX: R320.1, U302.6 (GPB5)
- new net SAFE_BOOT: J301.40 (GPIO99_SAFE_BOOT), U305.20 (GP15)
- new net SLED_DET: R321.1, U302.7 (GPB6)
- new net SW_LIME_A: U303.23 (GPA2)
- new net SW_LIME_B: U303.24 (GPA3)
- new net SW_RTLA_A: U301.5 (GPB4)
- new net SW_RTLA_B: U301.6 (GPB5)
- new net SW_RTLB_A: U301.7 (GPB6)
- new net SW_RTLB_B: U301.8 (GPB7)
- new net UART5_RX: J301.10 (GPIO23_UART5_RX)
- new net UART5_TX: J301.8 (GPIO22_UART5_TX)
- new net UART6_RX: J301.18 (GPIO27_UART6_RX), U304.P1.3 (TXD)
- new net UART6_TX: J301.16 (GPIO26_UART6_TX), U304.P1.4 (RXD)
- new net UART7_RX: J301.29 (GPIO31_UART7_RX), U305.1 (GP0)
- new net UART7_TX: J301.32 (GPIO30_UART7_TX), U305.2 (GP1)
- new net VCC_5V_PERI: J301.2 (5V), J301.4 (5V), U304.P1.1 (VCC)
- no-connect marks 0 -> 27
Other:
- note added: "E3 - Керування, Pico HMI, GPIO, GNSS і IMU (1/3)"
- note added: "GNSS"
- note added: "MCP23017 control"
- note added: "Pico HMI"
- note added: "Q6A header"
- note added: "RTC"
- note added: "Мережі з однаковими глобальними мітками електрично з'єднані на всіх аркушах. Фізичні/функціональні контакти: див. design/ і OPEN_ITEMS.md."
- company: (none) -> SR-RX-v2
- title: (none) -> E3 - Керування, Pico HMI, GPIO, GNSS і IMU (1/3)
