File: sat-receiver-audit/build/kicad/E3.kicad_sch (KiCad schematic)
At the start: 46 parts, among them J301 Q6A J20 2x20 3.3V GPIO, J302 Power-board control harness D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, J303 Q6A J11 RTC battery 1.25mm, Q301 2N7002, U301 MCP23017-E/SO #1 0x20, U302 MCP23017-E/SO #3 0x22, U303 MCP23017-E/SO #4 0x23, U304 Waveshare LC76G GNSS 24370, U305 Raspberry Pi Pico SC0915

Commit message: SR-RX-v2.1: review fixes on the Codex branch, readable schematic, one-file bundle
Independent review of the Codex branch (schematic vs STACK.md, hard rules,
security, tests) found no blockers; this commit applies its findings:

- rules in code: Cospas-Sarsat 406.0-406.1 MHz added to the no-data mask;
  Q6A Wi-Fi/BT off in the field/QUIET root (modprobe blacklist, udev
  authorized=0 on FE1.1s port 4, rfkill) with self-checks; device denylist
  completed per STACK (gr-gsm, gr-iridium, kalibrate, pager/trunking decoders,
  TX-capable tools); W1-2 WIFI_PWR_EN as blocking open item E5-10
- STACK.md is the source of truth again; v2.1 changes recorded in it; the
  "historical" marker kept only on ISDT/raw-balance rows; gender-neutral wording
- schematic data: open values shown as TBD with start values and notes, U503
  TPS2553DBVR-1, Lime X2/X4 RX mapping TBD, 37 open items drawn on the sheets
- schematic readability: wired groups, junctions, GND symbols, standard
  transistor/diode symbols; netlist unchanged (603 nets identical)
- tooling: reproducible run_checks (no timestamps or machine paths), pinned
  dependencies, bundle excludes cache folders, clean-checkout bundle check
- regenerated: KiCad export (14 pages), netlist/ERC, module lab, PCB inputs,
  readiness contract, acceptance hashes, SR-RX-v2-ves-proekt.html

Checks: ERC 0 errors/0 warnings, netlist comparison PASS, 432 tests (431
passed, 1 skipped), deployment tests OK, bundle check PASS on a clean checkout.

History note: earlier versions of the generated SR-RX-v2-ves-proekt.html and
handoff/handoff-bundle.zip were removed from history; only the final versions
are kept. The Codex merge commit is now attributed to Codex.

Co-Authored-By: Claude Opus 5.5 <noreply@anthropic.com>
Claude-Session: https://claude.ai/code/session_01W9CKpimWpgkUmrDQQMiKtF
Parts:
- removed C307: 10u 10V, symbol sr_rx_v2_completed:C_C307
- removed C308: 100n 16V, symbol sr_rx_v2_completed:C_C308
- removed D301: SS14, Diode_SMD:D_SMA, symbol sr_rx_v2_completed:C_D301
- removed J301: Q6A J20 2x20 3.3V GPIO, symbol sr_rx_v2_completed:C_J301
- removed J302: Power-board control harness DESIGN, symbol sr_rx_v2_completed:C_J302
- removed Q301: 2N7002, Package_TO_SOT_SMD:SOT-23, symbol sr_rx_v2_completed:C_Q301
- removed R301: 10k, symbol sr_rx_v2_completed:C_R301
- removed R302: 10k, symbol sr_rx_v2_completed:C_R302
- removed R303: 10k DNP, symbol sr_rx_v2_completed:C_R303
- removed R304: 10k DNP, symbol sr_rx_v2_completed:C_R304
- removed R326: 100k, symbol sr_rx_v2_completed:C_R326
- removed U304: Waveshare LC76G GNSS 24370, symbol sr_rx_v2_completed:C_U304
- removed U305: Raspberry Pi Pico SC0915, symbol sr_rx_v2_completed:C_U305
- added C310: 100n 16V, symbol sr_rx_v2_completed:C_C310
- added C311: 100n 16V, symbol sr_rx_v2_completed:C_C311
- added C312: 100n 16V, symbol sr_rx_v2_completed:C_C312
- added C313: 1u 10V, symbol sr_rx_v2_completed:C_C313
- added C340: 10u 10V, symbol sr_rx_v2_completed:C_C340
- added C341: 100n 16V, symbol sr_rx_v2_completed:C_C341
- added Q306: 2N7002,215, Package_TO_SOT_SMD:SOT-23, symbol sr_rx_v2_completed:C_Q306
- added R332: 10k 1%, symbol sr_rx_v2_completed:C_R332
- added R333: 10k 1%, symbol sr_rx_v2_completed:C_R333
- added R334: 10k, symbol sr_rx_v2_completed:C_R334
- added R335: 2.2k, symbol sr_rx_v2_completed:C_R335
- added R336: 100, symbol sr_rx_v2_completed:C_R336
- added R337: 2.2k, symbol sr_rx_v2_completed:C_R337
- added R338: 100, symbol sr_rx_v2_completed:C_R338
- added R339: 2.2k, symbol sr_rx_v2_completed:C_R339
- added R340: 100, symbol sr_rx_v2_completed:C_R340
- added R341: 2.2k, symbol sr_rx_v2_completed:C_R341
- added R342: 100, symbol sr_rx_v2_completed:C_R342
- added R343: 2.2k, symbol sr_rx_v2_completed:C_R343
- added R344: 100, symbol sr_rx_v2_completed:C_R344
- added R345: 2.2k, symbol sr_rx_v2_completed:C_R345
- added R346: 100, symbol sr_rx_v2_completed:C_R346
- added R347: 2.2k, symbol sr_rx_v2_completed:C_R347
- added R348: 100, symbol sr_rx_v2_completed:C_R348
- added R349: 2.2k, symbol sr_rx_v2_completed:C_R349
- added R350: 100, symbol sr_rx_v2_completed:C_R350
- added R390: 10k, symbol sr_rx_v2_completed:C_R390
- added R391: 1k, symbol sr_rx_v2_completed:C_R391
- added R393: 100, symbol sr_rx_v2_completed:C_R393
- added R394: 100k, symbol sr_rx_v2_completed:C_R394
- added R395: 1k, symbol sr_rx_v2_completed:C_R395
- added SW302: HOME momentary NO, symbol sr_rx_v2_completed:C_SW302
- added SW303: BACK momentary NO, symbol sr_rx_v2_completed:C_SW303
- added SW304: REC momentary NO, symbol sr_rx_v2_completed:C_SW304
- added SW305: MARK momentary NO, symbol sr_rx_v2_completed:C_SW305
- added SW306: FN momentary NO, symbol sr_rx_v2_completed:C_SW306
- added SW307: LOCK momentary NO, symbol sr_rx_v2_completed:C_SW307
- added SW308: ENC1_PRESS momentary NO, symbol sr_rx_v2_completed:C_SW308
- added SW309: ENC2_PRESS momentary NO, symbol sr_rx_v2_completed:C_SW309
- added TH301: Semiware MF52A103F3950, symbol sr_rx_v2_completed:C_TH301
- added TH302: Semiware MF52A103F3950, symbol sr_rx_v2_completed:C_TH302
- added U306: PI4IOE5V9555LEX 0x20, Package_SO:TSSOP-24_4.4x7.8mm_P0.65mm, symbol sr_rx_v2_completed:C_U306
- added U309: Waveshare RP2040-Zero 20187, symbol sr_rx_v2_completed:C_U309
- added U310: TPD4E1U06DBVR, Package_TO_SOT_SMD:SOT-23-6, symbol sr_rx_v2_completed:C_U310
- added U311: TPD4E1U06DBVR, Package_TO_SOT_SMD:SOT-23-6, symbol sr_rx_v2_completed:C_U311
- added U314: Adafruit 4754 BNO085 SPI, symbol sr_rx_v2_completed:C_U314
Connections:
- net E3_ADC3V0: now also R332.1, R333.1
- net E3_CASE_TEMP: now also C311.1, R333.2, TH302.1
- net E3_HMI_INT: now also R334.1, U306.1 (INT_N)
- net E3_HMI_SCL: now also U306.22 (SCL)
- net E3_HMI_SDA: now also U306.23 (SDA)
- net E3_MCP_RESET_ASSERT: now also R393.1, R395.2
- net E3_MCP_RESET_N: now also Q306.3 (D)
- net E3_PANEL_TEMP: now also C310.1, R332.2, TH301.1
- net E3_PICO3V3: now also C312.1, C313.1, R334.2, R335.2, R337.2, R339.2, R341.2, R343.2, R345.2, R347.2, R349.2, R395.1, U306.24 (VCC)
- net GND: now also C310.2, C311.2, C312.2, C313.2, C340.2, C341.2, Q306.2 (S), R394.2, SW302.2 (B), SW303.2 (B), SW304.2 (B), SW305.2 (B), SW306.2 (B), SW307.2 (B), SW308.2 (B), SW309.2 (B), TH301.2, TH302.2, U306.12 (GND), U306.2 (A1), U306.21 (A0), U306.3 (A2), U309.GND, U310.2 (GND), U311.2 (GND), U314.GND
- net IMU_RX: now also U309.GP1
- net IMU_TX: now also U309.GP0
- new net E3_BACK: R337.1, R338.1, U306.5 (IO0_1)
- new net E3_BACK_EXT: R338.2, SW303.1 (A), U310.3 (D2+)
- new net E3_ENC1_PRESS: R347.1, R348.1, U306.10 (IO0_6)
- new net E3_ENC1_PRESS_EXT: R348.2, SW308.1 (A), U311.4 (D2-)
- new net E3_ENC2_PRESS: R349.1, R350.1, U306.11 (IO0_7)
- new net E3_ENC2_PRESS_EXT: R350.2, SW309.1 (A), U311.6 (D1-)
- new net E3_FN: R343.1, R344.1, U306.8 (IO0_4)
- new net E3_FN_EXT: R344.2, SW306.1 (A), U311.1 (D1+)
- new net E3_HOME: R335.1, R336.1, U306.4 (IO0_0)
- new net E3_HOME_EXT: R336.2, SW302.1 (A), U310.1 (D1+)
- new net E3_IMU3V3: C341.1, R390.2, R391.2, U309.3V3 (3V3_OUT), U314.P1 (PS1), U314.VIN
- new net E3_IMU_CS_N: R390.1, U309.GP5, U314.CS (CS_N)
- new net E3_IMU_INT_N: U309.GP6, U314.INT (INT_N)
- new net E3_IMU_MISO: U309.GP4, U314.SDA (SDA_SPI_MISO)
- new net E3_IMU_MOSI: U309.GP3, U314.DI (DI_SPI_MOSI)
- new net E3_IMU_RST_N: U309.GP7, U314.RST (RST_N)
- new net E3_IMU_SCK: U309.GP2, U314.SCL (SCL_SPI_SCK)
- new net E3_IMU_WAKE_N: R391.1, U309.GP8, U314.P0 (PS0)
- new net E3_LOCK: R345.1, R346.1, U306.9 (IO0_5)
- new net E3_LOCK_EXT: R346.2, SW307.1 (A), U311.3 (D2+)
- new net E3_MARK: R341.1, R342.1, U306.7 (IO0_3)
- new net E3_MARK_EXT: R342.2, SW305.1 (A), U310.6 (D1-)
- new net E3_MCP_RESET_GATE: Q306.1 (G), R393.2, R394.1
- new net E3_REC: R339.1, R340.1, U306.6 (IO0_2)
- new net E3_REC_EXT: R340.2, SW304.1 (A), U310.4 (D2-)
- new net E5_IMU_VIN: C340.1, U309.5V (5V_IN)
- no-connect marks 27 -> 44
Other:
- note added: "BOM candidate Semiware MF52A103F3950 is selected for both NTCs; purchased-lot curve, attachment, lag and installed calibration remain unqualified. Ворота (стенд): Verify 10k +/-1% at 25 C and manufacturer B25/50 = 3950 +/-1%; use the exact maker R/T table. Fit an insulated bead/strain relief on the panel spreader and frame, check 25/60/68 C against a reference thermometer, qualify lag and open/sh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"
- note added: "E3 - Керування, Pico HMI, GPIO, GNSS і IMU (1/2)"
- note added: "E3-01 — OPEN, блокує випуск — STACK §2.8; §5.2; §8 (пак IMU); §8.1 (пак IMU)"
- note added: "E3-05 — OPEN, блокує випуск — STACK §5.2 (MCP23017 #3/#4)"
- note added: "E3-06 — OPEN, блокує випуск — STACK §5.6; §8 (тепло)"
- note added: "E3-08 — OPEN, блокує випуск — STACK §5.2; §5.4"
- note added: "External IMU"
- note added: "HMI buttons"
- note added: "IMU assembly and two metre single-ended UART need bench verification. Internal named-pad wiring is specified, but no physical harness has been measured. Ворота (стенд): Check actual module revision, GX16 plug/socket viewing direction and continuity to E5 design pinout; validate input Schottky and TVS at both ends; 1e6 frames with zero CRC errors. Upgrade to differential interface if errors occur."
- note added: "MCP hardware watchdog reset"
- note added: "Pico watchdog, MicroPython GPIO/UART adapter and host handshake implemented 20.10.2026 and tested on the host. Actual GPIO timing, reset levels, WDT/brownout behavior and Linux/serial fault recovery have not been qualified on the device. Ворота (стенд): Run the implemented firmware with the actual accepted Pico/Q6A assembly: scope MCP RESET assertion/release, safe output image including CHG_INHIB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"
- note added: "Shared MCP interrupt requires open-drain configuration before interrupts are enabled, plus measured I2C rise time and VOL. Ворота (стенд): Set ODR=1 and MIRROR=1 first. Validate 100kHz, rise <=1000ns, 1e6 reads under load, 20 cold/20 warm boots, and 10us FAULT capture."
- note added: "Thermal sensors"
- note added: "Дроти з'єднують контакти всередині функціональної групи; кожне дерево дротів має одну глобальну мітку з канонічною назвою мережі (рамка-стрілка — мережа виходить за межі групи, пряма рамка — мережа лише цієї групи). Однакові мітки з'єднані на всіх аркушах; земля — символ GND. Рамки OPEN — незакриті ворота з design/E#.json (повний реєстр: OPEN_ITEMS.md); «TBD» у значенні — STACK номіналу не задає,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"
- note added: "Позначення фізичних джерел живлення (ERC)"
- note removed: "E3 - Керування, Pico HMI, GPIO, GNSS і IMU (1/3)"
- note removed: "GNSS"
- note removed: "Pico HMI"
- note removed: "Q6A header"
- note removed: "Мережі з однаковими глобальними мітками електрично з'єднані на всіх аркушах. Фізичні/функціональні контакти: див. design/ і OPEN_ITEMS.md."
- title: E3 - Керування, Pico HMI, GPIO, GNSS і IMU (1/3) -> E3 - Керування, Pico HMI, GPIO, GNSS і IMU (1/2)
- moved on the sheet: J303, U301, U302, U303
