File: sat-receiver-audit/build/kicad/E3.kicad_sch (KiCad schematic)
At the start: 79 parts, among them J303 Q6A J11 RTC battery 1.25mm, Q306 2N7002,215, SW302 HOME momentary NO, SW303 BACK momentary NO, SW304 REC momentary NO, SW305 MARK momentary NO, SW306 FN momentary NO, SW307 LOCK momentary NO, SW308 ENC1_PRESS momentary NO, SW309 ENC2_PRESS momentary NO, U301 MCP23017-E/SO #1 0x20, U302 MCP23017-E/SO #3 0x22, U303 MCP23017-E/SO #4 0x23, U306 PI4IOE5V9555LEX 0x20, U309 Waveshare RP2040-Zero 20187, U310 TPD4E1U06DBVR, U311 TPD4E1U06DBVR, U314 Adafruit 4754 BNO085 SPI

Commit message: Stage 2 integration: CAD and DC_CORE re-freeze from CI run 40094234222; bound-count test and PCB hash lists follow
Co-Authored-By: Claude Opus 5.5 <noreply@anthropic.com>
Parts:
- removed C340: 10u 10V, symbol sr_rx_v2_completed:C_C340
- removed C341: 100n 16V, symbol sr_rx_v2_completed:C_C341
- removed R390: 10k, symbol sr_rx_v2_completed:C_R390
- removed R391: 1k, symbol sr_rx_v2_completed:C_R391
- removed U309: Waveshare RP2040-Zero 20187, symbol sr_rx_v2_completed:C_U309
- removed U314: Adafruit 4754 BNO085 SPI, symbol sr_rx_v2_completed:C_U314
- added D302: BAT54, Package_TO_SOT_SMD:SOT-23, symbol sr_rx_v2_completed:C_D302
- added D303: BAT54, Package_TO_SOT_SMD:SOT-23, symbol sr_rx_v2_completed:C_D303
- added J301: Q6A J20 2x20 3.3V GPIO, symbol sr_rx_v2_completed:C_J301
- added J302: Power-board control harness DESIGN, symbol sr_rx_v2_completed:C_J302
- added Q302: 2N7002, Package_TO_SOT_SMD:SOT-23, symbol sr_rx_v2_completed:C_Q302
- added R301: 10k, symbol sr_rx_v2_completed:C_R301
- added R302: 10k, symbol sr_rx_v2_completed:C_R302
- added R303: 10k DNP, symbol sr_rx_v2_completed:C_R303
- added R304: 10k DNP, symbol sr_rx_v2_completed:C_R304
- added R330: 10k, symbol sr_rx_v2_completed:C_R330
- added R331: 100k, symbol sr_rx_v2_completed:C_R331
- added SW301: Power button momentary NO, symbol sr_rx_v2_completed:C_SW301
Connections:
- net 3V3_Q6A: now also J301.1 (3V3), J301.17 (3V3), J302.1 (3V3_Q6A), R301.2, R302.2, R303.2, R304.2
- net E3_PICO3V3: now also R330.2
- net GND: now also J301.14 (GND), J301.20 (GND), J301.25 (GND), J301.30 (GND), J301.34 (GND), J301.39 (GND), J301.6 (GND), J301.9 (GND), J302.2 (GND), Q302.2 (S), R331.2, SW301.2 (B)
- net I2C2_SCL: now also J301.28 (GPIO9_I2C2_SCL), J302.4 (SCL), R304.1
- net I2C2_SDA: now also J301.27 (GPIO8_I2C2_SDA), J302.3 (SDA), R303.1
- net MCP_INT: now also J301.5 (GPIO25), J302.5 (INT), R302.1
- new net E3_BUTTON_SENSE: D302.1 (A), R330.1
- new net E3_GNSS_PPS: J301.7 (GPIO96)
- new net E3_PICO_RUN: J301.38 (GPIO98_RUN)
- new net E3_PICO_SWCLK: J301.12 (GPIO97_SWCLK)
- new net E3_PICO_SWDIO: J301.35 (GPIO100_SWDIO)
- new net E3_Q6A_KEY_GATE: Q302.1 (G), R331.1
- new net I2C0_SCL: J301.15 (GPIO1_I2C0_SCL)
- new net I2C0_SDA: J301.13 (GPIO0_I2C0_SDA)
- new net INA228_ALERT: J301.3 (GPIO24), R301.1
- new net PWR_BUTTON: D302.3 (K), D303.3 (K), SW301.1 (A)
- new net PWR_ON_KEY: D303.1 (A), Q302.3 (D)
- new net SAFE_BOOT: J301.40 (GPIO99_SAFE_BOOT)
- new net UART5_RX: J301.10 (GPIO23_UART5_RX)
- new net UART5_TX: J301.8 (GPIO22_UART5_TX)
- new net UART6_RX: J301.18 (GPIO27_UART6_RX)
- new net UART6_TX: J301.16 (GPIO26_UART6_TX)
- new net UART7_RX: J301.29 (GPIO31_UART7_RX)
- new net UART7_TX: J301.32 (GPIO30_UART7_TX)
- new net VCC_5V_PERI: J301.2 (5V), J301.4 (5V)
- no-connect marks 44 -> 35
Other:
- note added: "E3-04 — OPEN, блокує випуск — STACK §5.2 (UART7, PPS, SWD); §8.1 (UART7; PPS)"
- note added: "Pico power control"
- note added: "Q6A header"
- note added: "UM3304 UART7/PPS/SWD cable capacitance and power-off behavior cannot be proven by ERC. Ворота (стенд): Check <=20cm wiring, UART7 loopback, boot glitches and absence of Q6A backfeed with Pico on/Q6A off. Verify TX high-impedance sequencing or add hardware isolation."
- note removed: "E3-01 — OPEN, блокує випуск — STACK §2.8; §5.2; §8 (пак IMU); §8.1 (пак IMU)"
- note removed: "External IMU"
- note removed: "IMU assembly and two metre single-ended UART need bench verification. Internal named-pad wiring is specified, but no physical harness has been measured. Ворота (стенд): Check actual module revision, GX16 plug/socket viewing direction and continuity to E5 design pinout; validate input Schottky and TVS at both ends; 1e6 frames with zero CRC errors. Upgrade to differential interface if errors occur."
- moved on the sheet: BT301, J303, U303
