File: sat-receiver-audit/build/kicad/E2_02.kicad_sch (KiCad schematic)
At the start: 58 parts, among them U204 LT3045EMSE#PBF, U205 LT3045EMSE#PBF, U206 TPS2553DBVR-1, U207 TPS2553DBVR-1, U208 TPS2553DBVR-1

Commit message: SR-RX-v2.1: review fixes on the Codex branch, readable schematic, one-file bundle
Independent review of the Codex branch (schematic vs STACK.md, hard rules,
security, tests) found no blockers; this commit applies its findings:

- rules in code: Cospas-Sarsat 406.0-406.1 MHz added to the no-data mask;
  Q6A Wi-Fi/BT off in the field/QUIET root (modprobe blacklist, udev
  authorized=0 on FE1.1s port 4, rfkill) with self-checks; device denylist
  completed per STACK (gr-gsm, gr-iridium, kalibrate, pager/trunking decoders,
  TX-capable tools); W1-2 WIFI_PWR_EN as blocking open item E5-10
- STACK.md is the source of truth again; v2.1 changes recorded in it; the
  "historical" marker kept only on ISDT/raw-balance rows; gender-neutral wording
- schematic data: open values shown as TBD with start values and notes, U503
  TPS2553DBVR-1, Lime X2/X4 RX mapping TBD, 37 open items drawn on the sheets
- schematic readability: wired groups, junctions, GND symbols, standard
  transistor/diode symbols; netlist unchanged (603 nets identical)
- tooling: reproducible run_checks (no timestamps or machine paths), pinned
  dependencies, bundle excludes cache folders, clean-checkout bundle check
- regenerated: KiCad export (14 pages), netlist/ERC, module lab, PCB inputs,
  readiness contract, acceptance hashes, SR-RX-v2-ves-proekt.html

Checks: ERC 0 errors/0 warnings, netlist comparison PASS, 432 tests (431
passed, 1 skipped), deployment tests OK, bundle check PASS on a clean checkout.

History note: earlier versions of the generated SR-RX-v2-ves-proekt.html and
handoff/handoff-bundle.zip were removed from history; only the final versions
are kept. The Codex merge commit is now attributed to Codex.

Co-Authored-By: Claude Opus 5.5 <noreply@anthropic.com>
Claude-Session: https://claude.ai/code/session_01W9CKpimWpgkUmrDQQMiKtF
Parts:
- removed C221: 10uF 50V X7R C3225X7R1H106K250AC, Capacitor_SMD:C_1210_3225Metric, symbol sr_rx_v2_completed:C_C221
- removed C222: 47uF 50V EEUFR1H470, symbol sr_rx_v2_completed:C_C222
- removed C232: 1uF 50V X7R C2012X7R1H105K125AB, Capacitor_SMD:C_0805_2012Metric, symbol sr_rx_v2_completed:C_C232
- removed C233: 1uF 50V X7R C2012X7R1H105K125AB, Capacitor_SMD:C_0805_2012Metric, symbol sr_rx_v2_completed:C_C233
- removed C234: 1uF 50V X7R C2012X7R1H105K125AB, Capacitor_SMD:C_0805_2012Metric, symbol sr_rx_v2_completed:C_C234
- removed C235: 47uF 50V EEUFR1H470, symbol sr_rx_v2_completed:C_C235
- removed C236: 1uF 50V X7R C2012X7R1H105K125AB, Capacitor_SMD:C_0805_2012Metric, symbol sr_rx_v2_completed:C_C236
- removed C237: 1uF 50V X7R C2012X7R1H105K125AB, Capacitor_SMD:C_0805_2012Metric, symbol sr_rx_v2_completed:C_C237
- removed C238: 1uF 50V X7R C2012X7R1H105K125AB, Capacitor_SMD:C_0805_2012Metric, symbol sr_rx_v2_completed:C_C238
- removed C239: 47uF 50V EEUFR1H470, symbol sr_rx_v2_completed:C_C239
- removed L206: 1uH XAL5030-102MEC, symbol sr_rx_v2_completed:C_L206
- removed L207: 1uH XAL5030-102MEC, symbol sr_rx_v2_completed:C_L207
- removed R223: 0.22R 1% 0.25W, symbol sr_rx_v2_completed:C_R223
- removed R228: 88.7k 1%, symbol sr_rx_v2_completed:C_R228
- removed R229: 100k 1%, symbol sr_rx_v2_completed:C_R229
- removed R231: 0.200R 0.1% 0.25W Kelvin, symbol sr_rx_v2_completed:C_R231
- removed R232: 0.22R 1% 0.25W, symbol sr_rx_v2_completed:C_R232
- removed R233: 88.7k 1%, symbol sr_rx_v2_completed:C_R233
- removed R234: 100k 1%, symbol sr_rx_v2_completed:C_R234
- removed R236: 0.200R 0.1% 0.25W Kelvin, symbol sr_rx_v2_completed:C_R236
- removed R237: 0.22R 1% 0.25W, symbol sr_rx_v2_completed:C_R237
- removed TP204: AUX12, symbol sr_rx_v2_completed:C_TP204
- removed TP206: BIAS_CH1, symbol sr_rx_v2_completed:C_TP206
- removed TP207: BIAS_CH2, symbol sr_rx_v2_completed:C_TP207
- removed U206: TPS2553DBVR-1, symbol sr_rx_v2_completed:C_U206
- removed U207: TPS2553DBVR-1, symbol sr_rx_v2_completed:C_U207
- added C244: 1uF 50V X7R C2012X7R1H105K125AB, Capacitor_SMD:C_0805_2012Metric, symbol sr_rx_v2_completed:C_C244
- added C245: 1uF 50V X7R C2012X7R1H105K125AB, Capacitor_SMD:C_0805_2012Metric, symbol sr_rx_v2_completed:C_C245
- added C246: 1uF 50V X7R C2012X7R1H105K125AB, Capacitor_SMD:C_0805_2012Metric, symbol sr_rx_v2_completed:C_C246
- added C247: 47uF 50V EEUFR1H470, symbol sr_rx_v2_completed:C_C247
- added C248: 1uF 50V X7R C2012X7R1H105K125AB, Capacitor_SMD:C_0805_2012Metric, symbol sr_rx_v2_completed:C_C248
- added C249: 1uF 50V X7R C2012X7R1H105K125AB, Capacitor_SMD:C_0805_2012Metric, symbol sr_rx_v2_completed:C_C249
- added C250: 1uF 50V X7R C2012X7R1H105K125AB, Capacitor_SMD:C_0805_2012Metric, symbol sr_rx_v2_completed:C_C250
- added C251: 47uF 50V EEUFR1H470, symbol sr_rx_v2_completed:C_C251
- added C286: 10nF 50V C0G C1608C0G1H103J080AA, Capacitor_SMD:C_0603_1608Metric, symbol sr_rx_v2_completed:C_C286
- added C287: 100nF 50V X7R C1608X7R1H104K080AA, Capacitor_SMD:C_0603_1608Metric, symbol sr_rx_v2_completed:C_C287
- added C288: 100nF 50V X7R C1608X7R1H104K080AA, Capacitor_SMD:C_0603_1608Metric, symbol sr_rx_v2_completed:C_C288
- added L209: 1uH XAL5030-102MEC, symbol sr_rx_v2_completed:C_L209
- added L210: 1uH XAL5030-102MEC, symbol sr_rx_v2_completed:C_L210
- added R243: 162k 1%, symbol sr_rx_v2_completed:C_R243
- added R244: 100k 1%, symbol sr_rx_v2_completed:C_R244
- added R246: 0.200R 0.1% 0.25W Kelvin, symbol sr_rx_v2_completed:C_R246
- added R247: 0.22R 1% 0.25W, symbol sr_rx_v2_completed:C_R247
- added R248: RILIM TBD (start 56.2k 1%), symbol sr_rx_v2_completed:C_R248
- added R249: 100k 1%, symbol sr_rx_v2_completed:C_R249
- added R251: 0.22R 1% 0.25W, symbol sr_rx_v2_completed:C_R251
- added R286: 73.2k 0.1%, symbol sr_rx_v2_completed:C_R286
- added R287: 10.0k 0.1%, symbol sr_rx_v2_completed:C_R287
- added R288: TNPW0805332KBYEA 332k 0.1%10ppm, symbol sr_rx_v2_completed:C_R288
- added R289: TNPW08052K00BYEA 2.00k 0.1%10ppm, symbol sr_rx_v2_completed:C_R289
- added R290: TNPW080510K0BYEA 10.0k 0.1%10ppm, symbol sr_rx_v2_completed:C_R290
- added R291: 4.70k 1%, symbol sr_rx_v2_completed:C_R291
- added R292: 100k 1%, symbol sr_rx_v2_completed:C_R292
- added TP209: BIAS_CH4, symbol sr_rx_v2_completed:C_TP209
- added TP210: VBUS_RTLB, symbol sr_rx_v2_completed:C_TP210
- added TP215: OVP_LNB_N, symbol sr_rx_v2_completed:C_TP215
- added U209: TPS2553DBVR-1, symbol sr_rx_v2_completed:C_U209
- added U210: TPS2553DBVR-1, symbol sr_rx_v2_completed:C_U210
- added U219: TLV3011BIDBVR, symbol sr_rx_v2_completed:C_U219
- added U220: TPS3701DDCR, symbol sr_rx_v2_completed:C_U220
Connections:
- net AUX12: now also R286.1
- net GND: now also C244.2, C245.2, C246.2, C247.2 (-), C248.2, C249.2, C250.2, C251.2 (-), C286.2, C287.2, C288.2, R243.2, R244.2, R248.2, R249.2, R287.2, R290.2, R292.2, U209.2 (GND), U210.2 (GND), U219.2 (V-), U220.2 (GND), U220.3 (INA)
- net LAB5: now also C248.1, U210.1 (IN)
- net LNA4V5: now also C244.1, U209.1 (IN)
- new net 3V3_Q6A: C287.1, U219.6 (V+)
- new net BIAS_CH4: C246.1, L209.2, R247.1, TP209.1 (TP)
- new net BIAS_CH4_DAMP: C247.1 (+), R247.2
- new net E1_SW: C288.1, U220.5 (VDD)
- new net E2_LNA4_SHUNT: C245.1, L209.1, R246.2
- new net E2_LNA4_SW: R246.1, U209.6 (OUT)
- new net E2_LNB_LDO: R288.1
- new net E2_LNB_OV_DIV_MID: R288.2, R289.1
- new net E2_LNB_PRECISE_SENSE: R289.2, R290.1, U220.4 (INB)
- new net E2_RTLB_SW: C249.1, L210.1, U210.6 (OUT)
- new net E2_U209_ILIM: R243.1, U209.5 (ILIM)
- new net E2_U210_ILIM: R248.1, U210.5 (ILIM)
- new net E2_U219_REF: U219.4 (IN-), U219.5 (REF)
- new net E2_U219_SENSE: C286.1, R286.2, R287.1, U219.3 (IN+)
- new net EN_LNA4: R244.1, U209.3 (EN)
- new net EN_LNB: R291.1
- new net EN_RTLB: R249.1, U210.3 (EN)
- new net FAULT_LNA4: U209.4 (FAULT)
- new net FAULT_RTLB: U210.4 (FAULT)
- new net OVP_LNB_N: R291.2, R292.1, TP215.1 (TP), U220.6 (OUTB)
- new net PTC_AUX: U219.1 (OUT)
- new net VBUS_RTLB: C250.1, L210.2, R251.1, TP210.1 (TP)
- new net VBUS_RTLB_DAMP: C251.1 (+), R251.2
- no-connect marks 2 -> 3
Other:
- note added: "AUX12: контроль напруги після PTC"
- note added: "E2 - Захищені рейки, LNA і моніторинг струму (2/4)"
- note added: "E2-01 — OPEN, блокує випуск — STACK §5.1 (LNA4V5, LNB13V2, BONI13V8); §8 (пара LT3045; TPS7A4701)"
- note added: "E2-03 — OPEN, блокує випуск — STACK §5.1 (VBUS RTL-B, BONI13V8); §8 (струми; TPS2553DBVR-1 п. 3); §8.1 RF-2, HF-8/RF-5"
- note added: "E2-04 — OPEN, блокує випуск — STACK §5.1 (LNA4V5); §8 (пара LT3045); §8.1 RF-3"
- note added: "LNA: канал 4"
- note added: "LNB: незалежне точне відсікання OVP"
- note added: "MPN L/C і діодів обрані. Ефективна ємність, ESR/ESL, демпфування LC та від’ємний викид OUT залежать від розведення і реальних деталей. Ворота (стенд): Перевірити COUT ≥10uF при робочому bias/температурі, ESR LT3045 <20mR і ESL <2nH; виконати тести ступінчастого навантаження, RF-шуму та від’ємного OUT ≥−0.4V."
- note added: "N-E2-01 — примітка — STACK §5.1 (VBUS RTL-B); §8 (TPS2553DBVR-1 п. 3)"
- note added: "R248 = RILIM TBD (старт 56.2k 1%, ≈0.47 A ном.). STACK не задає номінал для VBUS RTL-B, лише правило: RILIM = 1.5–2× виміряного струму. Ворота: E2-03 (20 холодних і теплих пусків, пусковий струм до deglitch 5 ms)."
- note added: "RTL-B: комутований VBUS"
- note added: "Дроти з'єднують контакти всередині функціональної групи; кожне дерево дротів має одну глобальну мітку з канонічною назвою мережі (рамка-стрілка — мережа виходить за межі групи, пряма рамка — мережа лише цієї групи). Однакові мітки з'єднані на всіх аркушах; земля — символ GND. Рамки OPEN — незакриті ворота з design/E#.json (повний реєстр: OPEN_ITEMS.md); «TBD» у значенні — STACK номіналу не задає,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"
- note added: "Остаточні ILIM і пускові струми RTL-B, Lime, LNB, Boni та LaNA WB потребують натурних вимірів; ємність riser і комерційних модулів не опублікована. Поріг OVLO Boni (R263/R264, стартовий розрахунок 112k/10.0k) STACK §5.1 вимагає перерахувати для 13.8 V; на стенді його не перевірено. Ворота (стенд): FNB58/INA228/INA3221: 20 холодних і теплих пусків, струми стримінгу, КЗ і SOA. Установити ILIM 1.5–2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"
- note added: "Потрібне підтвердження запасу напруги, розподілу струму й температури пари LT3045 на 4.5V. Сума індивідуальних номінальних ILIM LNA більша за 1A пари. Ворота (стенд): Перевірити LAB5 min, навантаження пари до 1A, температуру кожного LT3045 та спад до антени. Дотримуватися контракту R-E2-17: сума INA LNA1–4 + резерв 65mA S-band ≤1A; разом із резервом LAB-порту ≤1.5A."
- note removed: "AUX12: верхній ключ і PTC"
- note removed: "E2 - Захищені рейки, LNA і моніторинг струму (2/5)"
- note removed: "LNA: канал 1"
- note removed: "LNA: канал 2"
- note removed: "Мережі з однаковими глобальними мітками електрично з'єднані на всіх аркушах. Фізичні/функціональні контакти: див. design/ і OPEN_ITEMS.md."
- title: E2 - Захищені рейки, LNA і моніторинг струму (2/5) -> E2 - Захищені рейки, LNA і моніторинг струму (2/4)
- moved on the sheet: U204, U205, U208
