File: sat-receiver-audit/build/kicad/E2_03.kicad_sch (KiCad schematic)
At the start: 56 parts, among them U209 TPS2553DBVR-1, U210 TPS2553DBVR-1, U211 TPS7A4701RGWT, U212 TPS259630DDAR, U213 TPS7A4701RGWT

Commit message: SR-RX-v2.1: review fixes on the Codex branch, readable schematic, one-file bundle
Independent review of the Codex branch (schematic vs STACK.md, hard rules,
security, tests) found no blockers; this commit applies its findings:

- rules in code: Cospas-Sarsat 406.0-406.1 MHz added to the no-data mask;
  Q6A Wi-Fi/BT off in the field/QUIET root (modprobe blacklist, udev
  authorized=0 on FE1.1s port 4, rfkill) with self-checks; device denylist
  completed per STACK (gr-gsm, gr-iridium, kalibrate, pager/trunking decoders,
  TX-capable tools); W1-2 WIFI_PWR_EN as blocking open item E5-10
- STACK.md is the source of truth again; v2.1 changes recorded in it; the
  "historical" marker kept only on ISDT/raw-balance rows; gender-neutral wording
- schematic data: open values shown as TBD with start values and notes, U503
  TPS2553DBVR-1, Lime X2/X4 RX mapping TBD, 37 open items drawn on the sheets
- schematic readability: wired groups, junctions, GND symbols, standard
  transistor/diode symbols; netlist unchanged (603 nets identical)
- tooling: reproducible run_checks (no timestamps or machine paths), pinned
  dependencies, bundle excludes cache folders, clean-checkout bundle check
- regenerated: KiCad export (14 pages), netlist/ERC, module lab, PCB inputs,
  readiness contract, acceptance hashes, SR-RX-v2-ves-proekt.html

Checks: ERC 0 errors/0 warnings, netlist comparison PASS, 432 tests (431
passed, 1 skipped), deployment tests OK, bundle check PASS on a clean checkout.

History note: earlier versions of the generated SR-RX-v2-ves-proekt.html and
handoff/handoff-bundle.zip were removed from history; only the final versions
are kept. The Codex merge commit is now attributed to Codex.

Co-Authored-By: Claude Opus 5.5 <noreply@anthropic.com>
Claude-Session: https://claude.ai/code/session_01W9CKpimWpgkUmrDQQMiKtF
Parts:
- removed C244: 1uF 50V X7R C2012X7R1H105K125AB, Capacitor_SMD:C_0805_2012Metric, symbol sr_rx_v2_completed:C_C244
- removed C245: 1uF 50V X7R C2012X7R1H105K125AB, Capacitor_SMD:C_0805_2012Metric, symbol sr_rx_v2_completed:C_C245
- removed C246: 1uF 50V X7R C2012X7R1H105K125AB, Capacitor_SMD:C_0805_2012Metric, symbol sr_rx_v2_completed:C_C246
- removed C247: 47uF 50V EEUFR1H470, symbol sr_rx_v2_completed:C_C247
- removed C248: 1uF 50V X7R C2012X7R1H105K125AB, Capacitor_SMD:C_0805_2012Metric, symbol sr_rx_v2_completed:C_C248
- removed C249: 1uF 50V X7R C2012X7R1H105K125AB, Capacitor_SMD:C_0805_2012Metric, symbol sr_rx_v2_completed:C_C249
- removed C250: 1uF 50V X7R C2012X7R1H105K125AB, Capacitor_SMD:C_0805_2012Metric, symbol sr_rx_v2_completed:C_C250
- removed C251: 47uF 50V EEUFR1H470, symbol sr_rx_v2_completed:C_C251
- removed L209: 1uH XAL5030-102MEC, symbol sr_rx_v2_completed:C_L209
- removed L210: 1uH XAL5030-102MEC, symbol sr_rx_v2_completed:C_L210
- removed R243: 162k 1%, symbol sr_rx_v2_completed:C_R243
- removed R244: 100k 1%, symbol sr_rx_v2_completed:C_R244
- removed R246: 0.200R 0.1% 0.25W Kelvin, symbol sr_rx_v2_completed:C_R246
- removed R247: 0.22R 1% 0.25W, symbol sr_rx_v2_completed:C_R247
- removed R248: 56.2k 1%, symbol sr_rx_v2_completed:C_R248
- removed R249: 100k 1%, symbol sr_rx_v2_completed:C_R249
- removed R251: 0.22R 1% 0.25W, symbol sr_rx_v2_completed:C_R251
- removed TP209: BIAS_CH4, symbol sr_rx_v2_completed:C_TP209
- removed TP210: VBUS_RTLB, symbol sr_rx_v2_completed:C_TP210
- removed U209: TPS2553DBVR-1, symbol sr_rx_v2_completed:C_U209
- removed U210: TPS2553DBVR-1, symbol sr_rx_v2_completed:C_U210
- added C269: 100nF 50V X7R C1608X7R1H104K080AA, Capacitor_SMD:C_0603_1608Metric, symbol sr_rx_v2_completed:C_C269
- added C270: 1uF 50V X7R C2012X7R1H105K125AB, Capacitor_SMD:C_0805_2012Metric, symbol sr_rx_v2_completed:C_C270
- added C271: 1uF 50V X7R C2012X7R1H105K125AB, Capacitor_SMD:C_0805_2012Metric, symbol sr_rx_v2_completed:C_C271
- added C272: 1uF 50V X7R C2012X7R1H105K125AB, Capacitor_SMD:C_0805_2012Metric, symbol sr_rx_v2_completed:C_C272
- added C273: 47uF 50V EEUFR1H470, symbol sr_rx_v2_completed:C_C273
- added C294: 22uF 50V X7R C3225X7R1H226M250AC, Capacitor_SMD:C_1210_3225Metric, symbol sr_rx_v2_completed:C_C294
- added D203: PMEG4030ER, Diode_SMD:Nexperia_CFP3_SOD-123W, symbol sr_rx_v2_completed:C_D203
- added L214: 1uH XAL5030-102MEC, symbol sr_rx_v2_completed:C_L214
- added R262: 7.87k 1%, symbol sr_rx_v2_completed:C_R262
- added R263: OVLO TBD (start 112k 0.1%), symbol sr_rx_v2_completed:C_R263
- added R264: OVLO TBD (start 10.0k 0.1%), symbol sr_rx_v2_completed:C_R264
- added R266: 0.200R 0.1% 0.25W Kelvin, symbol sr_rx_v2_completed:C_R266
- added R267: 0.22R 1% 0.25W, symbol sr_rx_v2_completed:C_R267
- added TP212: BONI13V8, symbol sr_rx_v2_completed:C_TP212
- added U214: TPS259630DDAR, symbol sr_rx_v2_completed:C_U214
Connections:
- net E2_BONI_LDO: now also C294.1, D203.1 (K), R263.1, U214.4 (IN)
- net EN_BONI: now also U214.3 (EN/UVLO)
- net GND: now also C269.2, C270.2, C271.2, C272.2, C273.2 (-), C294.2, D203.2 (A), R262.2, R264.2, U214.1 (GND), U214.EP
- new net BONI13V8: C272.1, L214.2, R267.1, TP212.1 (TP)
- new net BONI13V8_DAMP: C273.1 (+), R267.2
- new net E2_BONI_DVDT: C269.1, U214.2 (dVdt)
- new net E2_BONI_EF: C270.1, R266.1, U214.5 (OUT)
- new net E2_BONI_ILM: R262.1, U214.7 (ILM)
- new net E2_BONI_MON: C271.1, L214.1, R266.2
- new net E2_BONI_OV: R263.2, R264.1, U214.8 (OVLO)
- new net FLT_BONI: U214.6 (FLT)
Other:
- note added: "E2 - Захищені рейки, LNA і моніторинг струму (3/4)"
- note added: "E2-02 — OPEN, блокує випуск — STACK §5.1 (LNB13V2); §8 (TPS7A4701); §8.1 RF-4"
- note added: "N-E2-02 — примітка — STACK §5.1 (BONI13V8); §8.1 HF-8/RF-5"
- note added: "R263/R264 = OVLO TBD (старт 112k/10.0k 0.1%: 14.64 V ном., ≈14.24–14.92 V за R-E2-02). STACK §5.1 (BONI13V8): «OVLO перерахувати для 13.8 V» — номіналу в STACK немає. Ворота: E2-03 (стенд STACK §8.1 HF-8/RF-5: OVLO не спрацьовує в смузі 13.8 V; поріг вище 14.145 V і нижче 15 V)."
- note added: "Дроти з'єднують контакти всередині функціональної групи; кожне дерево дротів має одну глобальну мітку з канонічною назвою мережі (рамка-стрілка — мережа виходить за межі групи, пряма рамка — мережа лише цієї групи). Однакові мітки з'єднані на всіх аркушах; земля — символ GND. Рамки OPEN — незакриті ворота з design/E#.json (повний реєстр: OPEN_ITEMS.md); «TBD» у значенні — STACK номіналу не задає,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"
- note added: "Статичне вікно OVP LNB закрито TPS3701: 13.56–13.96V. Швидкий викид при відмові LDO не обмежено гарантованим максимальним часом у даташитах: 9.9µs компаратора і близько 12µs EN-off eFuse задані лише типово. Ворота (стенд): Без LNB і зі струмовим обмеженням подати на вузол LDO контрольований стрибок 13.2→16.4V; осцилографувати F-вихід при мін./макс. навантаженні, на холоді й при 50°C. Отримати гра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"
- note removed: "E2 - Захищені рейки, LNA і моніторинг струму (3/5)"
- note removed: "LNA: канал 4"
- note removed: "RTL-B: комутований VBUS"
- note removed: "Мережі з однаковими глобальними мітками електрично з'єднані на всіх аркушах. Фізичні/функціональні контакти: див. design/ і OPEN_ITEMS.md."
- title: E2 - Захищені рейки, LNA і моніторинг струму (3/5) -> E2 - Захищені рейки, LNA і моніторинг струму (3/4)
- moved on the sheet: U211, U212, U213
