File: sat-receiver-audit/build/kicad/E2_03.kicad_sch (KiCad schematic)
At the start: 50 parts, among them U211 TPS7A4701RGWT, U212 TPS259630DDAR, U213 TPS7A4701RGWT, U214 TPS259630DDAR

Commit message: Stage 2 integration: CAD and DC_CORE re-freeze from CI run 40094234222; bound-count test and PCB hash lists follow
Co-Authored-By: Claude Opus 5.5 <noreply@anthropic.com>
Parts:
- removed C252: 10uF 50V X7R C3225X7R1H106K250AC, Capacitor_SMD:C_1210_3225Metric, symbol sr_rx_v2_completed:C_C252
- removed C253: 10uF 50V X7R C3225X7R1H106K250AC, Capacitor_SMD:C_1210_3225Metric, symbol sr_rx_v2_completed:C_C253
- removed C254: 47uF 50V EEUFR1H470, symbol sr_rx_v2_completed:C_C254
- removed C255: 10uF 50V X7R C3225X7R1H106K250AC, Capacitor_SMD:C_1210_3225Metric, symbol sr_rx_v2_completed:C_C255
- removed C256: 22uF 50V X7R C3225X7R1H226M250AC, Capacitor_SMD:C_1210_3225Metric, symbol sr_rx_v2_completed:C_C256
- removed C257: 1uF 50V X7R C2012X7R1H105K125AB, Capacitor_SMD:C_0805_2012Metric, symbol sr_rx_v2_completed:C_C257
- removed C258: 47nF 50V X7R C1608X7R1H473K080AA, Capacitor_SMD:C_0603_1608Metric, symbol sr_rx_v2_completed:C_C258
- removed C259: 1uF 50V X7R C2012X7R1H105K125AB, Capacitor_SMD:C_0805_2012Metric, symbol sr_rx_v2_completed:C_C259
- removed C260: 1uF 50V X7R C2012X7R1H105K125AB, Capacitor_SMD:C_0805_2012Metric, symbol sr_rx_v2_completed:C_C260
- removed C261: 1uF 50V X7R C2012X7R1H105K125AB, Capacitor_SMD:C_0805_2012Metric, symbol sr_rx_v2_completed:C_C261
- removed C262: 47uF 50V EEUFR1H470, symbol sr_rx_v2_completed:C_C262
- removed C263: 10uF 50V X7R C3225X7R1H106K250AC, Capacitor_SMD:C_1210_3225Metric, symbol sr_rx_v2_completed:C_C263
- removed C264: 10uF 50V X7R C3225X7R1H106K250AC, Capacitor_SMD:C_1210_3225Metric, symbol sr_rx_v2_completed:C_C264
- removed C265: 47uF 50V EEUFR1H470, symbol sr_rx_v2_completed:C_C265
- removed C266: 10uF 50V X7R C3225X7R1H106K250AC, Capacitor_SMD:C_1210_3225Metric, symbol sr_rx_v2_completed:C_C266
- removed C267: 22uF 50V X7R C3225X7R1H226M250AC, Capacitor_SMD:C_1210_3225Metric, symbol sr_rx_v2_completed:C_C267
- removed C268: 1uF 50V X7R C2012X7R1H105K125AB, Capacitor_SMD:C_0805_2012Metric, symbol sr_rx_v2_completed:C_C268
- removed C269: 100nF 50V X7R C1608X7R1H104K080AA, Capacitor_SMD:C_0603_1608Metric, symbol sr_rx_v2_completed:C_C269
- removed C270: 1uF 50V X7R C2012X7R1H105K125AB, Capacitor_SMD:C_0805_2012Metric, symbol sr_rx_v2_completed:C_C270
- removed C271: 1uF 50V X7R C2012X7R1H105K125AB, Capacitor_SMD:C_0805_2012Metric, symbol sr_rx_v2_completed:C_C271
- removed C272: 1uF 50V X7R C2012X7R1H105K125AB, Capacitor_SMD:C_0805_2012Metric, symbol sr_rx_v2_completed:C_C272
- removed C273: 47uF 50V EEUFR1H470, symbol sr_rx_v2_completed:C_C273
- removed C293: 22uF 50V X7R C3225X7R1H226M250AC, Capacitor_SMD:C_1210_3225Metric, symbol sr_rx_v2_completed:C_C293
- removed C294: 22uF 50V X7R C3225X7R1H226M250AC, Capacitor_SMD:C_1210_3225Metric, symbol sr_rx_v2_completed:C_C294
- removed D202: PMEG4030ER, Diode_SMD:Nexperia_CFP3_SOD-123W, symbol sr_rx_v2_completed:C_D202
- removed D203: PMEG4030ER, Diode_SMD:Nexperia_CFP3_SOD-123W, symbol sr_rx_v2_completed:C_D203
- removed L211: 1uH XAL5030-102MEC, symbol sr_rx_v2_completed:C_L211
- removed L212: 1uH XAL5030-102MEC, symbol sr_rx_v2_completed:C_L212
- removed L213: 1uH XAL5030-102MEC, symbol sr_rx_v2_completed:C_L213
- removed L214: 1uH XAL5030-102MEC, symbol sr_rx_v2_completed:C_L214
- removed R252: 0.22R 1% 0.25W, symbol sr_rx_v2_completed:C_R252
- removed R253: 100k 1%, symbol sr_rx_v2_completed:C_R253
- removed R254: 2.05k 1%, symbol sr_rx_v2_completed:C_R254
- removed R255: 110k 0.5%, symbol sr_rx_v2_completed:C_R255
- removed R256: 10.0k 0.5%, symbol sr_rx_v2_completed:C_R256
- removed R258: 0.100R 0.1% 0.25W Kelvin, symbol sr_rx_v2_completed:C_R258
- removed R259: 0.22R 1% 0.25W, symbol sr_rx_v2_completed:C_R259
- removed R260: 0.22R 1% 0.25W, symbol sr_rx_v2_completed:C_R260
- removed R261: 100k 1%, symbol sr_rx_v2_completed:C_R261
- removed R262: 7.87k 1%, symbol sr_rx_v2_completed:C_R262
- removed R263: OVLO TBD (start 112k 0.1%), symbol sr_rx_v2_completed:C_R263
- removed R264: OVLO TBD (start 10.0k 0.1%), symbol sr_rx_v2_completed:C_R264
- removed R266: 0.200R 0.1% 0.25W Kelvin, symbol sr_rx_v2_completed:C_R266
- removed R267: 0.22R 1% 0.25W, symbol sr_rx_v2_completed:C_R267
- removed TP211: LNB13V2, symbol sr_rx_v2_completed:C_TP211
- removed TP212: BONI13V8, symbol sr_rx_v2_completed:C_TP212
- removed U211: TPS7A4701RGWT, symbol sr_rx_v2_completed:C_U211
- removed U212: TPS259630DDAR, symbol sr_rx_v2_completed:C_U212
- removed U213: TPS7A4701RGWT, symbol sr_rx_v2_completed:C_U213
- removed U214: TPS259630DDAR, symbol sr_rx_v2_completed:C_U214
- added C240: 1uF 50V X7R C2012X7R1H105K125AB, Capacitor_SMD:C_0805_2012Metric, symbol sr_rx_v2_completed:C_C240
- added C241: 1uF 50V X7R C2012X7R1H105K125AB, Capacitor_SMD:C_0805_2012Metric, symbol sr_rx_v2_completed:C_C241
- added C242: 1uF 50V X7R C2012X7R1H105K125AB, Capacitor_SMD:C_0805_2012Metric, symbol sr_rx_v2_completed:C_C242
- added C243: 47uF 50V EEUFR1H470, symbol sr_rx_v2_completed:C_C243
- added C248: 1uF 50V X7R C2012X7R1H105K125AB, Capacitor_SMD:C_0805_2012Metric, symbol sr_rx_v2_completed:C_C248
- added C249: 1uF 50V X7R C2012X7R1H105K125AB, Capacitor_SMD:C_0805_2012Metric, symbol sr_rx_v2_completed:C_C249
- added C250: 1uF 50V X7R C2012X7R1H105K125AB, Capacitor_SMD:C_0805_2012Metric, symbol sr_rx_v2_completed:C_C250
- added C251: 47uF 50V EEUFR1H470, symbol sr_rx_v2_completed:C_C251
- added C274: 100nF 50V X7R C1608X7R1H104K080AA, Capacitor_SMD:C_0603_1608Metric, symbol sr_rx_v2_completed:C_C274
- added C275: 100nF 50V X7R C1608X7R1H104K080AA, Capacitor_SMD:C_0603_1608Metric, symbol sr_rx_v2_completed:C_C275
- added C276: 100nF 50V X7R C1608X7R1H104K080AA, Capacitor_SMD:C_0603_1608Metric, symbol sr_rx_v2_completed:C_C276
- added C277: 100nF 50V X7R C1608X7R1H104K080AA, Capacitor_SMD:C_0603_1608Metric, symbol sr_rx_v2_completed:C_C277
- added C278: 100nF 50V X7R C1608X7R1H104K080AA, Capacitor_SMD:C_0603_1608Metric, symbol sr_rx_v2_completed:C_C278
- added C279: 100nF 50V X7R C1608X7R1H104K080AA, Capacitor_SMD:C_0603_1608Metric, symbol sr_rx_v2_completed:C_C279
- added C280: 100nF 50V X7R C1608X7R1H104K080AA, Capacitor_SMD:C_0603_1608Metric, symbol sr_rx_v2_completed:C_C280
- added C281: 100nF 50V X7R C1608X7R1H104K080AA, Capacitor_SMD:C_0603_1608Metric, symbol sr_rx_v2_completed:C_C281
- added C2902: 1uF 50V X7R C2012X7R1H105K125AB, Capacitor_SMD:C_0805_2012Metric, symbol sr_rx_v2_completed:C_C2902
- added C2912: 100nF 50V X7R C1608X7R1H104K080AA, Capacitor_SMD:C_0603_1608Metric, symbol sr_rx_v2_completed:C_C2912
- added C295: 1uF 50V X7R C2012X7R1H105K125AB, Capacitor_SMD:C_0805_2012Metric, symbol sr_rx_v2_completed:C_C295
- added C296: 1uF 50V X7R C2012X7R1H105K125AB, Capacitor_SMD:C_0805_2012Metric, symbol sr_rx_v2_completed:C_C296
- added C297: 1uF 50V X7R C2012X7R1H105K125AB, Capacitor_SMD:C_0805_2012Metric, symbol sr_rx_v2_completed:C_C297
- added C298: 47uF 50V EEUFR1H470, symbol sr_rx_v2_completed:C_C298
- added D2902: BZX84C10-7-F, Package_TO_SOT_SMD:SOT-23, symbol sr_rx_v2_completed:C_D2902
- added L208: 1uH XAL5030-102MEC, symbol sr_rx_v2_completed:C_L208
- added L210: 1uH XAL5030-102MEC, symbol sr_rx_v2_completed:C_L210
- added L215: 1uH XAL5030-102MEC, symbol sr_rx_v2_completed:C_L215
- added Q2902: DMP6050SSD-13, Package_SO:SOIC-8_3.9x4.9mm_P1.27mm, symbol sr_rx_v2_completed:C_Q2902
- added Q2912: 2N7002, Package_TO_SOT_SMD:SOT-23, symbol sr_rx_v2_completed:C_Q2912
- added R238: 88.7k 1%, symbol sr_rx_v2_completed:C_R238
- added R239: 100k 1%, symbol sr_rx_v2_completed:C_R239
- added R241: 0.200R 0.1% 0.25W Kelvin, symbol sr_rx_v2_completed:C_R241
- added R242: 0.22R 1% 0.25W, symbol sr_rx_v2_completed:C_R242
- added R248: RILIM TBD (start 56.2k 1%), symbol sr_rx_v2_completed:C_R248
- added R249: 100k 1%, symbol sr_rx_v2_completed:C_R249
- added R251: 0.22R 1% 0.25W, symbol sr_rx_v2_completed:C_R251
- added R268: 10.0R 1%, symbol sr_rx_v2_completed:C_R268
- added R269: 10.0R 1%, symbol sr_rx_v2_completed:C_R269
- added R270: 10.0R 1%, symbol sr_rx_v2_completed:C_R270
- added R271: 10.0R 1%, symbol sr_rx_v2_completed:C_R271
- added R272: 10.0R 1%, symbol sr_rx_v2_completed:C_R272
- added R273: 10.0R 1%, symbol sr_rx_v2_completed:C_R273
- added R274: 10.0R 1%, symbol sr_rx_v2_completed:C_R274
- added R275: 10.0R 1%, symbol sr_rx_v2_completed:C_R275
- added R276: 10.0R 1%, symbol sr_rx_v2_completed:C_R276
- added R277: 10.0R 1%, symbol sr_rx_v2_completed:C_R277
- added R278: 10.0R 1%, symbol sr_rx_v2_completed:C_R278
- added R279: 10.0R 1%, symbol sr_rx_v2_completed:C_R279
- added R2902: 220k 1%, Resistor_SMD:R_0603_1608Metric, symbol sr_rx_v2_completed:C_R2902
- added R2912: 4.7k 1% ≥0.25W, Resistor_SMD:R_1210_3225Metric, symbol sr_rx_v2_completed:C_R2912
- added R2922: 4.7k 1%, Resistor_SMD:R_0603_1608Metric, symbol sr_rx_v2_completed:C_R2922
- added R293: 162k 1%, symbol sr_rx_v2_completed:C_R293
- added R294: 100k 1%, symbol sr_rx_v2_completed:C_R294
- added R295: 0.22R 1%0.25W, symbol sr_rx_v2_completed:C_R295
- added TP208: BIAS_CH3, symbol sr_rx_v2_completed:C_TP208
- added TP210: VBUS_RTLB, symbol sr_rx_v2_completed:C_TP210
- added TP216: BIAS_SB_LNA, symbol sr_rx_v2_completed:C_TP216
- added TP2902: BIAS_CH3_PORT, symbol sr_rx_v2_completed:C_TP2902
- added U208: TPS2553DBVR-1, symbol sr_rx_v2_completed:C_U208
- added U210: TPS2553DBVR-1, symbol sr_rx_v2_completed:C_U210
- added U215: INA3221AIRGVR, symbol sr_rx_v2_completed:C_U215
- added U216: INA3221AIRGVR, symbol sr_rx_v2_completed:C_U216
- added U221: TPS2553DBVR-1, symbol sr_rx_v2_completed:C_U221
Connections:
- net E2_BONI_EF: now also R278.1
- net E2_BONI_MON: now also R279.1
- net E2_LNB_EF: now also R276.1
- net E2_LNB_MON: now also R277.1
- net GND: now also C240.2, C241.2, C242.2, C243.2 (-), C248.2, C249.2, C250.2, C251.2 (-), C277.2, C281.2, C2902.2, C295.2, C296.2, C297.2, C298.2 (-), Q2912.2 (S), R238.2, R239.2, R248.2, R249.2, R2922.2, R293.2, R294.2, U208.2 (GND), U210.2 (GND), U215.3 (GND), U215.EP, U216.3 (GND), U216.EP, U221.2 (GND)
- new net 3V3_Q6A: C277.1, C281.1, U215.16 (VPU), U215.4 (VS), U215.5 (A0), U216.16 (VPU), U216.4 (VS)
- new net BIAS_CH3: C242.1, L208.2, Q2902.7 (D1), Q2902.8 (D1), R242.1, R2922.1, TP208.1 (TP)
- new net BIAS_CH3_DAMP: C243.1 (+), R242.2
- new net BIAS_CH3_PORT: C2902.1, Q2902.5 (D2), Q2902.6 (D2), TP2902.1 (TP)
- new net BIAS_SB_LNA: C297.1, L215.2, R295.1, TP216.1 (TP)
- new net E2_BLK3_G: C2912.2, D2902.1 (A), Q2902.2 (G1), Q2902.4 (G2), R2902.2, R2912.1
- new net E2_BLK3_S: C2912.1, D2902.3 (K), Q2902.1 (S1), Q2902.3 (S2), R2902.1
- new net E2_BLK3_SINK: Q2912.3 (D), R2912.2
- new net E2_LNA1_SHUNT: R269.1
- new net E2_LNA1_SW: R268.1
- new net E2_LNA2_SHUNT: R271.1
- new net E2_LNA2_SW: R270.1
- new net E2_LNA3_SHUNT: C241.1, L208.1, R241.2, R273.1
- new net E2_LNA3_SW: R241.1, R272.1, U208.6 (OUT)
- new net E2_LNA4_SHUNT: R275.1
- new net E2_LNA4_SW: R274.1
- new net E2_RTLB_SW: C249.1, L210.1, U210.6 (OUT)
- new net E2_SB_DAMP: C298.1 (+), R295.2
- new net E2_SB_ILIM: R293.1, U221.5 (ILIM)
- new net E2_SB_SW: C296.1, L215.1, U221.6 (OUT)
- new net E2_U208_ILIM: R238.1, U208.5 (ILIM)
- new net E2_U210_ILIM: R248.1, U210.5 (ILIM)
- new net E2_U215_IM1: C274.2, R269.2, U215.11 (IN-1)
- new net E2_U215_IM2: C275.2, R271.2, U215.14 (IN-2)
- new net E2_U215_IM3: C276.2, R273.2, U215.1 (IN-3)
- new net E2_U215_IP1: C274.1, R268.2, U215.12 (IN+1)
- new net E2_U215_IP2: C275.1, R270.2, U215.15 (IN+2)
- new net E2_U215_IP3: C276.1, R272.2, U215.2 (IN+3)
- new net E2_U216_IM1: C278.2, R275.2, U216.11 (IN-1)
- new net E2_U216_IM2: C279.2, R277.2, U216.14 (IN-2)
- new net E2_U216_IM3: C280.2, R279.2, U216.1 (IN-3)
- new net E2_U216_IP1: C278.1, R274.2, U216.12 (IN+1)
- new net E2_U216_IP2: C279.1, R276.2, U216.15 (IN+2)
- new net E2_U216_IP3: C280.1, R278.2, U216.2 (IN+3)
- new net EN_LNA3: Q2912.1 (G), R239.1, U208.3 (EN)
- new net EN_RTLB: R249.1, U210.3 (EN)
- new net EN_SB_LNA: R294.1, U221.3 (EN)
- new net FAULT_LNA3: U208.4 (FAULT)
- new net FAULT_RTLB: U210.4 (FAULT)
- new net FLT_SB_LNA: U221.4 (FAULT)
- new net I2C2_SCL: U215.6 (SCL), U216.5 (A0), U216.6 (SCL)
- new net I2C2_SDA: U215.7 (SDA), U216.7 (SDA)
- new net LAB5: C248.1, C295.1, U210.1 (IN), U221.1 (IN)
- new net LNA4V5: C240.1, U208.1 (IN)
- new net VBUS_RTLB: C250.1, L210.2, R251.1, TP210.1 (TP)
- new net VBUS_RTLB_DAMP: C251.1 (+), R251.2
- no-connect marks 14 -> 9
Other:
- note added: "E2 - Захищені рейки, LNA і моніторинг струму (3/5)"
- note added: "E2-03 — OPEN, блокує випуск — STACK §5.1 (VBUS RTL-B, BONI13V8); §8 (струми; TPS2553DBVR-1 п. 3); §8.1 RF-2, HF-8/RF-5"
- note added: "INA3221: струми LNA1–3"
- note added: "INA3221: струми LNA4, LNB і Boni"
- note added: "LNA: канал 3"
- note added: "N-E2-01 — примітка — STACK §5.1 (VBUS RTL-B); §8 (TPS2553DBVR-1 п. 3)"
- note added: "R248 = RILIM TBD (старт 56.2k 1%, ≈0.47 A ном.). STACK не задає номінал для VBUS RTL-B, лише правило: RILIM = 1.5–2× виміряного струму. Ворота: E2-03 (20 холодних і теплих пусків, пусковий струм до deglitch 5 ms)."
- note added: "RTL-B: комутований VBUS"
- note added: "S-band LaNA WB: захищена шина 5 V"
- note added: "Остаточні ILIM і пускові струми RTL-B, Lime, LNB, Boni та LaNA WB потребують натурних вимірів; ємність riser і комерційних модулів не опублікована. Поріг OVLO Boni (R263/R264, стартовий розрахунок 112k/10.0k) STACK §5.1 вимагає перерахувати для 13.8 V; на стенді його не перевірено. Ворота (стенд): FNB58/INA228/INA3221: 20 холодних і теплих пусків, струми стримінгу, КЗ і SOA. Установити ILIM 1.5–2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"
- note removed: "Boni: малошумна захищена шина"
- note removed: "E2 - Захищені рейки, LNA і моніторинг струму (3/4)"
- note removed: "E2-02 — OPEN, блокує випуск — STACK §5.1 (LNB13V2); §8 (TPS7A4701); §8.1 RF-4"
- note removed: "LNB: малошумна захищена шина"
- note removed: "N-E2-02 — примітка — STACK §5.1 (BONI13V8); §8.1 HF-8/RF-5"
- note removed: "R263/R264 = OVLO TBD (старт 112k/10.0k 0.1%: 14.64 V ном., ≈14.24–14.92 V за R-E2-02). STACK §5.1 (BONI13V8): «OVLO перерахувати для 13.8 V» — номіналу в STACK немає. Ворота: E2-03 (стенд STACK §8.1 HF-8/RF-5: OVLO не спрацьовує в смузі 13.8 V; поріг вище 14.145 V і нижче 15 V)."
- note removed: "Статичне вікно OVP LNB закрито TPS3701: 13.56–13.96V. Швидкий викид при відмові LDO не обмежено гарантованим максимальним часом у даташитах: 9.9µs компаратора і близько 12µs EN-off eFuse задані лише типово. Ворота (стенд): Без LNB і зі струмовим обмеженням подати на вузол LDO контрольований стрибок 13.2→16.4V; осцилографувати F-вихід при мін./макс. навантаженні, на холоді й при 50°C. Отримати гра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"
- title: E2 - Захищені рейки, LNA і моніторинг струму (3/4) -> E2 - Захищені рейки, LNA і моніторинг струму (3/5)

Commit message: GENERATED: CAD, documents, verification reports, DC_CORE re-freeze and module-lab inventory for f3f57e8
Applied unchanged from the cad-regenerated artifact of CI run 40109759054
(workflow_dispatch, refreeze_pcb=true, KiCad 10.0.7): schematics, SVG, PDF,
netlist, OPEN_ITEMS.md, COMPLETION.md, verification/{electrical-invariants,
independent-netlist-review,netlist,pcb-review,pcb-prototype-review,
pdf-export,validation}, pcb/generated and the re-frozen DC_CORE starter and
routed prototype with their pinned hashes. Inputs: the stage 3A merge,
design/E2.json (PICO-2 text) and STACK.md (2.7 row).

deployment/module_lab/inventory.json: source_snapshots only, from
deployment/module_lab/refresh_inventory.py (E2.json and STACK.md bytes).

Co-Authored-By: Claude Opus 5.5 <noreply@anthropic.com>
Parts:
- removed C278: 100nF 50V X7R C1608X7R1H104K080AA, Capacitor_SMD:C_0603_1608Metric, symbol sr_rx_v2_completed:C_C278
- removed C279: 100nF 50V X7R C1608X7R1H104K080AA, Capacitor_SMD:C_0603_1608Metric, symbol sr_rx_v2_completed:C_C279
- removed C280: 100nF 50V X7R C1608X7R1H104K080AA, Capacitor_SMD:C_0603_1608Metric, symbol sr_rx_v2_completed:C_C280
- removed C281: 100nF 50V X7R C1608X7R1H104K080AA, Capacitor_SMD:C_0603_1608Metric, symbol sr_rx_v2_completed:C_C281
- removed R274: 10.0R 1%, symbol sr_rx_v2_completed:C_R274
- removed R275: 10.0R 1%, symbol sr_rx_v2_completed:C_R275
- removed R276: 10.0R 1%, symbol sr_rx_v2_completed:C_R276
- removed R277: 10.0R 1%, symbol sr_rx_v2_completed:C_R277
- removed R278: 10.0R 1%, symbol sr_rx_v2_completed:C_R278
- removed R279: 10.0R 1%, symbol sr_rx_v2_completed:C_R279
- removed U216: INA3221AIRGVR, symbol sr_rx_v2_completed:C_U216
- added C244: 1uF 50V X7R C2012X7R1H105K125AB, Capacitor_SMD:C_0805_2012Metric, symbol sr_rx_v2_completed:C_C244
- added C245: 1uF 50V X7R C2012X7R1H105K125AB, Capacitor_SMD:C_0805_2012Metric, symbol sr_rx_v2_completed:C_C245
- added C246: 1uF 50V X7R C2012X7R1H105K125AB, Capacitor_SMD:C_0805_2012Metric, symbol sr_rx_v2_completed:C_C246
- added C247: 47uF 50V EEUFR1H470, symbol sr_rx_v2_completed:C_C247
- added L209: 1uH XAL5030-102MEC, symbol sr_rx_v2_completed:C_L209
- added R243: 162k 1%, symbol sr_rx_v2_completed:C_R243
- added R244: 100k 1%, symbol sr_rx_v2_completed:C_R244
- added R246: 0.200R 0.1% 0.25W Kelvin, symbol sr_rx_v2_completed:C_R246
- added R247: 0.22R 1% 0.25W, symbol sr_rx_v2_completed:C_R247
- added TP209: BIAS_CH4, symbol sr_rx_v2_completed:C_TP209
- added U209: TPS2553DBVR-1, symbol sr_rx_v2_completed:C_U209
Connections:
- net E2_LNA4_SHUNT: now also C245.1, L209.1, R246.2
- net E2_LNA4_SW: now also R246.1, U209.6 (OUT)
- net GND: now also C244.2, C245.2, C246.2, C247.2 (-), R243.2, R244.2, U209.2 (GND)
- net LNA4V5: now also C244.1, U209.1 (IN)
- new net BIAS_CH4: C246.1, L209.2, R247.1, TP209.1 (TP)
- new net BIAS_CH4_DAMP: C247.1 (+), R247.2
- new net E2_U209_ILIM: R243.1, U209.5 (ILIM)
- new net EN_LNA4: R244.1, U209.3 (EN)
- new net FAULT_LNA4: U209.4 (FAULT)
- no-connect marks 9 -> 5
Other:
- note added: "LNA: канал 4"
- note removed: "INA3221: струми LNA4, LNB і Boni"
- moved on the sheet: C248, C249, C250, C251, C274, C275, C276, C277, C295, C296, C297, C298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
