File: sat-receiver-audit/build/kicad/E3_02.kicad_sch (KiCad schematic)
At the start: 56 parts, among them Q302 2N7002, SW301 Power button momentary NO, SW302 HOME momentary NO, SW303 BACK momentary NO, SW304 REC momentary NO, SW305 MARK momentary NO, SW306 FN momentary NO, SW307 LOCK momentary NO, SW308 ENC1_PRESS momentary NO, SW309 ENC2_PRESS momentary NO, U306 PI4IOE5V9555LEX 0x20, U307 LM4040C30IDBZR, U310 TPD4E1U06DBVR, U311 TPD4E1U06DBVR

Commit message: SR-RX-v2.1: review fixes on the Codex branch, readable schematic, one-file bundle
Independent review of the Codex branch (schematic vs STACK.md, hard rules,
security, tests) found no blockers; this commit applies its findings:

- rules in code: Cospas-Sarsat 406.0-406.1 MHz added to the no-data mask;
  Q6A Wi-Fi/BT off in the field/QUIET root (modprobe blacklist, udev
  authorized=0 on FE1.1s port 4, rfkill) with self-checks; device denylist
  completed per STACK (gr-gsm, gr-iridium, kalibrate, pager/trunking decoders,
  TX-capable tools); W1-2 WIFI_PWR_EN as blocking open item E5-10
- STACK.md is the source of truth again; v2.1 changes recorded in it; the
  "historical" marker kept only on ISDT/raw-balance rows; gender-neutral wording
- schematic data: open values shown as TBD with start values and notes, U503
  TPS2553DBVR-1, Lime X2/X4 RX mapping TBD, 37 open items drawn on the sheets
- schematic readability: wired groups, junctions, GND symbols, standard
  transistor/diode symbols; netlist unchanged (603 nets identical)
- tooling: reproducible run_checks (no timestamps or machine paths), pinned
  dependencies, bundle excludes cache folders, clean-checkout bundle check
- regenerated: KiCad export (14 pages), netlist/ERC, module lab, PCB inputs,
  readiness contract, acceptance hashes, SR-RX-v2-ves-proekt.html

Checks: ERC 0 errors/0 warnings, netlist comparison PASS, 432 tests (431
passed, 1 skipped), deployment tests OK, bundle check PASS on a clean checkout.

History note: earlier versions of the generated SR-RX-v2-ves-proekt.html and
handoff/handoff-bundle.zip were removed from history; only the final versions
are kept. The Codex merge commit is now attributed to Codex.

Co-Authored-By: Claude Opus 5.5 <noreply@anthropic.com>
Claude-Session: https://claude.ai/code/session_01W9CKpimWpgkUmrDQQMiKtF
Parts:
- removed C310: 100n 16V, symbol sr_rx_v2_completed:C_C310
- removed C311: 100n 16V, symbol sr_rx_v2_completed:C_C311
- removed C312: 100n 16V, symbol sr_rx_v2_completed:C_C312
- removed C313: 1u 10V, symbol sr_rx_v2_completed:C_C313
- removed R332: 10k 1%, symbol sr_rx_v2_completed:C_R332
- removed R333: 10k 1%, symbol sr_rx_v2_completed:C_R333
- removed R334: 10k, symbol sr_rx_v2_completed:C_R334
- removed R335: 2.2k, symbol sr_rx_v2_completed:C_R335
- removed R336: 100, symbol sr_rx_v2_completed:C_R336
- removed R337: 2.2k, symbol sr_rx_v2_completed:C_R337
- removed R338: 100, symbol sr_rx_v2_completed:C_R338
- removed R339: 2.2k, symbol sr_rx_v2_completed:C_R339
- removed R340: 100, symbol sr_rx_v2_completed:C_R340
- removed R341: 2.2k, symbol sr_rx_v2_completed:C_R341
- removed R342: 100, symbol sr_rx_v2_completed:C_R342
- removed R343: 2.2k, symbol sr_rx_v2_completed:C_R343
- removed R344: 100, symbol sr_rx_v2_completed:C_R344
- removed R345: 2.2k, symbol sr_rx_v2_completed:C_R345
- removed R346: 100, symbol sr_rx_v2_completed:C_R346
- removed R347: 2.2k, symbol sr_rx_v2_completed:C_R347
- removed R348: 100, symbol sr_rx_v2_completed:C_R348
- removed R349: 2.2k, symbol sr_rx_v2_completed:C_R349
- removed R350: 100, symbol sr_rx_v2_completed:C_R350
- removed SW302: HOME momentary NO, symbol sr_rx_v2_completed:C_SW302
- removed SW303: BACK momentary NO, symbol sr_rx_v2_completed:C_SW303
- removed SW304: REC momentary NO, symbol sr_rx_v2_completed:C_SW304
- removed SW305: MARK momentary NO, symbol sr_rx_v2_completed:C_SW305
- removed SW306: FN momentary NO, symbol sr_rx_v2_completed:C_SW306
- removed SW307: LOCK momentary NO, symbol sr_rx_v2_completed:C_SW307
- removed SW308: ENC1_PRESS momentary NO, symbol sr_rx_v2_completed:C_SW308
- removed SW309: ENC2_PRESS momentary NO, symbol sr_rx_v2_completed:C_SW309
- removed TH301: Semiware MF52A103F3950, symbol sr_rx_v2_completed:C_TH301
- removed TH302: Semiware MF52A103F3950, symbol sr_rx_v2_completed:C_TH302
- removed U306: PI4IOE5V9555LEX 0x20, Package_SO:TSSOP-24_4.4x7.8mm_P0.65mm, symbol sr_rx_v2_completed:C_U306
- removed U310: TPD4E1U06DBVR, Package_TO_SOT_SMD:SOT-23-6, symbol sr_rx_v2_completed:C_U310
- removed U311: TPD4E1U06DBVR, Package_TO_SOT_SMD:SOT-23-6, symbol sr_rx_v2_completed:C_U311
- added BZ301: CPT-1207-3TH, symbol sr_rx_v2_completed:C_BZ301
- added C307: 10u 10V, symbol sr_rx_v2_completed:C_C307
- added C308: 100n 16V, symbol sr_rx_v2_completed:C_C308
- added C316: 10n 16V, symbol sr_rx_v2_completed:C_C316
- added C317: 10n 16V, symbol sr_rx_v2_completed:C_C317
- added C318: 10u 10V, symbol sr_rx_v2_completed:C_C318
- added C319: 100n 16V, symbol sr_rx_v2_completed:C_C319
- added C320: 10u 10V, symbol sr_rx_v2_completed:C_C320
- added C342: 10u 10V, symbol sr_rx_v2_completed:C_C342
- added C343: 100n 16V, symbol sr_rx_v2_completed:C_C343
- added D301: SS14, Diode_SMD:D_SMA, symbol sr_rx_v2_completed:C_D301
- added D304: WP7113LSECK/J3 red, symbol sr_rx_v2_completed:C_D304
- added D305: SS14 flyback, Diode_SMD:D_SMA, symbol sr_rx_v2_completed:C_D305
- added D306: SS14 flyback, Diode_SMD:D_SMA, symbol sr_rx_v2_completed:C_D306
- added ENC302: PEC11R-4220F encoder, symbol sr_rx_v2_completed:C_ENC302
- added FAN301: NoctuaNF-A4x10 5V nonPWM, symbol sr_rx_v2_completed:C_FAN301
- added FAN302: Delta BFB0305HA-C 5V 2wire, symbol sr_rx_v2_completed:C_FAN302
- added J301: Q6A J20 2x20 3.3V GPIO, symbol sr_rx_v2_completed:C_J301
- added J302: Power-board control harness DESIGN, symbol sr_rx_v2_completed:C_J302
- added Q301: 2N7002, Package_TO_SOT_SMD:SOT-23, symbol sr_rx_v2_completed:C_Q301
- added Q303: AO3400A, Package_TO_SOT_SMD:SOT-23, symbol sr_rx_v2_completed:C_Q303
- added Q304: AO3401A, Package_TO_SOT_SMD:SOT-23, symbol sr_rx_v2_completed:C_Q304
- added Q305: AO3400A, Package_TO_SOT_SMD:SOT-23, symbol sr_rx_v2_completed:C_Q305
- added R301: 10k, symbol sr_rx_v2_completed:C_R301
- added R302: 10k, symbol sr_rx_v2_completed:C_R302
- added R303: 10k DNP, symbol sr_rx_v2_completed:C_R303
- added R304: 10k DNP, symbol sr_rx_v2_completed:C_R304
- added R326: 100k, symbol sr_rx_v2_completed:C_R326
- added R357: 10k, symbol sr_rx_v2_completed:C_R357
- added R358: 10k, symbol sr_rx_v2_completed:C_R358
- added R359: 100, symbol sr_rx_v2_completed:C_R359
- added R360: 100, symbol sr_rx_v2_completed:C_R360
- added R361: 4.7k, symbol sr_rx_v2_completed:C_R361
- added R362: 4.7k, symbol sr_rx_v2_completed:C_R362
- added R363: 150, symbol sr_rx_v2_completed:C_R363
- added R364: 680, symbol sr_rx_v2_completed:C_R364
- added R365: 100, symbol sr_rx_v2_completed:C_R365
- added R366: 100k, symbol sr_rx_v2_completed:C_R366
- added R367: 100k, symbol sr_rx_v2_completed:C_R367
- added R368: 10k, symbol sr_rx_v2_completed:C_R368
- added R369: 2.2k, symbol sr_rx_v2_completed:C_R369
- added R370: 100, symbol sr_rx_v2_completed:C_R370
- added R371: 100k, symbol sr_rx_v2_completed:C_R371
- added U304: Waveshare LC76G GNSS 24370, symbol sr_rx_v2_completed:C_U304
- added U305: Raspberry Pi Pico SC0915, symbol sr_rx_v2_completed:C_U305
- added U308: Adafruit4162 VEML7700 0x10, symbol sr_rx_v2_completed:C_U308
- added U312: TPD4E1U06DBVR, Package_TO_SOT_SMD:SOT-23-6, symbol sr_rx_v2_completed:C_U312
- added U313: TPD4E1U06DBVR, Package_TO_SOT_SMD:SOT-23-6, symbol sr_rx_v2_completed:C_U313
Connections:
- net 3V3_Q6A: now also J301.1 (3V3), J301.17 (3V3), J302.1 (3V3_Q6A), R301.2, R302.2, R303.2, R304.2
- net E3_ADC3V0: now also U305.35 (ADC_VREF)
- net E3_BUTTON_SENSE: now also U305.15 (GP11)
- net E3_CASE_TEMP: now also U305.34 (GP28)
- net E3_ENC1_A: now also U305.4 (GP2)
- net E3_ENC1_A_RAW: now also U312.1 (D1+)
- net E3_ENC1_B: now also U305.5 (GP3)
- net E3_ENC1_B_RAW: now also U312.3 (D2+)
- net E3_ENC2_A: now also C316.1, U305.9 (GP6)
- net E3_ENC2_A_RAW: now also ENC302.A, U312.4 (D2-)
- net E3_HMI_INT: now also U305.14 (GP10)
- net E3_HMI_SCL: now also R360.1, R362.1, U305.7 (GP5)
- net E3_HMI_SDA: now also R359.1, R361.1, U305.6 (GP4)
- net E3_PANEL_TEMP: now also U305.31 (GP26)
- net E3_PICO3V3: now also C308.1, R357.2, R361.2, R362.2, R368.2, U305.36 (3V3_OUT), U308.VIN
- net E3_Q6A_KEY_GATE: now also U305.16 (GP12)
- net E3_Q6A_ON_SENSE: now also U305.19 (GP14)
- net GND: now also BZ301.- (MINUS), C307.2, C308.2, C316.2, C317.2, C318.2, C319.2, C320.2, D304.K, D305.2 (A), ENC302.C (COMMON), FAN301.GND, J301.14 (GND), J301.20 (GND), J301.25 (GND), J301.30 (GND), J301.34 (GND), J301.39 (GND), J301.6 (GND), J301.9 (GND), J302.2 (GND), Q301.2 (S), Q303.2 (S), Q305.2 (S), R326.2, R366.2, R371.2, U304.GPS1.1 (GND), U304.GPS1.3 (GND), U304.GPS1.4 (GND), U304.P1.2 (GND), U305.13 (GND), U305.18 (GND), U305.23 (GND), U305.28 (GND), U305.3 (GND), U305.33 (GND), U305.38 (GND), U305.8 (GND), U305.SWD_GND, U308.GND, U312.2 (GND), U313.2 (GND)
- new net E1_BAT_ADC: U305.32 (GP27)
- new net E3_BEZEL_SCL: R360.2, U308.SCL, U313.3 (D2+)
- new net E3_BEZEL_SDA: R359.2, U308.SDA, U313.1 (D1+)
- new net E3_BLOWER_EN: R370.1, U305.25 (GP19)
- new net E3_BLOWER_GATE: Q305.1 (G), R370.2, R371.1
- new net E3_BLOWER_GND: C342.2, C343.2, D306.2 (A), FAN302.BLACK (BLACK_MINUS), Q305.3 (D)
- new net E3_ENC2_B: C317.1, R358.2, U305.10 (GP7)
- new net E3_ENC2_B_RAW: ENC302.B, R357.1, R358.1, U312.6 (D1-)
- new net E3_FAN5: C318.1, C319.1, D305.1 (K), FAN301.V+ (+5V), Q304.3 (D)
- new net E3_FAN_EN: R365.1, U305.24 (GP18)
- new net E3_FAN_NG: Q303.1 (G), R365.2, R366.1
- new net E3_FAN_PG: Q303.3 (D), Q304.1 (G), R367.1
- new net E3_FAN_TACH: R369.2, U305.29 (GP22)
- new net E3_FAN_TACH_RAW: FAN301.TACH, R368.1, R369.1
- new net E3_GNSS_PPS: J301.7 (GPIO96), U304.P1.5 (1PPS)
- new net E3_GNSS_RESET_GATE: Q301.1 (G), R326.1
- new net E3_GNSS_RESET_N: Q301.3 (D), U304.P1.6 (RESET_N)
- new net E3_LED_A: D304.A, R364.2
- new net E3_LED_DRIVE: R364.1, U305.27 (GP21)
- new net E3_MCP_RESET_ASSERT: U305.22 (GP17)
- new net E3_PICO_RUN: J301.38 (GPIO98_RUN), U305.30 (RUN)
- new net E3_PICO_SWCLK: J301.12 (GPIO97_SWCLK), U305.SWCLK
- new net E3_PICO_SWDIO: J301.35 (GPIO100_SWDIO), U305.SWDIO
- new net E3_PICO_VSYS: C307.1, D301.1 (K), U305.39 (VSYS)
- new net E3_PIEZO_DRIVE: R363.1, U305.26 (GP20)
- new net E3_PIEZO_OUT: BZ301.+ (PLUS), R363.2
- new net GNSS_ANT: U304.GPS1.2 (ANT)
- new net I2C0_SCL: J301.15 (GPIO1_I2C0_SCL)
- new net I2C0_SDA: J301.13 (GPIO0_I2C0_SDA)
- new net I2C2_SCL: J301.28 (GPIO9_I2C2_SCL), J302.4 (SCL), R304.1
- new net I2C2_SDA: J301.27 (GPIO8_I2C2_SDA), J302.3 (SDA), R303.1
- new net IMU_RX: U305.11 (GP8)
- new net IMU_TX: U305.12 (GP9)
- new net INA228_ALERT: J301.3 (GPIO24), R301.1
- new net LAB5: C320.1, C342.1, C343.1, D301.2 (A), D306.1 (K), FAN302.RED (RED_PLUS), Q304.2 (S), R367.2
- new net MCP_INT: J301.5 (GPIO25), J302.5 (INT), R302.1
- new net PICO_DISP_EN: U305.21 (GP16)
- new net PICO_OFF: U305.17 (GP13)
- new net SAFE_BOOT: J301.40 (GPIO99_SAFE_BOOT), U305.20 (GP15)
- new net UART5_RX: J301.10 (GPIO23_UART5_RX)
- new net UART5_TX: J301.8 (GPIO22_UART5_TX)
- new net UART6_RX: J301.18 (GPIO27_UART6_RX), U304.P1.3 (TXD)
- new net UART6_TX: J301.16 (GPIO26_UART6_TX), U304.P1.4 (RXD)
- new net UART7_RX: J301.29 (GPIO31_UART7_RX), U305.1 (GP0)
- new net UART7_TX: J301.32 (GPIO30_UART7_TX), U305.2 (GP1)
- new net VCC_5V_PERI: J301.2 (5V), J301.4 (5V), U304.P1.1 (VCC)
- no-connect marks 12 -> 22
Other:
- note added: "Ambient sensor"
- note added: "BOM candidate Delta BFB0305HA-C is selected; final mechanical fit, installed airflow, start/stall current, LAB5 concurrency and noise remain unqualified. Ворота (стенд): Fit the body envelope 30.5x30.5x10.5 mm plus duct/lead clearance into CAD before cutting the enclosure. Measure the 0.25 A design continuous reserve and the provisional 0.50 A startup limit rather than claiming peak from the data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"
- note added: "Battery ADC shutdown accuracy must be calibrated. Divider/reference initial tolerances can contribute about +/-0.28 V near 12.9 V; a nominal ADC code does not establish the 12.9 +/-0.1 V cutoff. Ворота (стенд): Calibrate gain/offset against a calibrated voltmeter at two pack-equivalent voltages such as 12.6 V and 16.4 V; cross-check INA228. Independently verify the physical 12.9 V software cutoff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"
- note added: "Brightness control requires confirmed DDC/CI support or an exact Wisecoco KEY/Backlight interface. Pico GP17 is now reserved for MCP watchdog reset and unavailable for brightness. Ворота (стенд): Demonstrate ddcutil brightness through the specified RA620 link, or obtain the exact KEY/Backlight revision pinout and design a new interface using a free MCP GPIO if suitable. Verify thermal dimming; do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"
- note added: "Cooling"
- note added: "E3 - Керування, Pico HMI, GPIO, GNSS і IMU (2/2)"
- note added: "E3-02 — OPEN, блокує випуск — STACK §2.6; §5.2; §8.1 (шлях димінгу)"
- note added: "E3-03 — OPEN, блокує випуск — STACK §5.6; §8 (тепло); §8.1 (потік повітря)"
- note added: "E3-04 — OPEN, блокує випуск — STACK §5.2 (UART7, PPS, SWD); §8.1 (UART7; PPS)"
- note added: "E3-07 — OPEN, блокує випуск — STACK §5.1; §5.2; §8 (Pico ADC)"
- note added: "GNSS"
- note added: "Indicators"
- note added: "Q6A header"
- note added: "UM3304 UART7/PPS/SWD cable capacitance and power-off behavior cannot be proven by ERC. Ворота (стенд): Check <=20cm wiring, UART7 loopback, boot glitches and absence of Q6A backfeed with Pico on/Q6A off. Verify TX high-impedance sequencing or add hardware isolation."
- note added: "Дроти з'єднують контакти всередині функціональної групи; кожне дерево дротів має одну глобальну мітку з канонічною назвою мережі (рамка-стрілка — мережа виходить за межі групи, пряма рамка — мережа лише цієї групи). Однакові мітки з'єднані на всіх аркушах; земля — символ GND. Рамки OPEN — незакриті ворота з design/E#.json (повний реєстр: OPEN_ITEMS.md); «TBD» у значенні — STACK номіналу не задає,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"
- note removed: "E3 - Керування, Pico HMI, GPIO, GNSS і IMU (2/3)"
- note removed: "HMI buttons"
- note removed: "Thermal sensors"
- note removed: "Мережі з однаковими глобальними мітками електрично з'єднані на всіх аркушах. Фізичні/функціональні контакти: див. design/ і OPEN_ITEMS.md."
- title: E3 - Керування, Pico HMI, GPIO, GNSS і IMU (2/3) -> E3 - Керування, Pico HMI, GPIO, GNSS і IMU (2/2)
- moved on the sheet: ENC301, U307
