File: sat-receiver-audit/build/kicad/E3_02.kicad_sch (KiCad schematic)
At the start: 68 parts, among them J301 Q6A J20 2x20 3.3V GPIO, J302 Power-board control harness D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, Q301 2N7002, Q302 2N7002, Q303 AO3400A, Q304 AO3401A, Q305 AO3400A, SW301 Power button momentary NO, U304 Waveshare LC76G GNSS 24370, U305 Raspberry Pi Pico SC0915, U307 LM4040C30IDBZR, U308 Adafruit4162 VEML7700 0x10, U312 TPD4E1U06DBVR, U313 TPD4E1U06DBVR

Commit message: Stage 2 integration: CAD and DC_CORE re-freeze from CI run 40094234222; bound-count test and PCB hash lists follow
Co-Authored-By: Claude Opus 5.5 <noreply@anthropic.com>
Parts:
- removed D302: BAT54, Package_TO_SOT_SMD:SOT-23, symbol sr_rx_v2_completed:C_D302
- removed D303: BAT54, Package_TO_SOT_SMD:SOT-23, symbol sr_rx_v2_completed:C_D303
- removed J301: Q6A J20 2x20 3.3V GPIO, symbol sr_rx_v2_completed:C_J301
- removed J302: Power-board control harness DESIGN, symbol sr_rx_v2_completed:C_J302
- removed Q302: 2N7002, Package_TO_SOT_SMD:SOT-23, symbol sr_rx_v2_completed:C_Q302
- removed R301: 10k, symbol sr_rx_v2_completed:C_R301
- removed R302: 10k, symbol sr_rx_v2_completed:C_R302
- removed R303: 10k DNP, symbol sr_rx_v2_completed:C_R303
- removed R304: 10k DNP, symbol sr_rx_v2_completed:C_R304
- removed R330: 10k, symbol sr_rx_v2_completed:C_R330
- removed R331: 100k, symbol sr_rx_v2_completed:C_R331
- removed SW301: Power button momentary NO, symbol sr_rx_v2_completed:C_SW301
- added C340: 10u 10V, symbol sr_rx_v2_completed:C_C340
- added C341: 100n 16V, symbol sr_rx_v2_completed:C_C341
- added R390: 10k, symbol sr_rx_v2_completed:C_R390
- added R391: 1k, symbol sr_rx_v2_completed:C_R391
- added U309: Waveshare RP2040-Zero 20187, symbol sr_rx_v2_completed:C_U309
- added U314: Adafruit 4754 BNO085 SPI, symbol sr_rx_v2_completed:C_U314
Connections:
- net GND: now also C340.2, C341.2, U309.GND, U314.GND
- net IMU_RX: now also U309.GP1
- net IMU_TX: now also U309.GP0
- new net E3_IMU3V3: C341.1, R390.2, R391.2, U309.3V3 (3V3_OUT), U314.P1 (PS1), U314.VIN
- new net E3_IMU_CS_N: R390.1, U309.GP5, U314.CS (CS_N)
- new net E3_IMU_INT_N: U309.GP6, U314.INT (INT_N)
- new net E3_IMU_MISO: U309.GP4, U314.SDA (SDA_SPI_MISO)
- new net E3_IMU_MOSI: U309.GP3, U314.DI (DI_SPI_MOSI)
- new net E3_IMU_RST_N: U309.GP7, U314.RST (RST_N)
- new net E3_IMU_SCK: U309.GP2, U314.SCL (SCL_SPI_SCK)
- new net E3_IMU_WAKE_N: R391.1, U309.GP8, U314.P0 (PS0)
- new net E5_IMU_VIN: C340.1, U309.5V (5V_IN)
- no-connect marks 22 -> 31
Other:
- note added: "E3-01 — OPEN, блокує випуск — STACK §2.8; §5.2; §8 (пак IMU); §8.1 (пак IMU)"
- note added: "External IMU"
- note added: "IMU assembly and two metre single-ended UART need bench verification. Internal named-pad wiring is specified, but no physical harness has been measured. Ворота (стенд): Check actual module revision, GX16 plug/socket viewing direction and continuity to E5 design pinout; validate input Schottky and TVS at both ends; 1e6 frames with zero CRC errors. Upgrade to differential interface if errors occur."
- note removed: "E3-04 — OPEN, блокує випуск — STACK §5.2 (UART7, PPS, SWD); §8.1 (UART7; PPS)"
- note removed: "Pico power control"
- note removed: "Q6A header"
- note removed: "UM3304 UART7/PPS/SWD cable capacitance and power-off behavior cannot be proven by ERC. Ворота (стенд): Check <=20cm wiring, UART7 loopback, boot glitches and absence of Q6A backfeed with Pico on/Q6A off. Verify TX high-impedance sequencing or add hardware isolation."
- moved on the sheet: BZ301, C314, C315, C316, C317, D304, ENC301, ENC302, Q301, R326, R351, R352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
