File: sat-receiver-audit/build/kicad/E4_03.kicad_sch (KiCad schematic)
At the start: 53 parts, among them Q450 AO3400A, Q451 AO3400A, Q456 AO3400A, Q457 AO3400A, U405 HMC7992LP3DE A, U406 HMC7992LP3DE B, U407 HMC7992LP3DE C, U450 TLV3012BIDBVR, U451 TLV3012BIDBVR, U456 TLV3012BIDBVR, U457 TLV3012BIDBVR, U458 LM4040A20IDBZR 2.048 V 0.1% s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

Commit message: SR-RX-v2.1: review fixes on the Codex branch, readable schematic, one-file bundle
Independent review of the Codex branch (schematic vs STACK.md, hard rules,
security, tests) found no blockers; this commit applies its findings:

- rules in code: Cospas-Sarsat 406.0-406.1 MHz added to the no-data mask;
  Q6A Wi-Fi/BT off in the field/QUIET root (modprobe blacklist, udev
  authorized=0 on FE1.1s port 4, rfkill) with self-checks; device denylist
  completed per STACK (gr-gsm, gr-iridium, kalibrate, pager/trunking decoders,
  TX-capable tools); W1-2 WIFI_PWR_EN as blocking open item E5-10
- STACK.md is the source of truth again; v2.1 changes recorded in it; the
  "historical" marker kept only on ISDT/raw-balance rows; gender-neutral wording
- schematic data: open values shown as TBD with start values and notes, U503
  TPS2553DBVR-1, Lime X2/X4 RX mapping TBD, 37 open items drawn on the sheets
- schematic readability: wired groups, junctions, GND symbols, standard
  transistor/diode symbols; netlist unchanged (603 nets identical)
- tooling: reproducible run_checks (no timestamps or machine paths), pinned
  dependencies, bundle excludes cache folders, clean-checkout bundle check
- regenerated: KiCad export (14 pages), netlist/ERC, module lab, PCB inputs,
  readiness contract, acceptance hashes, SR-RX-v2-ves-proekt.html

Checks: ERC 0 errors/0 warnings, netlist comparison PASS, 432 tests (431
passed, 1 skipped), deployment tests OK, bundle check PASS on a clean checkout.

History note: earlier versions of the generated SR-RX-v2-ves-proekt.html and
handoff/handoff-bundle.zip were removed from history; only the final versions
are kept. The Codex merge commit is now attributed to Codex.

Co-Authored-By: Claude Opus 5.5 <noreply@anthropic.com>
Claude-Session: https://claude.ai/code/session_01W9CKpimWpgkUmrDQQMiKtF
Parts:
- removed C4420: 100 pF C0G 50 V, symbol sr_rx_v2_completed:C_C4420
- removed C4421: 10 nF C0G 50 V, symbol sr_rx_v2_completed:C_C4421
- removed D451: BAV199 sense clamps, Package_TO_SOT_SMD:SOT-23, symbol sr_rx_v2_completed:C_D451
- removed Q450: AO3400A, Package_TO_SOT_SMD:SOT-23, symbol sr_rx_v2_completed:C_Q450
- removed Q451: AO3400A, Package_TO_SOT_SMD:SOT-23, symbol sr_rx_v2_completed:C_Q451
- removed R435: 100kΩ 1%, symbol sr_rx_v2_completed:C_R435
- removed R440: 1kΩ 1%, symbol sr_rx_v2_completed:C_R440
- removed R441: 1kΩ 1%, symbol sr_rx_v2_completed:C_R441
- removed R442: 1kΩ 1%, symbol sr_rx_v2_completed:C_R442
- removed R4420: 24.9 kΩ 0.1% 0402 RF tap, symbol sr_rx_v2_completed:C_R4420
- removed R4421: 24.9 kΩ 0.1% 0402, symbol sr_rx_v2_completed:C_R4421
- removed R4422: 49.8 kΩ 0.1%, symbol sr_rx_v2_completed:C_R4422
- removed R4423: 100 Ω, symbol sr_rx_v2_completed:C_R4423
- removed R4424: 100 kΩ, symbol sr_rx_v2_completed:C_R4424
- removed R4425: 100 Ω, symbol sr_rx_v2_completed:C_R4425
- removed R4426: 100 kΩ, symbol sr_rx_v2_completed:C_R4426
- removed R443: 1kΩ 1%, symbol sr_rx_v2_completed:C_R443
- removed R444: 1kΩ 1%, symbol sr_rx_v2_completed:C_R444
- removed R445: 1kΩ 1%, symbol sr_rx_v2_completed:C_R445
- removed R4460: 249 Ω 1% ≥0.5 W, Resistor_SMD:R_1210_3225Metric, symbol sr_rx_v2_completed:C_R4460
- removed R4461: 249 Ω 1% ≥0.5 W, Resistor_SMD:R_1210_3225Metric, symbol sr_rx_v2_completed:C_R4461
- removed U405: HMC7992LP3DE A, symbol sr_rx_v2_completed:C_U405
- removed U406: HMC7992LP3DE B, symbol sr_rx_v2_completed:C_U406
- removed U407: HMC7992LP3DE C, symbol sr_rx_v2_completed:C_U407
- removed U450: TLV3012BIDBVR, Package_TO_SOT_SMD:SOT-23-6, symbol sr_rx_v2_completed:C_U450
- removed U451: TLV3012BIDBVR, Package_TO_SOT_SMD:SOT-23-6, symbol sr_rx_v2_completed:C_U451
- added C4430: 100 pF C0G 50 V, symbol sr_rx_v2_completed:C_C4430
- added C4431: 10 nF C0G 50 V, symbol sr_rx_v2_completed:C_C4431
- added D452: BAV199 sense clamps, Package_TO_SOT_SMD:SOT-23, symbol sr_rx_v2_completed:C_D452
- added Q452: AO3400A, Package_TO_SOT_SMD:SOT-23, symbol sr_rx_v2_completed:C_Q452
- added Q453: AO3400A, Package_TO_SOT_SMD:SOT-23, symbol sr_rx_v2_completed:C_Q453
- added R4430: 24.9 kΩ 0.1% 0402 RF tap, symbol sr_rx_v2_completed:C_R4430
- added R4431: 24.9 kΩ 0.1% 0402, symbol sr_rx_v2_completed:C_R4431
- added R4432: 49.8 kΩ 0.1%, symbol sr_rx_v2_completed:C_R4432
- added R4433: 100 Ω, symbol sr_rx_v2_completed:C_R4433
- added R4434: 100 kΩ, symbol sr_rx_v2_completed:C_R4434
- added R4435: 100 Ω, symbol sr_rx_v2_completed:C_R4435
- added R4436: 100 kΩ, symbol sr_rx_v2_completed:C_R4436
- added R4464: 249 Ω 1% ≥0.5 W, Resistor_SMD:R_1210_3225Metric, symbol sr_rx_v2_completed:C_R4464
- added R4465: 249 Ω 1% ≥0.5 W, Resistor_SMD:R_1210_3225Metric, symbol sr_rx_v2_completed:C_R4465
- added R4466: 249 Ω 1% ≥0.5 W, Resistor_SMD:R_1210_3225Metric, symbol sr_rx_v2_completed:C_R4466
- added R4467: 249 Ω 1% ≥0.5 W, Resistor_SMD:R_1210_3225Metric, symbol sr_rx_v2_completed:C_R4467
- added U452: TLV3012BIDBVR, Package_TO_SOT_SMD:SOT-23-6, symbol sr_rx_v2_completed:C_U452
- added U453: TLV3012BIDBVR, Package_TO_SOT_SMD:SOT-23-6, symbol sr_rx_v2_completed:C_U453
Connections:
- net 3V3_Q6A: now also U452.6 (V+), U453.6 (V+)
- net E4_DCS_HIGH: now also U453.3 (IN+)
- net E4_DCS_LOW: now also U452.4 (IN-)
- net E4_DCS_REF: now also D452.2 (K2), R4432.1
- net E4_DCS_RETURN: now also Q453.2 (S)
- net GND: now also C4430.2, C4431.2, D452.1 (A1), R4434.2, R4436.2, R4467.2, U452.2 (V-), U453.2 (V-)
- new net DCS_LBAND: Q452.3 (D)
- new net E4_DCS_LBAND_BLEED_1: R4464.2, R4465.1
- new net E4_DCS_LBAND_BLEED_2: R4465.2, R4466.1
- new net E4_DCS_LBAND_BLEED_3: R4466.2, R4467.1
- new net E4_DCS_LBAND_HIGH_GATE: Q453.1 (G), R4435.2, R4436.1
- new net E4_DCS_LBAND_HIGH_OK: R4435.1, U453.1 (OUT)
- new net E4_DCS_LBAND_LOW_GATE: Q452.1 (G), R4433.2, R4434.1
- new net E4_DCS_LBAND_LOW_OK: R4433.1, U452.1 (OUT)
- new net E4_DCS_LBAND_SENSE: C4431.1, D452.3 (K1_A2), R4431.2, R4432.2, U452.3 (IN+), U453.4 (IN-)
- new net E4_DCS_LBAND_SINK_MID: Q452.2 (S), Q453.3 (D)
- new net E4_DCS_LBAND_TAP: C4430.1, R4430.2, R4431.1
- new net E4_P3: R4430.1, R4464.1
Other:
- note added: "DC detectors: LBAND"
- note added: "E4 - РЧ-тракт: DC-розв'язка, перемикачі, приймачі (3/4)"
- note added: "E4-06 — OPEN, блокує випуск — STACK §5.3 (DC-sense); §8.1 HF-10"
- note added: "N-E4-01 — примітка — STACK §5.3 (DC-sense)"
- note added: "Three concrete protected bipolar DC-window detectors are designed; threshold, RF loading and power-off backfeed still need prototype qualification. Ворота (стенд): Verify each DCS LOW at 0 V and HIGH by ±0.100 V in both sweep directions over the admitted temperature/supply range; record thresholds/hysteresis. Test ±30 V limited foreign DC with Q6A ON/OFF and require 3V3_Q6A <0.1 V when OFF. Measu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"
- note added: "Дроти з'єднують контакти всередині функціональної групи; кожне дерево дротів має одну глобальну мітку з канонічною назвою мережі (рамка-стрілка — мережа виходить за межі групи, пряма рамка — мережа лише цієї групи). Однакові мітки з'єднані на всіх аркушах; земля — символ GND. Рамки OPEN — незакриті ворота з design/E#.json (повний реєстр: OPEN_ITEMS.md); «TBD» у значенні — STACK номіналу не задає,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"
- note added: "Позначення R44xx/C44xx (4400–4499) — задокументований розширений діапазон E4 для DC-детекторів (design/E4-review.md), щоб не перетинатися з E5. Решта позначень E4 — у діапазоні 400–499."
- note removed: "DC detectors: UHF"
- note removed: "E4 - РЧ-тракт: DC-розвʼязка, перемикачі, реле та приймачі (3/4)"
- note removed: "RF passives and drivers"
- note removed: "SP4T switches"
- note removed: "Мережі з однаковими глобальними мітками електрично з'єднані на всіх аркушах. Фізичні/функціональні контакти: див. design/ і OPEN_ITEMS.md."
- title: E4 - РЧ-тракт і DC-захист (3/4) -> E4 - РЧ-тракт: DC-розв'язка, перемикачі, приймачі (3/4)
- moved on the sheet: U456, U457, U458
