File: sat-receiver-audit/build/kicad/E4_03.kicad_sch (KiCad schematic)
At the start: 45 parts, among them Q452 AO3400A, Q453 AO3400A, Q456 AO3400A, Q457 AO3400A, U452 TLV3012BIDBVR, U453 TLV3012BIDBVR, U456 TLV3012BIDBVR, U457 TLV3012BIDBVR, U458 LM4040A20IDBZR 2.048 V 0.1% s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

Commit message: GENERATED: CAD, netlist, ERC, documents and re-frozen DC_CORE PCB chain from CI
Applied verbatim from the cad-regenerated artifacts of run 40087342176
(for source commit c17ae81) and run 40090126917 (for the review fixes,
source commit 4740951); KiCad 10.0.7, refreeze_pcb=true.

Co-Authored-By: Claude Opus 5.5 <noreply@anthropic.com>
Parts:
- added A409: BLK-89-S+, symbol sr_rx_v2_completed:C_A409
- added A410: ANNE-50+ 50 Ω load, symbol sr_rx_v2_completed:C_A410
- added A418: Uputronics 440 Rev 3.0 external LNA, symbol sr_rx_v2_completed:C_A418
- added A419: GOES / H1 / iO / active patch external LNA, symbol sr_rx_v2_completed:C_A419
- added J402: P2 UHF SMA: 4.3 V, symbol sr_rx_v2_completed:C_J402
- added J403: P3 L-band SMA: 4.3 V, symbol sr_rx_v2_completed:C_J403
- added J414: RX2 panel SMA, symbol sr_rx_v2_completed:C_J414
- added J415: REF IN panel SMA, symbol sr_rx_v2_completed:C_J415
- added J416: UHF antenna feed / A418 input interface, symbol sr_rx_v2_completed:C_J416
- added J417: L-band antenna feed / A419 input interface, symbol sr_rx_v2_completed:C_J417
- added W404: RX2 → Lime X4 MHF4 coax, symbol sr_rx_v2_completed:C_W404
- added W405: REF IN → J4 MHF4 coax, symbol sr_rx_v2_completed:C_W405
- added W406: CAB.01075 X1 → ANNE-50+ captive coax, symbol sr_rx_v2_completed:C_W406
Connections:
- net E4_P3: now also A419.OUT, J403.CENTER
- net GND: now also A409.SHIELDS, A410.END_B, A418.SHIELDS, A419.SHIELDS, J402.SHIELD, J403.SHIELD, J414.SHIELD, J415.SHIELD, J416.SHIELD, J417.SHIELD, W404.SHIELDS, W405.SHIELDS, W406.SHIELDS
- new net E4_LIME_REF: W405.END_B
- new net E4_LIME_RX2: A409.IN, J414.CENTER
- new net E4_LIME_TX: W406.END_A
- new net E4_LIME_X4_RX: W404.END_B
- new net E4_P2: A418.OUT, J402.CENTER
- new net E4_P2_ANT: A418.IN, J416.CENTER
- new net E4_P3_ANT: A419.IN, J417.CENTER
- new net E4_REF_IN: J415.CENTER, W405.END_A
- new net E4_RX2_BLK: A409.OUT, W404.END_A
- new net E4_TX_LOAD: A410.END_A, W406.END_B
Other:
- note added: "RF and receiver interfaces (продовження)"
- note added: "Three concrete protected bipolar DC-window detectors are designed; threshold, RF loading and power-off backfeed still need prototype qualification. v2.1 (owner decision): each sensed bias branch has an E2 back-to-back P-MOSFET blocking element (Q2901/Q2902/Q2903 DMP6050SSD-13 with a 100 nF gate-source capacitor, held open by low EN_LNA2/EN_LNA3/EN_BONI) between the protected E2 node (TPS2553/INA3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"
- note removed: "Three concrete protected bipolar DC-window detectors are designed; threshold, RF loading and power-off backfeed still need prototype qualification. The ±30 V foreign-DC envelope covers the detector tap only: the assembled P2/P3/HF_CM ports share their DC node with E2 TPS2553/INA3221/U214 and polarized capacitors, which own bias OFF does not isolate, so a hardware blocking element is required. Вор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"
- moved on the sheet: C4400, C4401, C4402, C4403, C4404, C4405, C4406, C4430, C4431, D450, D452, Q452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
