File: sat-receiver-audit/build/kicad/E4_03.kicad_sch (KiCad schematic)
At the start: 45 parts, among them Q452 AO3400A, Q453 AO3400A, Q456 AO3400A, Q457 AO3400A, U452 TLV3012BIDBVR, U453 TLV3012BIDBVR, U456 TLV3012BIDBVR, U457 TLV3012BIDBVR, U458 LM4040A20IDBZR 2.048 V 0.1% s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

Commit message: Stage 2 integration: CAD and DC_CORE re-freeze from CI run 40094234222; bound-count test and PCB hash lists follow
Co-Authored-By: Claude Opus 5.5 <noreply@anthropic.com>
Other:
- note added: "Three concrete protected bipolar DC-window detectors are designed; threshold, RF loading and power-off backfeed still need prototype qualification. v2.1 (owner decision): each sensed bias branch has an E2 back-to-back P-MOSFET blocking element (Q2901/Q2902/Q2903 DMP6050SSD-13 with a 100 nF gate-source capacitor, held open by low EN_LNA2/EN_LNA3/EN_BONI) between the protected E2 node (TPS2553/INA3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"
- note removed: "Three concrete protected bipolar DC-window detectors are designed; threshold, RF loading and power-off backfeed still need prototype qualification. The ±30 V foreign-DC envelope covers the detector tap only: the assembled P2/P3/HF_CM ports share their DC node with E2 TPS2553/INA3221/U214 and polarized capacitors, which own bias OFF does not isolate, so a hardware blocking element is required. Вор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"
- moved on the sheet: C4400, C4401, C4402, C4403, C4404, C4405, C4406, C4430, C4431, D450, D452, Q452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
