File: sat-receiver-audit/build/kicad/E4_04.kicad_sch (KiCad schematic)
At the start: 52 parts, among them Q452 AO3400A, Q453 AO3400A, Q454 AO3400A, Q455 AO3400A, U452 TLV3012BIDBVR, U453 TLV3012BIDBVR, U454 TLV3012BIDBVR, U455 TLV3012BIDBVR

Commit message: SR-RX-v2.1: review fixes on the Codex branch, readable schematic, one-file bundle
Independent review of the Codex branch (schematic vs STACK.md, hard rules,
security, tests) found no blockers; this commit applies its findings:

- rules in code: Cospas-Sarsat 406.0-406.1 MHz added to the no-data mask;
  Q6A Wi-Fi/BT off in the field/QUIET root (modprobe blacklist, udev
  authorized=0 on FE1.1s port 4, rfkill) with self-checks; device denylist
  completed per STACK (gr-gsm, gr-iridium, kalibrate, pager/trunking decoders,
  TX-capable tools); W1-2 WIFI_PWR_EN as blocking open item E5-10
- STACK.md is the source of truth again; v2.1 changes recorded in it; the
  "historical" marker kept only on ISDT/raw-balance rows; gender-neutral wording
- schematic data: open values shown as TBD with start values and notes, U503
  TPS2553DBVR-1, Lime X2/X4 RX mapping TBD, 37 open items drawn on the sheets
- schematic readability: wired groups, junctions, GND symbols, standard
  transistor/diode symbols; netlist unchanged (603 nets identical)
- tooling: reproducible run_checks (no timestamps or machine paths), pinned
  dependencies, bundle excludes cache folders, clean-checkout bundle check
- regenerated: KiCad export (14 pages), netlist/ERC, module lab, PCB inputs,
  readiness contract, acceptance hashes, SR-RX-v2-ves-proekt.html

Checks: ERC 0 errors/0 warnings, netlist comparison PASS, 432 tests (431
passed, 1 skipped), deployment tests OK, bundle check PASS on a clean checkout.

History note: earlier versions of the generated SR-RX-v2-ves-proekt.html and
handoff/handoff-bundle.zip were removed from history; only the final versions
are kept. The Codex merge commit is now attributed to Codex.

Co-Authored-By: Claude Opus 5.5 <noreply@anthropic.com>
Claude-Session: https://claude.ai/code/session_01W9CKpimWpgkUmrDQQMiKtF
Parts:
- removed C4410: 100 nF X7R 10 V local decoupling, symbol sr_rx_v2_completed:C_C4410
- removed C4411: 100 nF X7R 10 V local decoupling, symbol sr_rx_v2_completed:C_C4411
- removed C4412: 100 nF X7R 10 V local decoupling, symbol sr_rx_v2_completed:C_C4412
- removed C4413: 100 nF X7R 10 V local decoupling, symbol sr_rx_v2_completed:C_C4413
- removed C4414: 100 nF X7R 10 V local decoupling, symbol sr_rx_v2_completed:C_C4414
- removed C4415: 100 nF X7R 10 V local decoupling, symbol sr_rx_v2_completed:C_C4415
- removed C4416: 100 nF X7R 10 V local decoupling, symbol sr_rx_v2_completed:C_C4416
- removed C4417: 100 nF X7R 10 V local decoupling, symbol sr_rx_v2_completed:C_C4417
- removed C4430: 100 pF C0G 50 V, symbol sr_rx_v2_completed:C_C4430
- removed C4431: 10 nF C0G 50 V, symbol sr_rx_v2_completed:C_C4431
- removed C447: 100 pF C0G 50 V, symbol sr_rx_v2_completed:C_C447
- removed C448: 10 nF C0G 50 V, symbol sr_rx_v2_completed:C_C448
- removed C449: 100 pF C0G 50 V, symbol sr_rx_v2_completed:C_C449
- removed C450: 10 nF C0G 50 V, symbol sr_rx_v2_completed:C_C450
- removed C451: 100 pF C0G 50 V, symbol sr_rx_v2_completed:C_C451
- removed C452: 10 nF C0G 50 V, symbol sr_rx_v2_completed:C_C452
- removed D452: BAV199 sense clamps, Package_TO_SOT_SMD:SOT-23, symbol sr_rx_v2_completed:C_D452
- removed Q452: AO3400A, Package_TO_SOT_SMD:SOT-23, symbol sr_rx_v2_completed:C_Q452
- removed Q453: AO3400A, Package_TO_SOT_SMD:SOT-23, symbol sr_rx_v2_completed:C_Q453
- removed R4430: 24.9 kΩ 0.1% 0402 RF tap, symbol sr_rx_v2_completed:C_R4430
- removed R4431: 24.9 kΩ 0.1% 0402, symbol sr_rx_v2_completed:C_R4431
- removed R4432: 49.8 kΩ 0.1%, symbol sr_rx_v2_completed:C_R4432
- removed R4433: 100 Ω, symbol sr_rx_v2_completed:C_R4433
- removed R4434: 100 kΩ, symbol sr_rx_v2_completed:C_R4434
- removed R4435: 100 Ω, symbol sr_rx_v2_completed:C_R4435
- removed R4436: 100 kΩ, symbol sr_rx_v2_completed:C_R4436
- removed R4464: 249 Ω 1% ≥0.5 W, Resistor_SMD:R_1210_3225Metric, symbol sr_rx_v2_completed:C_R4464
- removed R4465: 249 Ω 1% ≥0.5 W, Resistor_SMD:R_1210_3225Metric, symbol sr_rx_v2_completed:C_R4465
- removed R4466: 249 Ω 1% ≥0.5 W, Resistor_SMD:R_1210_3225Metric, symbol sr_rx_v2_completed:C_R4466
- removed R4467: 249 Ω 1% ≥0.5 W, Resistor_SMD:R_1210_3225Metric, symbol sr_rx_v2_completed:C_R4467
- removed U452: TLV3012BIDBVR, Package_TO_SOT_SMD:SOT-23-6, symbol sr_rx_v2_completed:C_U452
- removed U453: TLV3012BIDBVR, Package_TO_SOT_SMD:SOT-23-6, symbol sr_rx_v2_completed:C_U453
- added C4420: 100 pF C0G 50 V, symbol sr_rx_v2_completed:C_C4420
- added C4421: 10 nF C0G 50 V, symbol sr_rx_v2_completed:C_C4421
- added D451: BAV199 sense clamps, Package_TO_SOT_SMD:SOT-23, symbol sr_rx_v2_completed:C_D451
- added Q450: AO3400A, Package_TO_SOT_SMD:SOT-23, symbol sr_rx_v2_completed:C_Q450
- added Q451: AO3400A, Package_TO_SOT_SMD:SOT-23, symbol sr_rx_v2_completed:C_Q451
- added R4420: 24.9 kΩ 0.1% 0402 RF tap, symbol sr_rx_v2_completed:C_R4420
- added R4421: 24.9 kΩ 0.1% 0402, symbol sr_rx_v2_completed:C_R4421
- added R4422: 49.8 kΩ 0.1%, symbol sr_rx_v2_completed:C_R4422
- added R4423: 100 Ω, symbol sr_rx_v2_completed:C_R4423
- added R4424: 100 kΩ, symbol sr_rx_v2_completed:C_R4424
- added R4425: 100 Ω, symbol sr_rx_v2_completed:C_R4425
- added R4426: 100 kΩ, symbol sr_rx_v2_completed:C_R4426
- added R4460: 249 Ω 1% ≥0.5 W, Resistor_SMD:R_1210_3225Metric, symbol sr_rx_v2_completed:C_R4460
- added R4461: 249 Ω 1% ≥0.5 W, Resistor_SMD:R_1210_3225Metric, symbol sr_rx_v2_completed:C_R4461
- added U450: TLV3012BIDBVR, Package_TO_SOT_SMD:SOT-23-6, symbol sr_rx_v2_completed:C_U450
- added U451: TLV3012BIDBVR, Package_TO_SOT_SMD:SOT-23-6, symbol sr_rx_v2_completed:C_U451
Connections:
- net 3V3_Q6A: now also U450.6 (V+), U451.6 (V+)
- net E4_DCS_HIGH: now also U451.3 (IN+)
- net E4_DCS_LOW: now also U450.4 (IN-)
- net E4_DCS_REF: now also D451.2 (K2), R4422.1
- net E4_DCS_RETURN: now also Q451.2 (S)
- net E4_DCS_UHF_BLEED_2: now also R4461.2
- net GND: now also C4420.2, C4421.2, D451.1 (A1), R4424.2, R4426.2, U450.2 (V-), U451.2 (V-)
- new net DCS_UHF: Q450.3 (D)
- new net E4_DCS_UHF_BLEED_1: R4460.2, R4461.1
- new net E4_DCS_UHF_HIGH_GATE: Q451.1 (G), R4425.2, R4426.1
- new net E4_DCS_UHF_HIGH_OK: R4425.1, U451.1 (OUT)
- new net E4_DCS_UHF_LOW_GATE: Q450.1 (G), R4423.2, R4424.1
- new net E4_DCS_UHF_LOW_OK: R4423.1, U450.1 (OUT)
- new net E4_DCS_UHF_SENSE: C4421.1, D451.3 (K1_A2), R4421.2, R4422.2, U450.3 (IN+), U451.4 (IN-)
- new net E4_DCS_UHF_SINK_MID: Q450.2 (S), Q451.3 (D)
- new net E4_DCS_UHF_TAP: C4420.1, R4420.2, R4421.1
- new net E4_P2: R4420.1, R4460.1
Other:
- note added: "E4 - РЧ-тракт: DC-розв'язка, перемикачі, приймачі (4/4)"
- note added: "Дроти з'єднують контакти всередині функціональної групи; кожне дерево дротів має одну глобальну мітку з канонічною назвою мережі (рамка-стрілка — мережа виходить за межі групи, пряма рамка — мережа лише цієї групи). Однакові мітки з'єднані на всіх аркушах; земля — символ GND. Рамки OPEN — незакриті ворота з design/E#.json (повний реєстр: OPEN_ITEMS.md); «TBD» у значенні — STACK номіналу не задає,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"
- note removed: "DC detectors: LBAND"
- note removed: "DC detectors: local power"
- note removed: "E4 - РЧ-тракт: DC-розвʼязка, перемикачі, реле та приймачі (4/4)"
- note removed: "RF bias injector local decoupling"
- note removed: "Мережі з однаковими глобальними мітками електрично з'єднані на всіх аркушах. Фізичні/функціональні контакти: див. design/ і OPEN_ITEMS.md."
- title: E4 - РЧ-тракт і DC-захист (4/4) -> E4 - РЧ-тракт: DC-розв'язка, перемикачі, приймачі (4/4)
- moved on the sheet: U454, U455
