File: sat-receiver-audit/build/kicad/E5_02.kicad_sch (KiCad schematic)
At the start: 24 parts, among them J502 UART5 console 3pin locking, J504 Olimex GX16-4 IMU DESIGN pino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, J505 LAB BUS 6pin locking DESIGN, J522 Q6A factory EDL button functi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, J530 Q6A MKEY host lane0 functiona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, J550 IMU pack cable termination DE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, SW501 EDL recessed momentary NO, U506 LM66100DCKR HDMI5V ideal diode, U507 TCA9517DR, U520 Wisecoco display/controller a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, U530 ADT-Link R44SF 5cm modified r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, U551 TPD4E1U06DBVR, U552 TPD4E1U06DBVR

Commit message: SR-RX-v2.1: review fixes on the Codex branch, readable schematic, one-file bundle
Independent review of the Codex branch (schematic vs STACK.md, hard rules,
security, tests) found no blockers; this commit applies its findings:

- rules in code: Cospas-Sarsat 406.0-406.1 MHz added to the no-data mask;
  Q6A Wi-Fi/BT off in the field/QUIET root (modprobe blacklist, udev
  authorized=0 on FE1.1s port 4, rfkill) with self-checks; device denylist
  completed per STACK (gr-gsm, gr-iridium, kalibrate, pager/trunking decoders,
  TX-capable tools); W1-2 WIFI_PWR_EN as blocking open item E5-10
- STACK.md is the source of truth again; v2.1 changes recorded in it; the
  "historical" marker kept only on ISDT/raw-balance rows; gender-neutral wording
- schematic data: open values shown as TBD with start values and notes, U503
  TPS2553DBVR-1, Lime X2/X4 RX mapping TBD, 37 open items drawn on the sheets
- schematic readability: wired groups, junctions, GND symbols, standard
  transistor/diode symbols; netlist unchanged (603 nets identical)
- tooling: reproducible run_checks (no timestamps or machine paths), pinned
  dependencies, bundle excludes cache folders, clean-checkout bundle check
- regenerated: KiCad export (14 pages), netlist/ERC, module lab, PCB inputs,
  readiness contract, acceptance hashes, SR-RX-v2-ves-proekt.html

Checks: ERC 0 errors/0 warnings, netlist comparison PASS, 432 tests (431
passed, 1 skipped), deployment tests OK, bundle check PASS on a clean checkout.

History note: earlier versions of the generated SR-RX-v2-ves-proekt.html and
handoff/handoff-bundle.zip were removed from history; only the final versions
are kept. The Codex merge commit is now attributed to Codex.

Co-Authored-By: Claude Opus 5.5 <noreply@anthropic.com>
Claude-Session: https://claude.ai/code/session_01W9CKpimWpgkUmrDQQMiKtF
Parts:
- removed C550: 100nF X7R 10V, symbol sr_rx_v2_completed:C_C550
- removed C551: 100nF X7R 10V, symbol sr_rx_v2_completed:C_C551
- removed J530: Q6A MKEY host lane0 functional interface, symbol sr_rx_v2_completed:C_J530
- removed R550: 4.7k 1%, Resistor_SMD:R_0603_1608Metric, symbol sr_rx_v2_completed:C_R550
- removed R551: 4.7k 1%, Resistor_SMD:R_0603_1608Metric, symbol sr_rx_v2_completed:C_R551
- removed U507: TCA9517DR, Package_SO:SOIC-8_3.9x4.9mm_P1.27mm, symbol sr_rx_v2_completed:C_U507
- removed U530: ADT-Link R44SF 5cm modified riser, symbol sr_rx_v2_completed:C_U530
- added J520: Q6A HDMI Type-A existing port, symbol sr_rx_v2_completed:C_J520
Connections:
- net E5_HDMI_5V_Q6A: now also J520.18 (+5V)
- net E5_HDMI_CEC: now also J520.13 (CEC)
- net E5_HDMI_CLK_N: now also J520.12 (TMDSCLK−)
- net E5_HDMI_CLK_P: now also J520.10 (TMDSCLK+)
- net E5_HDMI_D0_N: now also J520.9 (TMDS0−)
- net E5_HDMI_D0_P: now also J520.7 (TMDS0+)
- net E5_HDMI_D1_N: now also J520.6 (TMDS1−)
- net E5_HDMI_D1_P: now also J520.4 (TMDS1+)
- net E5_HDMI_D2_N: now also J520.3 (TMDS2−)
- net E5_HDMI_D2_P: now also J520.1 (TMDS2+)
- net E5_HDMI_HPD: now also J520.19 (HPD)
- net E5_HDMI_SCL: now also J520.15 (DDC SCL)
- net E5_HDMI_SDA: now also J520.16 (DDC SDA)
- net GND: now also J520.11 (TMDSCLK shield), J520.17 (DDC ground), J520.2 (TMDS2 shield), J520.5 (TMDS1 shield), J520.8 (TMDS0 shield)
Other:
- note added: "E5-01 — OPEN, блокує випуск — STACK §2.6; §8 (плата дисплея, D5)"
- note added: "E5-02 — OPEN, блокує випуск — STACK §2.8; §5.2; §8 (пак IMU)"
- note added: "E5-06 — OPEN, блокує випуск — STACK §5.2; §8 (зворотне живлення)"
- note added: "E5-07 — OPEN, блокує випуск — STACK §5.2; §8.1 (EDL)"
- note added: "E5-08 — OPEN, блокує випуск — STACK §2.9; §5.8"
- note added: "EDL factory button pads and cable orientation not physically located on the exact received Q6A. Ворота (стенд): Use the factory button first; continuity-identify its two switch nets before fitting parallel SW501. Unplug T7 for EDL and confirm 05c6:9008."
- note added: "HDMI/display/hub and receiver backfeed paths through signal lines need physical power-state validation. Ворота (стенд): Verify Q6A off / LAB5 on / display on combinations using DMM/FNB58. Q6A HDMI 5 V and Q6A USB VBUS should remain 0 V within measurement resolution. Check DDC/HPD after U506 installation and no phantom receiver power."
- note added: "IMU cable and exact received board revisions are unverified physical assemblies; E3 now defines RP2040-Zero/BNO085 internal wiring. Ворота (стенд): Verify E3 board-pad map on received revisions; confirm chosen GX16 harness orientation, 3.3V UART and diode-fed E5_IMU_VIN; run 1e6 CRC-clean frames and 100 cold starts."
- note added: "Project locking connector/GX16 numbers have been assigned but final keyed part footprints/orientation and wire lengths are not released. Ворота (стенд): Record exact supplier part numbers, face-view and wire-color tables; no-power continuity plus first energization current limit."
- note added: "Received Wisecoco board DC barrel size/polarity and USBTP/USB-C touch wiring still undocumented; no-VBUS enumeration must work. Ворота (стенд): Obtain the exact board photo/schematic, DMM mapping, vendor confirmation and enumerate with only D+/D−/GND. Never substitute guessed connector numbering."
- note added: "Дроти з'єднують контакти всередині функціональної групи; кожне дерево дротів має одну глобальну мітку з канонічною назвою мережі (рамка-стрілка — мережа виходить за межі групи, пряма рамка — мережа лише цієї групи). Однакові мітки з'єднані на всіх аркушах; земля — символ GND. Рамки OPEN — незакриті ворота з design/E#.json (повний реєстр: OPEN_ITEMS.md); «TBD» у значенні — STACK номіналу не задає,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"
- note removed: "LAB BUS I2C buffer"
- note removed: "PCIe x1 riser та Lime"
- note removed: "Мережі з однаковими глобальними мітками електрично з'єднані на всіх аркушах. Фізичні/функціональні контакти: див. design/ і OPEN_ITEMS.md."
- note removed: "Позначення фізичних джерел живлення (ERC)"
- moved on the sheet: J502, J504, J505, J522, J550, U506, U520, U551, U552
