File: sat-receiver-audit/build/kicad/E4_02.kicad_sch (KiCad schematic)
At the start: 58 parts, among them J422 Existing S-band helix feed SMA, K401 G6K-2F-RF-S DC5 HF, K402 G6K-2F-RF-S DC5 VHF, Q401 AO3400A, Q402 AO3400A

Commit message: SR-RX-v2.1: review fixes on the Codex branch, readable schematic, one-file bundle
Independent review of the Codex branch (schematic vs STACK.md, hard rules,
security, tests) found no blockers; this commit applies its findings:

- rules in code: Cospas-Sarsat 406.0-406.1 MHz added to the no-data mask;
  Q6A Wi-Fi/BT off in the field/QUIET root (modprobe blacklist, udev
  authorized=0 on FE1.1s port 4, rfkill) with self-checks; device denylist
  completed per STACK (gr-gsm, gr-iridium, kalibrate, pager/trunking decoders,
  TX-capable tools); W1-2 WIFI_PWR_EN as blocking open item E5-10
- STACK.md is the source of truth again; v2.1 changes recorded in it; the
  "historical" marker kept only on ISDT/raw-balance rows; gender-neutral wording
- schematic data: open values shown as TBD with start values and notes, U503
  TPS2553DBVR-1, Lime X2/X4 RX mapping TBD, 37 open items drawn on the sheets
- schematic readability: wired groups, junctions, GND symbols, standard
  transistor/diode symbols; netlist unchanged (603 nets identical)
- tooling: reproducible run_checks (no timestamps or machine paths), pinned
  dependencies, bundle excludes cache folders, clean-checkout bundle check
- regenerated: KiCad export (14 pages), netlist/ERC, module lab, PCB inputs,
  readiness contract, acceptance hashes, SR-RX-v2-ves-proekt.html

Checks: ERC 0 errors/0 warnings, netlist comparison PASS, 432 tests (431
passed, 1 skipped), deployment tests OK, bundle check PASS on a clean checkout.

History note: earlier versions of the generated SR-RX-v2-ves-proekt.html and
handoff/handoff-bundle.zip were removed from history; only the final versions
are kept. The Codex merge commit is now attributed to Codex.

Co-Authored-By: Claude Opus 5.5 <noreply@anthropic.com>
Claude-Session: https://claude.ai/code/session_01W9CKpimWpgkUmrDQQMiKtF
Parts:
- added A410: ANNE-50+ 50 Ω load, symbol sr_rx_v2_completed:C_A410
- added A418: Uputronics 440 Rev 3.0 external LNA, symbol sr_rx_v2_completed:C_A418
- added A419: GOES / H1 / iO / active patch external LNA, symbol sr_rx_v2_completed:C_A419
- added A422: Nooelec LaNA WB 100845, symbol sr_rx_v2_completed:C_A422
- added A423: sysmocom cf2235-kt30 2170–2300 MHz, symbol sr_rx_v2_completed:C_A423
- added C4410: 100 nF X7R 10 V local decoupling, symbol sr_rx_v2_completed:C_C4410
- added C4411: 100 nF X7R 10 V local decoupling, symbol sr_rx_v2_completed:C_C4411
- added C4412: 100 nF X7R 10 V local decoupling, symbol sr_rx_v2_completed:C_C4412
- added C4413: 100 nF X7R 10 V local decoupling, symbol sr_rx_v2_completed:C_C4413
- added C4414: 100 nF X7R 10 V local decoupling, symbol sr_rx_v2_completed:C_C4414
- added C4415: 100 nF X7R 10 V local decoupling, symbol sr_rx_v2_completed:C_C4415
- added C4416: 100 nF X7R 10 V local decoupling, symbol sr_rx_v2_completed:C_C4416
- added C4417: 100 nF X7R 10 V local decoupling, symbol sr_rx_v2_completed:C_C4417
- added J402: P2 UHF SMA: 4.5 V, symbol sr_rx_v2_completed:C_J402
- added J403: P3 L-band SMA: 4.5 V, symbol sr_rx_v2_completed:C_J403
- added J416: UHF antenna feed / A418 input interface, symbol sr_rx_v2_completed:C_J416
- added J417: L-band antenna feed / A419 input interface, symbol sr_rx_v2_completed:C_J417
- added R435: 100kΩ 1%, symbol sr_rx_v2_completed:C_R435
- added R440: 1kΩ 1%, symbol sr_rx_v2_completed:C_R440
- added R441: 1kΩ 1%, symbol sr_rx_v2_completed:C_R441
- added R442: 1kΩ 1%, symbol sr_rx_v2_completed:C_R442
- added R443: 1kΩ 1%, symbol sr_rx_v2_completed:C_R443
- added R444: 1kΩ 1%, symbol sr_rx_v2_completed:C_R444
- added R445: 1kΩ 1%, symbol sr_rx_v2_completed:C_R445
- added U405: HMC7992LP3DE A, symbol sr_rx_v2_completed:C_U405
- added U406: HMC7992LP3DE B, symbol sr_rx_v2_completed:C_U406
- added U407: HMC7992LP3DE C, symbol sr_rx_v2_completed:C_U407
- added W406: CAB.01075 X1 → ANNE-50+ captive coax, symbol sr_rx_v2_completed:C_W406
- added W422: RG316 SMA-M/M 0.10 m helix → LaNA, symbol sr_rx_v2_completed:C_W422
- added W423: RG316 SMA-M/M 0.10 m LaNA → DC block, symbol sr_rx_v2_completed:C_W423
- added W424: RG316 SMA-M/M 1.00 m pod → RX2, symbol sr_rx_v2_completed:C_W424
- C440, C441, C442: value 100 nF X7R 10 V -> 100 nF X7R 10 V
- R408, R409, R410, R411, R414, R415, R434: value 100kΩ 1% -> 100kΩ 1%
- R412, R413: value 100Ω -> 100Ω
Connections:
- net 3V3_Q6A: now also C4410.1, C4411.1, C4412.1, C4413.1, C4414.1, C4415.1, C4416.1, C4417.1, U405.6 (VDD), U406.6 (VDD), U407.6 (VDD)
- net E4_LIME_CTL_A: now also R444.2, U407.8 (A)
- net E4_LIME_CTL_B: now also R435.1, R445.2, U407.7 (B)
- net E4_LIME_RF1: now also U407.12 (RF1)
- net E4_LIME_RF3: now also U407.4 (RF3)
- net E4_LIME_RFC: now also U407.15 (RFC)
- net E4_LIME_RFSPARE: now also U407.1 (RF4)
- net E4_LIME_TO_RTLB: now also U407.9 (RF2)
- net E4_P2: now also A418.OUT, J402.CENTER
- net E4_P3: now also A419.OUT, J403.CENTER
- net E4_RTLA_CTL_A: now also R440.2, U405.8 (A)
- net E4_RTLA_CTL_B: now also R441.2, U405.7 (B)
- net E4_RTLA_RF1: now also U405.12 (RF1)
- net E4_RTLA_RF2: now also U405.9 (RF2)
- net E4_RTLA_RF3: now also U405.4 (RF3)
- net E4_RTLA_RF4: now also U405.1 (RF4)
- net E4_RTLA_RFC: now also U405.15 (RFC)
- net E4_RTLB_CTL_A: now also R442.2, U406.8 (A)
- net E4_RTLB_CTL_B: now also R443.2, U406.7 (B)
- net E4_RTLB_RF1: now also U406.12 (RF1)
- net E4_RTLB_RF2: now also U406.9 (RF2)
- net E4_RTLB_RF3: now also U406.4 (RF3)
- net E4_RTLB_RF4: now also U406.1 (RF4)
- net E4_RTLB_RFC: now also U406.15 (RFC)
- net E4_RX2_ANT: now also W422.ANT
- net E4_SB_FILTER_IN: now also A423.SMA_F_A
- net E4_SB_POD5: now also A422.USB_C_VBUS
- net E4_SB_PREBLOCK: now also W423.BLOCK
- net GND: now also A410.END_B, A418.SHIELDS, A419.SHIELDS, A422.SHIELDS, A422.USB_C_GND, A423.SHIELDS, C4410.2, C4411.2, C4412.2, C4413.2, C4414.2, C4415.2, C4416.2, C4417.2, J402.SHIELD, J403.SHIELD, J416.SHIELD, J417.SHIELD, R435.2, U405.10 (GND), U405.11 (GND), U405.13 (GND), U405.14 (GND), U405.16 (GND), U405.2 (GND), U405.3 (GND), U405.5 (GND), U405.EPAD, U406.10 (GND), U406.11 (GND), U406.13 (GND), U406.14 (GND), U406.16 (GND), U406.2 (GND), U406.3 (GND), U406.5 (GND), U406.EPAD, U407.10 (GND), U407.11 (GND), U407.13 (GND), U407.14 (GND), U407.16 (GND), U407.2 (GND), U407.3 (GND), U407.5 (GND), U407.EPAD, W406.SHIELDS, W422.SHIELDS, W423.SHIELDS, W424.SHIELDS
- new net E4_LIME_RX2: W424.PANEL
- new net E4_LIME_TX: W406.END_A
- new net E4_P2_ANT: A418.IN, J416.CENTER
- new net E4_P3_ANT: A419.IN, J417.CENTER
- new net E4_SB_FILTER_OUT: A423.SMA_F_B, W424.FILTER
- new net E4_SB_LNA_IN: A422.SMA_IN, W422.LNA
- new net E4_SB_LNA_OUT: A422.SMA_OUT, W423.LNA
- new net E4_TX_LOAD: A410.END_A, W406.END_B
- new net SW_LIME_A: R444.1
- new net SW_LIME_B: R445.1
- new net SW_RTLA_A: R440.1
- new net SW_RTLA_B: R441.1
- new net SW_RTLB_A: R442.1
- new net SW_RTLB_B: R443.1
Other:
- note added: "DC detectors: local power"
- note added: "E4 - РЧ-тракт: DC-розв'язка, перемикачі, приймачі (2/4)"
- note added: "E4-01 — OPEN, блокує випуск — STACK §5.3; §8 (РЧ-деталі); §8.1 RF-10"
- note added: "E4-04 — OPEN, блокує випуск — STACK §5.3 (S-band); поправки v2.1 (LaNA WB, cf2235-kt30)"
- note added: "E4-07 — OPEN, блокує випуск — STACK §5.3; §8 (HMC7992LP3DE; G6K-2F-RF-S); §8.1 RF-0/RF-1, HF-13"
- note added: "RF PCB, relay insertion loss, isolation, return loss and startup PARK are unmeasured. Ворота (стенд): VNA: HF selector 10 kHz–260 MHz IL ≤0.3 dB, RL ≥21 dB, isolation ≥35 dB at 162–260 MHz plus STACK LF/HF gates. HMC ≥40 dB isolation at 0.1–1.7 GHz (37–40 dB conditional and recorded); verify all DC blocks and startup. Check all SMT footprint pad numbers, dimensions, orientation and ground/exposed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"
- note added: "RF and receiver interfaces (продовження)"
- note added: "S-band module and supply selection are complete; external inline pod assembly, cable loss, gain/NF and thermal/current measurements remain unqualified. Ворота (стенд): Build the specified LaNA WB 100845 + cf2235 + DC blocks in the Hammond 1554U2GY pod; verify stacked fit/cable bends, weather seals and strain relief. Measure LaNA current/inrush at protected 5 V, 2.2–2.3 GHz S21/NF/linearity, and r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"
- note added: "SP4T switches"
- note added: "ch1–3 injector choke part selection is complete; final DC drop, thermal rise, RF impedance and footprint qualification remain open. Optional static bleeds stay DNP. Ворота (стенд): Verify selected 0805LS-471XGRC / 0805HP-221XGRC / 0603HP-47NXGRW manufacturer land patterns and target-band impedance under bias. VNA qualify IL/RL/isolation and DC heating at actual/worst protected current. The curren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"
- note added: "Дроти з'єднують контакти всередині функціональної групи; кожне дерево дротів має одну глобальну мітку з канонічною назвою мережі (рамка-стрілка — мережа виходить за межі групи, пряма рамка — мережа лише цієї групи). Однакові мітки з'єднані на всіх аркушах; земля — символ GND. Рамки OPEN — незакриті ворота з design/E#.json (повний реєстр: OPEN_ITEMS.md); «TBD» у значенні — STACK номіналу не задає,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"
- note removed: "E4 - РЧ-тракт: DC-розвʼязка, перемикачі, реле та приймачі (2/4)"
- note removed: "Мережі з однаковими глобальними мітками електрично з'єднані на всіх аркушах. Фізичні/функціональні контакти: див. design/ і OPEN_ITEMS.md."
- title: E4 - РЧ-тракт і DC-захист (2/4) -> E4 - РЧ-тракт: DC-розв'язка, перемикачі, приймачі (2/4)
- moved on the sheet: K401, K402

Commit message: Stage 2 integration: CAD and DC_CORE re-freeze from CI run 40094234222; bound-count test and PCB hash lists follow
Co-Authored-By: Claude Opus 5.5 <noreply@anthropic.com>
Parts:
- removed A410: ANNE-50+ 50 Ω load, symbol sr_rx_v2_completed:C_A410
- removed A418: Uputronics 440 Rev 3.0 external LNA, symbol sr_rx_v2_completed:C_A418
- removed A419: GOES / H1 / iO / active patch external LNA, symbol sr_rx_v2_completed:C_A419
- removed J402: P2 UHF SMA: 4.5 V, symbol sr_rx_v2_completed:C_J402
- removed J403: P3 L-band SMA: 4.5 V, symbol sr_rx_v2_completed:C_J403
- removed J416: UHF antenna feed / A418 input interface, symbol sr_rx_v2_completed:C_J416
- removed J417: L-band antenna feed / A419 input interface, symbol sr_rx_v2_completed:C_J417
- removed W406: CAB.01075 X1 → ANNE-50+ captive coax, symbol sr_rx_v2_completed:C_W406
Connections:
- net BIAS_CH2 renamed BIAS_CH2_PORT
- net BIAS_CH3 renamed BIAS_CH3_PORT
Other:
- note removed: "RF and receiver interfaces (продовження)"
- moved on the sheet: A422, A423, A425, C401, C406, C412, C414, C415, C417, C418, C419, C420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
